File: hardware/kajikia/driver_output.sch (KiCad schematic (older format))
At the start: 21 parts

Commit message: io assignments
Parts:
- C20, C21, C22, C23, C24, C25, C26: renamed from C?; footprint (none) -> _Generic:0603_Small
- D1, D2, D3: renamed from D?; footprint (none) -> Diode_SMD:D_SOD-123
- Q1, Q2: renamed from Q?; footprint (none) -> Package_SO:SOIC-8_3.9x4.9mm_P1.27mm
- R10, R2, R3, R4, R5, R6, R7, R8, R9: renamed from R?; footprint (none) -> _Generic:0603_Small
