File: hardware/kajikia/connector.sch (KiCad schematic (older format))
At the start: 66 parts

Commit message: power
Parts:
- removed D? (x4): D_Schottky_Small, symbol Device:D_Schottky_Small
- removed J? (x3): Conn_01x04, symbol Connector_Generic:Conn_01x04
- removed JP? (x2): SolderJumper_3_Open, symbol #PCB_Only:SolderJumper_3_Open
- removed R? (x4): 1k, symbol Device:R
- added C48, C49, C50, C51: 4.7u, symbol Device:C_Small
- added C?: 10u, symbol Device:C_Small
- added D10, D11, D12, D9: DNP, symbol Device:D_Zener
- added D13, D14, D15, D16: 3.6v, symbol Device:D_Zener
- added J43, J44, J45, J46: Conn_01x01, symbol #Connector:Conn_01x01
- added J47, J48, J49: Conn_01x04, symbol Connector_Generic:Conn_01x04
- added JP13: SolderJumper_2_Open, symbol #PCB_Only:SolderJumper_2_Open
- added JP14: SolderJumper_3_Open, symbol #PCB_Only:SolderJumper_3_Open
- added JP19: SolderJumper_4_Open, symbol #PCB_Only:SolderJumper_4_Open
- added R28, R29, R30, R31: DNP, symbol Device:R
- added R33, R34, R35, R36: 0R, symbol Device:R
- added R38, R39, R41, R43: 47k, symbol Device:R
- added R45, R46, R47, R48: 4.7k, symbol Device:R
- C38, C44: renamed from C?; value 10n -> 22n
- gave numbers to parts that had none: 51
Connections:
- net +12V: now also JP19.3 (O2)
- net +3V3: now also JP14.3 (B), R28.1, R29.1, R30.1, R31.1, R38.1, R39.1, R41.1, R43.1
- net +5V: now also JP13.2 (B), JP14.1 (A), JP19.2 (O1)
- net ENDSTOP1: now also D16.1 (K), R43.2, R45.1
- net ENDSTOP2: now also D15.1 (K), R41.2, R46.1
- net ENDSTOP3: now also D14.1 (K), R39.2, R47.1
- net ENDSTOP4: now also D13.1 (K), R38.2, R48.1
- net GND: now also J54.2 (Pin_2), J55.2 (Pin_2), J56.2 (Pin_2), J57.2 (Pin_2), C48.2, C49.2, C50.2, C51.2, C?.2, D10.2 (A), D11.2 (A), D12.2 (A), D13.2 (A), D14.2 (A), D15.2 (A), D16.2 (A), D9.2 (A), J47.4 (Pin_4), J48.4 (Pin_4), J49.4 (Pin_4); no longer J54.3 (Pin_3), J55.3 (Pin_3), J56.3 (Pin_3), J57.3 (Pin_3)
- net ISP_BOOT: now also J49.3 (Pin_3)
- net RXD: now also J49.2 (Pin_2)
- net SCL: now also J47.3 (Pin_3), J48.3 (Pin_3)
- net SDA: now also J47.2 (Pin_2), J48.2 (Pin_2)
- net TXD: now also J49.1 (Pin_1)
- net VBUS: now also C?.1, JP13.1 (A)
- net at J54.1 (Pin_1), J55.1 (Pin_1), J56.1 (Pin_1)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: now also C48.1, C49.1, C50.1, C51.1, JP19.1 (IN)
- net at R32.1, R37.1: now also J47.1 (Pin_1), J48.1 (Pin_1), JP14.2 (C)
- new net: J54.3 (Pin_3), R45.2
- new net: J55.3 (Pin_3), R46.2
- new net: J56.3 (Pin_3), R47.2
- new net: J57.3 (Pin_3), R48.2
- new net: J43.1 (Pin_1), R33.2
- new net: J44.1 (Pin_1), R34.2
- new net: J45.1 (Pin_1), R35.2
- new net: J46.1 (Pin_1), R36.2
- new net +24V: JP19.4 (O4)
- new net GENERICIO1: D12.1 (K), R31.2, R33.1
- new net GENERICIO2: D11.1 (K), R30.2, R34.1
- new net GENERICIO3: D10.1 (K), R29.2, R35.1
- new net GENERICIO4: D9.1 (K), R28.2, R36.1
- no-connect marks 13 -> 12
Other:
- note added: "place on edge"
- moved on the sheet: C37, C38, C39, C40, C41, C42, C43, C44, C45, C46, C47, C52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
