File: hardware/kajikia/controller.sch (KiCad schematic (older format))
At the start: 15 parts

Commit message: io assignments
Parts:
- C1, C2, C3, C4, C5, C6, C7, C8: renamed from C?; footprint (none) -> _Generic:0603_Small
- JP1: renamed from JP?; footprint (none) -> Jumper:SolderJumper-3_P1.3mm_Open_RoundedPad1.0x1.5mm_NumberLabels
- JP2: renamed from JP?; footprint (none) -> Connector_PinHeader_2.54mm:PinHeader_1x03_P2.54mm_Vertical
- R1: renamed from R?; footprint (none) -> _Generic:0603_Small
- SW1: renamed from SW?; footprint (none) -> Buzzer_Beeper:PUIAudio_SMT_0825_S_4_R
- Y1: renamed from Y?; footprint (none) -> Crystal:Crystal_SMD_3225-4Pin_3.2x2.5mm
- Y2: renamed from Y?; footprint (none) -> Crystal:Crystal_SMD_3215-2Pin_3.2x1.5mm
- gave numbers to parts that had none: 1
Connections:
- net labels added: I2C1_SCL, I2C1_SDA, I2C2_SCL, I2C2_SDA, JTCK-SWCLK, JTDI, JTDO, JTMS-SWDIO, NJTRST, OTG_FS_DM, OTG_FS_DP, OTG_HS_DM, OTG_HS_DP, QUADSPI_BK1_IO0, QUADSPI_BK1_IO1, QUADSPI_BK1_IO2, QUADSPI_BK1_IO3, QUADSPI_BK1_NCS, QUADSPI_CLK, SDMMC1_CK, SDMMC1_CMD, SDMMC1_D0, SDMMC1_D1, SDMMC1_D2, SDMMC1_D3, SDMMC2_CK, SDMMC2_CMD, SDMMC2_D0, SDMMC2_D1, SDMMC2_D2, SDMMC2_D3, SPI1_MISO, SPI1_MOSI, SPI1_SCK, USART1_RX, USART1_TX, USART2_RX, USART2_TX, USART6_RX, USART6_TX
- wire segments 109 -> 115
Other:
- note added: "tmc"

Commit message: io assignments
Connections:
- net labels added: ADC12_INP18, ADC12_INP19, ADC12_INP3, ADC12_INP7, ADC3_INP0, ADC3_INP1, ANALOG, DRV1_CS, DRV1_DCO, DRV1_DIAG0, DRV1_DIAG1, DRV1_DIR, DRV1_EN, DRV1_STEP, DRV_CLK, DRV_DCEN, DRV_DCIN, DRV_MISO, DRV_MOSI, DRV_SCK, MAX_SCK, MCO1, SPI2_SCK, SPI4_MISO, SPI4_MOSI, SPI4_SCK, STUPID, TIM_ADC, uart4rx_tim_adc
- wire segments 115 -> 142
- no-connect marks 0 -> 17
Other:
- note added: "SPI1 - tmc, max, header (display, sd)\nSPI2 - header, max\nSPI4 - header\nUSART1 - usbserial, header\nUSART2 - header\nI2C1 - header\nSDMMC1 - board\nSDMMC2 - header"
Changed lines of the file:
@@
 Text GLabel 4600 2100 1    50   Input ~ 0
 SDMMC2_D3
-Text GLabel 8300 2100 1    50   Input ~ 0
-SDMMC2_CMD
 Text GLabel 5700 1500 1    50   Input ~ 0
 OTG_HS_DP
@@
 Text GLabel 6600 1950 1    50   Input ~ 0
 USART6_RX
-Text Notes 7750 2000 0    50   ~ 0
+Text Notes 7750 1550 0    50   ~ 0
 tmc
 Text Notes 8450 1950 0    50   ~ 0
@@
 Text GLabel 5100 4800 3    50   Input ~ 0
 SPI1_MISO
-Text GLabel 4700 2100 1    50   Input ~ 0
+Text GLabel 8300 2100 1    50   Input ~ 0
 SPI1_MOSI
+Text GLabel 7900 2100 1    50   Input ~ 0
+SPI2_SCK
+Text GLabel 8100 4800 3    50   Input ~ 0
+SPI4_MISO
+Text GLabel 8200 4800 3    50   Input ~ 0
+SPI4_MOSI
+Text GLabel 8800 4800 3    50   Input ~ 0
+SPI4_SCK
+Text Notes 9650 1300 0    50   ~ 0
+SPI1 - tmc, max, header (display, sd)\nSPI2 - header, max\nSPI4 - header\nUSART1 - usbserial, header\nUSART2 - header\nI2C1 - header\nSDMMC1 - board\nSDMMC2 - header
+Text GLabel 3300 1400 1    50   Input ~ 0
+DRV_CLK
+Text GLabel 1550 1050 0    50   Output ~ 0
+DRV1_EN
+Text GLabel 1550 1150 0    50   Output ~ 0
+DRV1_DIR
+Text GLabel 1550 1250 0    50   Output ~ 0
+DRV1_STEP
+Text GLabel 1550 1400 0    50   Output ~ 0
+DRV1_CS
+Text GLabel 5300 5700 3    50   Output ~ 0
+DRV_SCK
+Text GLabel 5100 5700 3    50   Input ~ 0
+DRV_MISO
+Text GLabel 8300 1400 1    50   Output ~ 0
+DRV_MOSI
+Text GLabel 1550 1850 0    50   Input ~ 0
+DRV1_DIAG0
+Text GLabel 1550 1950 0    50   Input ~ 0
+DRV1_DIAG1
+Wire Wire Line
+	1550 1950 1650 1950
+Wire Wire Line
+	1650 1850 1550 1850
+Wire Wire Line
+	1550 1700 1650 1700
+Wire Wire Line
+	1650 1600 1550 1600
+Wire Wire Line
+	1550 1500 1650 1500
+Wire Wire Line
+	1650 1400 1550 1400
+Wire Wire Line
+	1550 1250 1650 1250
+Wire Wire Line
+	1650 1150 1550 1150
+Wire Wire Line
+	1550 1050 1650 1050
+Wire Wire Line
+	1650 900  1550 900
+Text GLabel 1550 2100 0    50   Output ~ 0
+DRV_DCEN
+Wire Wire Line
+	1550 2100 1650 2100
+Text GLabel 1550 2200 0    50   Input ~ 0
+DRV1_DCO
+Text GLabel 1550 2300 0    50   Output ~ 0
+DRV_DCIN
+Wire Wire Line
+	1550 2200 1650 2200
+Wire Wire Line
+	1550 2300 1650 2300
+Text GLabel 3300 2100 1    50   Input ~ 0
+MCO1
+Text GLabel 6100 2100 1    50   Input ~ 0
+ADC3_INP0
+Text GLabel 6200 2100 1    50   Input ~ 0
+ADC3_INP1
+Text GLabel 2900 2100 1    50   Input ~ 0
+ADC12_INP18
+Text GLabel 3000 2100 1    50   Input ~ 0
+ADC12_INP19
+Text GLabel 3100 2100 1    50   Input ~ 0
+ADC12_INP3
+Text GLabel 3200 2100 1    50   Input ~ 0
+ADC12_INP7
+Text GLabel 6100 4850 3    50   Input ~ 0
+STUPID
+Text GLabel 6300 4900 3    50   Input ~ 0
+STUPID
+Text GLabel 6400 4900 3    50   Input ~ 0
+STUPID
+Text GLabel 6500 5100 3    50   Input ~ 0
+TIM_ADC
+Text GLabel 6600 5100 3    50   Input ~ 0
+TIM_ADC
+Text GLabel 6700 5100 3    50   Input ~ 0
+TIM_ADC
+Text GLabel 6800 5100 3    50   Input ~ 0
+TIM_ADC
+Text GLabel 7000 4900 3    50   Input ~ 0
+STUPID
+Text GLabel 7100 4900 3    50   Input ~ 0
+STUPID
+Text GLabel 7200 4900 3    50   Input ~ 0
+STUPID
+Text GLabel 7300 4900 3    50   Input ~ 0
+STUPID
+Text GLabel 7400 4900 3    50   Input ~ 0
+STUPID
+Text GLabel 7600 4900 3    50   Input ~ 0
+STUPID
+Text GLabel 7700 4900 3    50   Input ~ 0
+STUPID
+Text GLabel 7900 4900 3    50   Input ~ 0
+STUPID
+Text GLabel 8000 4900 3    50   Input ~ 0
+STUPID
+Text GLabel 8900 4900 3    50   Input ~ 0
+STUPID
+Text GLabel 9000 4900 3    50   Input ~ 0
+STUPID
+Text GLabel 9100 4900 3    50   Input ~ 0
+STUPID
+Text GLabel 4200 4850 3    50   Input ~ 0
+STUPID
+Text GLabel 4300 4850 3    50   Input ~ 0
+STUPID
+Text GLabel 4400 4850 3    50   Input ~ 0
+STUPID
+Text GLabel 4500 4850 3    50   Input ~ 0
+STUPID
+Text GLabel 4600 4850 3    50   Input ~ 0
+STUPID
+Text GLabel 4700 4850 3    50   Input ~ 0
+STUPID
+Text GLabel 4900 4850 3    50   Input ~ 0
+STUPID
+Text GLabel 5000 4850 3    50   Input ~ 0
+STUPID
+Text GLabel 5400 4850 3    50   Input ~ 0
+STUPID
+Text GLabel 5500 4850 3    50   Input ~ 0
+STUPID
+Text GLabel 5600 4850 3    50   Input ~ 0
+STUPID
+Text GLabel 5700 4850 3    50   Input ~ 0
+STUPID
+Text GLabel 5200 4850 3    50   Input ~ 0
+STUPID
+Wire Wire Line
+	3400 2200 3400 2100
+Wire Wire Line
+	3500 2100 3500 2200
+Wire Wire Line
+	3600 2200 3600 2100
+Wire Wire Line
+	3700 2100 3700 2200
+Wire Wire Line
+	3800 2200 3800 2100
+Wire Wire Line
+	3900 2100 3900 2200
+Wire Wire Line
+	3300 2200 3300 2100
+Wire Wire Line
+	6100 2200 6100 2100
+Wire Wire Line
+	6200 2100 6200 2200
+Text GLabel 2500 2100 1    50   Input ~ 0
+SDMMC2_CMD
+Text GLabel 2600 2100 1    50   Input ~ 0
+uart4rx_tim_adc
+NoConn ~ 2600 1400
+NoConn ~ 2500 1400
+NoConn ~ 2700 1400
+NoConn ~ 2800 1400
+NoConn ~ 2900 1400
+NoConn ~ 3000 1400
+NoConn ~ 3100 1400
+NoConn ~ 3200 1400
+Text GLabel 4200 2100 1    50   Input ~ 0
+ANALOG
+Text GLabel 4300 2100 1    50   Input ~ 0
+ANALOG
+Text GLabel 4400 2100 1    50   Input ~ 0
+STUPID
+Wire Wire Line
+	4300 2100 4300 2200
+Wire Wire Line
+	4200 2200 4200 2100
+NoConn ~ 4200 1400
+NoConn ~ 4300 1400
+NoConn ~ 4500 1200
+NoConn ~ 4600 1200
+NoConn ~ 4700 1200
+Text GLabel 4900 2100 1    50   Input ~ 0
+I2C1_SDA
+NoConn ~ 4800 1400
+NoConn ~ 4900 1400
+NoConn ~ 5000 1400
+NoConn ~ 5100 1400
+Text GLabel 5400 2100 1    50   Input ~ 0
+STUPID
+Text GLabel 5500 2100 1    50   Input ~ 0
+STUPID
+Text GLabel 5900 2100 1    50   Input ~ 0
+STUPID
+Text GLabel 6000 2100 1    50   Input ~ 0
+STUPID
+Text GLabel 6300 2100 1    50   Input ~ 0
+STUPID
+Text GLabel 6400 2100 1    50   Input ~ 0
+STUPID
+Text GLabel 7600 2100 1    50   Input ~ 0
+STUPID
+Text GLabel 7700 2100 1    50   Input ~ 0
+STUPID
+Text GLabel 7800 2100 1    50   Input ~ 0
+STUPID
+Text GLabel 7900 1400 1    50   Input ~ 0
+MAX_SCK
+Text GLabel 8000 2100 1    50   Input ~ 0
+STUPID
+Text GLabel 8100 2100 1    50   Input ~ 0
+STUPID
+Text GLabel 8300 950  1    50   Input ~ 0
+SDMMC2_CMD
+Text GLabel 4700 1100 1    50   Input ~ 0
+SPI1_MOSI
+Wire Wire Line
+	5100 4800 5100 4700
+Wire Wire Line
+	5300 4700 5300 4800
+Wire Wire Line
+	4700 1100 4700 2200
 $EndSCHEMATC

Commit message: lpc, ios
Parts:
- removed C1: 1F, _Generic:0603_Small, symbol Device:CP1
- removed C2: 100n, _Generic:0603_Small, symbol Device:C
- removed C3, C4, C7, C8: C, _Generic:0603_Small, symbol Device:C
- removed JP1: SolderJumper_3_Open, Jumper:SolderJumper-3_P1.3mm_Open_RoundedPad1.0x1.5mm_NumberLabels, symbol Jumper:SolderJumper_3_Open
- removed JP2: Jumper_NC_Dual, Connector_PinHeader_2.54mm:PinHeader_1x03_P2.54mm_Vertical, symbol Device:Jumper_NC_Dual
- removed R1: 10k, _Generic:0603_Small, symbol Device:R
- removed SW1: SW_Push_Dual, Buzzer_Beeper:PUIAudio_SMT_0825_S_4_R, symbol Switch:SW_Push_Dual
- removed U1: STM32H753ZITx, Package_QFP:LQFP-144_20x20mm_P0.5mm, symbol MCU_ST_STM32H7:STM32H753ZITx
- removed Y2: 32.768KHz, Crystal:Crystal_SMD_3215-2Pin_3.2x1.5mm, symbol Device:Crystal
- added D? (x5): D_Schottky_Small, symbol Device:D_Schottky_Small
- added J1: USB_C_Receptacle, symbol Connector:USB_C_Receptacle
- added J2: Micro_SD_Card_Det, symbol Connector:Micro_SD_Card_Det
- added J? (x5): Conn_01x03, symbol Connector_Generic:Conn_01x03
- added J? (x2): Screw_Terminal_01x04, symbol Connector:Screw_Terminal_01x04
- added JP? (x5): SolderJumper_2_Open, symbol #PCB_Only:SolderJumper_2_Open
- added JP?: SolderJumper_3_Open, symbol #PCB_Only:SolderJumper_3_Open
- added Q? (x4): AON6144, symbol Device:Q_NMOS_SGD
- added R? (x5): 1k, symbol Device:R
- added R? (x4): 10, symbol Device:R
- added U1: LPC1769FBD100, Package_QFP:LQFP-100_14x14mm_P0.5mm, symbol MCU_NXP_LPC:LPC1769FBD100
- added U? (x2): IR4427S, symbol Driver_FET:MIC4427
- Y1: value 16MHz -> 12MHz
Connections:
- net labels added: +12V, +3.3V, +5V, A0, A1, A2, A3, A4, A5, CS, DIAG0_COMBINED, DRV2_CS, DRV2_DIAG1, DRV2_DIR, DRV2_EN, DRV2_STEP, DRV3_DIAG1, DRV3_DIR, DRV3_EN, DRV3_STEP, DRV4_DIAG1, DRV4_DIR, DRV4_EN, DRV4_STEP, DRV5_DIAG1, DRV5_DIR, DRV5_EN, DRV5_STEP, ISP_BOOT, JTAG_RTCK, JTAG_TCK, JTAG_TDI, JTAG_TDO, JTAG_TMS, JTAG_TRST, MAX6675, MISO, MOSI, P1.18, P1.18_POW, P1.19, P1.19_POW, P2.3, P2.3_ADV, P2.4, P2.4_ADV, P3.25, P3.25_POW, P3.26, P3.26_POW, RST, RXD0, RXD3, SCK, SCL0, SDA0, SD_CS, SD_MISO, SD_MOSI, SD_SCK, TH1, TH2, TH3, TH4, TXD0, TXD3, Thermo, USB_CONNECT, USB_D+, USB_D-, clkout, i2s_LED?, mc0b, mc1a, mc2a, mc2b, pwm6
- net labels removed: 3.3V, 3.3v, ADC12_INP18, ADC12_INP19, ADC12_INP3, ADC12_INP7, ADC3_INP0, ADC3_INP1, ANALOG, DRV1_DCO, DRV1_DIAG0, DRV_CLK, I2C1_SCL, I2C1_SDA, I2C2_SCL, I2C2_SDA, JTCK-SWCLK, JTDI, JTDO, JTMS-SWDIO, MAX_SCK, MCO1, NJTRST, OTG_FS_DM, OTG_FS_DP, OTG_HS_DM, OTG_HS_DP, QUADSPI_BK1_IO0, QUADSPI_BK1_IO1, QUADSPI_BK1_IO2, QUADSPI_BK1_IO3, QUADSPI_BK1_NCS, QUADSPI_CLK, SDMMC1_CK, SDMMC1_CMD, SDMMC1_D0, SDMMC1_D1, SDMMC1_D2, SDMMC1_D3, SDMMC2_CK, SDMMC2_CMD, SDMMC2_D0, SDMMC2_D1, SDMMC2_D2, SDMMC2_D3, SPI1_MISO, SPI1_MOSI, SPI1_SCK, SPI2_SCK, SPI4_MISO, SPI4_MOSI, SPI4_SCK, STUPID, TIM_ADC, USART1_RX, USART1_TX, USART2_RX, USART2_TX, USART6_RX, USART6_TX, VDD, uart4rx_tim_adc
- wire segments 142 -> 192
- no-connect marks 17 -> 5
Other:
- note added: "?"
- note added: "? leave dcstep"
- note removed: "SPI1 - tmc, max, header (display, sd)\nSPI2 - header, max\nSPI4 - header\nUSART1 - usbserial, header\nUSART2 - header\nI2C1 - header\nSDMMC1 - board\nSDMMC2 - header"
- note removed: "tmc"
- moved on the sheet: Y1

Commit message: max6675, cleanup
Parts:
- removed C5, C6: C, _Generic:0603_Small, symbol Device:C
- removed D? (x5): D_Schottky_Small, symbol Device:D_Schottky_Small
- removed J1: USB_C_Receptacle, symbol Connector:USB_C_Receptacle
- removed J2: Micro_SD_Card_Det, symbol Connector:Micro_SD_Card_Det
- removed J? (x5): Conn_01x03, symbol Connector_Generic:Conn_01x03
- removed J? (x2): Screw_Terminal_01x04, symbol Connector:Screw_Terminal_01x04
- removed JP?: SolderJumper_3_Open, symbol #PCB_Only:SolderJumper_3_Open
- removed Q? (x4): AON6144, symbol Device:Q_NMOS_SGD
- removed R? (x5): 1k, symbol Device:R
- removed R? (x4): 10, symbol Device:R
- removed U? (x2): IR4427S, symbol Driver_FET:MIC4427
- removed Y1: 12MHz, Crystal:Crystal_SMD_3225-4Pin_3.2x2.5mm, symbol Device:Crystal_GND24
- added C? (x10): 100n, symbol Device:C_Small
- added C? (x5): 10u, symbol Device:C_Small
- added C? (x2): 12p, symbol Device:C_Small
- added J? (x7): Conn_01x01, symbol #Connector:Conn_01x01
- added JP? (x7): SolderJumper_2_Open, symbol #PCB_Only:SolderJumper_2_Open
- added R? (x2): 1, symbol Device:R
- added R? (x3): 1k, symbol Device:R
- added R? (x2): 10k, symbol Device:R
- added SW? (x2): 3x6mm, symbol Switch:SW_Push
- added Y?: 12MHz, symbol Device:Crystal_GND24
Connections:
- net labels added: DRV3_CS, DRV4_CS, DRV5_CS, DRV_DIAG0, MAX1_CS, MAX2_CS, P0.0_IN, P0.16, P0.19_IN, P0.1_IN, P0.2, P0.20_IN, P0.21, P0.22_ADV, P0.23_A0, P0.24_A1, P0.25_A2, P0.26_A3, P0.3, P1.16, P1.17, P1.22_ADV, P1.25_ADV, P1.26_ADV, P1.27, P1.28_ADV, P1.29_ADV, P1.30_A4, P1.31_A5, P2.10, P2.11, P2.12, P2.13, P2.6, P2.7, P2.8, RXD, SCL, SDA, SD_DETECT, TXD, USB_CON, VDDA, VREFN, VREFP, VSSA
- net labels removed: +12V, +5V, A0, A1, A2, A3, A4, A5, DIAG0_COMBINED, DRV_DCEN, DRV_DCIN, MAX6675, P1.18, P1.19, P2.3, P2.4, P3.25, P3.26, SCL0, SDA0, TH1, TH2, TH3, TH4, Thermo, clkout, i2s_LED?, mc0b, mc1a, mc2a, mc2b, pwm6
- wire segments 192 -> 273
- no-connect marks 5 -> 3
Other:
- note removed: "?"
- note removed: "? leave dcstep"
- moved on the sheet: JP?, U1

Commit message: power
Parts:
- removed JP? (x12): SolderJumper_2_Open, symbol #PCB_Only:SolderJumper_2_Open
- added J1, J10, J11, J12, J13, J14, J15, J16, J17, J2, J25, J26, J27, J28, J29, J3, J30, J31, J32, J33, J34, J35, J36, J37, J38, J4, J5, J6, J7, J8, J9: Conn_01x01, symbol #Connector:Conn_01x01
- added JP1, JP10, JP11, JP12, JP2, JP3, JP4, JP5, JP6, JP7, JP8, JP9, JP?: SolderJumper_2_Open, symbol #PCB_Only:SolderJumper_2_Open
- gave numbers to parts that had none: 34
Connections:
- net P0.16 is gone; now on net DRV5_CS: U1.63 (P0[16])
- net P0.21 is gone; now on net DRV_DIAG0: U1.57 (P0[21])
- net P1.16 is gone; now on net DRV5_EN: U1.87 (P1[16])
- net P1.17 is gone; now on net DRV5_DIR: U1.86 (P1[17])
- net P1.27 is gone; now on net MAX1_CS: U1.43 (P1[27])
- net P2.11 is gone; now on net DRV3_DIAG1: U1.52 (P2[11])
- net P2.12 is gone; now on net DRV4_DIAG1: U1.51 (P2[12])
- net P2.13 is gone; now on net DRV5_DIAG1: U1.50 (P2[13])
- net P2.6 is gone; now on net DRV5_STEP: U1.67 (P2[6])
- net P2.7 is gone; now on net DRV1_DIAG1: U1.66 (P2[7])
- net P2.8 is gone; now on net DRV2_DIAG1: U1.65 (P2[8])
- net DRV1_DIAG1: now also J33.1 (Pin_1), JP4.1 (A)
- net DRV2_DIAG1: now also J34.1 (Pin_1), JP5.1 (A)
- net DRV3_DIAG1: now also J36.1 (Pin_1), JP6.1 (A)
- net DRV4_DIAG1: now also J37.1 (Pin_1), JP7.1 (A)
- net DRV5_CS: now also J10.1 (Pin_1), JP11.1 (A)
- net DRV5_DIAG1: now also J38.1 (Pin_1), JP12.1 (A)
- net DRV5_DIR: now also J26.1 (Pin_1), JP9.1 (A)
- net DRV5_EN: now also J25.1 (Pin_1), JP8.1 (A)
- net DRV5_STEP: now also J32.1 (Pin_1), JP10.1 (A)
- net DRV_DIAG0: now also J15.1 (Pin_1), JP3.1 (A)
- net DRV_MISO: now also J11.1 (Pin_1)
- net DRV_MOSI: now also J12.1 (Pin_1)
- net DRV_SCK: now also J9.1 (Pin_1)
- net ISP_BOOT: now also J35.1 (Pin_1), JP2.2 (B)
- net MAX1_CS: now also J31.1 (Pin_1), JP1.2 (B)
- net P0.2: now also J3.1 (Pin_1)
- net P0.3: now also J4.1 (Pin_1)
- net SCL: now also J17.1 (Pin_1)
- net SDA: now also J16.1 (Pin_1)
- net SD_CS: now also J5.1 (Pin_1)
- net SD_MISO: now also J7.1 (Pin_1)
- net SD_MOSI: now also J8.1 (Pin_1)
- net SD_SCK: now also J6.1 (Pin_1)
- net P1.20: now reaches U1.34 (P1[20])
- net P1.20: now also J27.1 (Pin_1)
- net P1.21: now reaches U1.35 (P1[21])
- net P1.21: now also J28.1 (Pin_1)
- net P1.23: now reaches U1.37 (P1[23])
- net P1.23: now also J29.1 (Pin_1)
- net P1.24: now reaches U1.38 (P1[24])
- net P1.24: now also J30.1 (Pin_1)
- net P4.28_GEN: now reaches U1.82 (P4[28])
- net P4.28_GEN: now also JP?.2 (B)
- net P4.29_GEN: now reaches U1.85 (P4[29])
- net P0.0_IN renamed P0.0_END
- net P0.0_END: now also J1.1 (Pin_1)
- net P0.19_IN renamed P0.19_END
- net P0.19_END: now also J13.1 (Pin_1)
- net P0.1_IN renamed P0.1_END
- net P0.1_END: now also J2.1 (Pin_1)
- net P0.20_IN renamed P0.20_END
- net P0.20_END: now also J14.1 (Pin_1)
- net P0.23_A0 renamed P0.23_TH0
- net P0.24_A1 renamed P0.24_TH1
- net P0.25_A2 renamed P0.25_TH2
- net P0.26_A3 renamed P0.26_TH3
- net P1.30_A4 renamed P1.30_GEN
- net P1.31_A5 renamed P1.31_GEN
- new net Sheet5C3B9891/MAX1_CS: JP1.1 (A)
- new net Sheet5C3B9891/MAX2_CS: JP2.1 (A)
- new net Sheet5C3B9891/SD_DETECT: JP?.1 (A)
- new net sheet60C2EDF9/DRV1_DIAG1: JP4.2 (B)
- new net sheet60C2EDF9/DRV2_DIAG1: JP5.2 (B)
- new net sheet60C2EDF9/DRV3_DIAG1: JP6.2 (B)
- new net sheet60C2EDF9/DRV4_DIAG1: JP7.2 (B)
- new net sheet60C2EDF9/DRV5_CS: JP11.2 (B)
- new net sheet60C2EDF9/DRV5_DIAG1: JP12.2 (B)
- new net sheet60C2EDF9/DRV5_DIR: JP9.2 (B)
- new net sheet60C2EDF9/DRV5_EN: JP8.2 (B)
- new net sheet60C2EDF9/DRV5_STEP: JP10.2 (B)
- new net sheet60C2EDF9/DRV_DIAG0: JP3.2 (B)
Other:
- note added: "CAPS\n12p, 0603, 50v\n470p, 0603, 50v\n22n, 0603, 100v\n100n, 0603, 50v\n470n, 0603, 25v\n4.7u, 0805, 50v\n10u, 0603, 16v\n390u, 8x12mm, 20v\n68u, 8x10mm, 50v"
- note added: "|\n| SPI\n|\n|\n|"
- moved on the sheet: C10, C2, C27, C28, C29, C3, C30, C31, C32, C33, C34, C35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
