File: hardware/kajikia/kajikia.sch (KiCad schematic (older format))
At the start: 0 parts

Commit message: hc, lc and  protected ios
Other:
- note added: "buzzer\nled"
Changed lines of the file:
@@
 $Descr A4 11693 8268
 encoding utf-8
-Sheet 1 3
+Sheet 1 6
 Title ""
 Date ""
@@
 F1 "mcu.sch" 50
 $EndSheet
+$Sheet
+S 6500 1600 550  200
+U 5AFECA39
+F0 "hc1" 50
+F1 "hc.sch" 50
+F2 "IN" I L 6500 1700 50
+F3 "OUT" I R 7050 1700 50
+$EndSheet
+$Sheet
+S 6500 2100 550  200
+U 5AFF08F7
+F0 "lc1" 50
+F1 "lc.sch" 50
+F2 "IN" I L 6500 2200 50
+F3 "OUT" I R 7050 2200 50
+$EndSheet
+Text Notes 10750 750  0    50   ~ 0
+buzzer\nled
+$Sheet
+S 6500 2550 550  200
+U 5AFF10F9
+F0 "hvio1" 50
+F1 "hvio.sch" 50
+F2 "IN" I L 6500 2650 50
+F3 "OUT" I R 7050 2650 50
+$EndSheet
 $EndSCHEMATC

Commit message: reorder started
Changed lines of the file:
@@
 $Descr A4 11693 8268
 encoding utf-8
-Sheet 1 6
+Sheet 1 8
 Title ""
 Date ""
@@
 Comment4 ""
 $EndDescr
-$Sheet
-S 1950 4300 850  2050
-U 5AF71FC6
-F0 "driver_1" 50
-F1 "driver.sch" 50
-F2 "GND" I L 1950 4700 50
-F3 "CLK" I L 1950 4850 50
-F4 "CS" I L 1950 5350 50
-F5 "SCK" I L 1950 5450 50
-F6 "MISO" O L 1950 5550 50
-F7 "MOSI" I L 1950 5650 50
-F8 "STEP" I L 1950 5200 50
-F9 "DIR" I L 1950 5100 50
-F10 "EN" I L 1950 5000 50
-F11 "DIAG0" O L 1950 5800 50
-F12 "DIAG1" O L 1950 5900 50
-F13 "5V" I L 1950 4500 50
-F14 "3.3V" I L 1950 4600 50
-F15 "VIN" I L 1950 4400 50
-F16 "DCO" O L 1950 6150 50
-F17 "DCEN" I L 1950 6050 50
-F18 "DCIN" I L 1950 6250 50
-F19 "OA1" O R 2800 4400 50
-F20 "OA2" O R 2800 4500 50
-F21 "OB1" O R 2800 4600 50
-F22 "OB2" O R 2800 4700 50
-$EndSheet
 $Sheet
 S 1950 1250 1750 1750
@@
 F3 "OUT" I R 7050 2650 50
 $EndSheet
+$Sheet
+S 1900 3800 750  1600
+U 5AF71FC6
+F0 "driver_1" 50
+F1 "driver.sch" 50
+F3 "CLK" I L 1900 3900 50
+F4 "CS" I L 1900 4400 50
+F5 "SCK" I L 1900 4500 50
+F6 "MISO" O L 1900 4600 50
+F7 "MOSI" I L 1900 4700 50
+F8 "STEP" I L 1900 4250 50
+F9 "DIR" I L 1900 4150 50
+F10 "EN" I L 1900 4050 50
+F11 "DIAG0" O L 1900 4850 50
+F12 "DIAG1" O L 1900 4950 50
+F16 "DCO" O L 1900 5200 50
+F17 "DCEN" I L 1900 5100 50
+F18 "DCIN" I L 1900 5300 50
+F19 "OA1" O R 2650 3900 50
+F20 "OA2" O R 2650 4000 50
+F21 "OB1" O R 2650 4100 50
+F22 "OB2" O R 2650 4200 50
+$EndSheet
 $EndSCHEMATC

Commit message: reorder
Changed lines of the file:
@@
 $EndDescr
 $Sheet
-S 1950 1250 1750 1750
+S 3050 1600 1000 1000
 U 5AF7E834
-F0 "mcu" 50
-F1 "mcu.sch" 50
-$EndSheet
-$Sheet
-S 6500 1600 550  200
-U 5AFECA39
-F0 "hc1" 50
-F1 "hc.sch" 50
-F2 "IN" I L 6500 1700 50
-F3 "OUT" I R 7050 1700 50
-$EndSheet
-$Sheet
-S 6500 2100 550  200
-U 5AFF08F7
-F0 "lc1" 50
-F1 "lc.sch" 50
-F2 "IN" I L 6500 2200 50
-F3 "OUT" I R 7050 2200 50
+F0 "controller" 50
+F1 "controller.sch" 50
 $EndSheet
 Text Notes 10750 750  0    50   ~ 0
 buzzer\nled
 $Sheet
-S 6500 2550 550  200
-U 5AFF10F9
-F0 "hvio1" 50
-F1 "hvio.sch" 50
-F2 "IN" I L 6500 2650 50
-F3 "OUT" I R 7050 2650 50
+S 1550 1600 1000 1000
+U 5B406A78
+F0 "power" 50
+F1 "power.sch" 50
 $EndSheet
 $Sheet
-S 1900 3800 750  1600
-U 5AF71FC6
-F0 "driver_1" 50
+S 6050 1600 1000 1000
+U 5B406A7B
+F0 "io" 50
+F1 "io.sch" 50
+$EndSheet
+$Sheet
+S 4550 1600 1000 1000
+U 5B406A82
+F0 "driver" 50
 F1 "driver.sch" 50
-F3 "CLK" I L 1900 3900 50
-F4 "CS" I L 1900 4400 50
-F5 "SCK" I L 1900 4500 50
-F6 "MISO" O L 1900 4600 50
-F7 "MOSI" I L 1900 4700 50
-F8 "STEP" I L 1900 4250 50
-F9 "DIR" I L 1900 4150 50
-F10 "EN" I L 1900 4050 50
-F11 "DIAG0" O L 1900 4850 50
-F12 "DIAG1" O L 1900 4950 50
-F16 "DCO" O L 1900 5200 50
-F17 "DCEN" I L 1900 5100 50
-F18 "DCIN" I L 1900 5300 50
-F19 "OA1" O R 2650 3900 50
-F20 "OA2" O R 2650 4000 50
-F21 "OB1" O R 2650 4100 50
-F22 "OB2" O R 2650 4200 50
 $EndSheet
 $EndSCHEMATC

Commit message: power
Changed lines of the file:
@@
 buzzer\nled
-$Sheet
-S 1550 1600 1000 1000
-U 5B406A78
-F0 "power" 50
-F1 "power.sch" 50
-$EndSheet
 $Sheet
 S 6050 1600 1000 1000
