File: hardware/kajikia/kajikia.sch (KiCad schematic (older format))
At the start: 0 parts

Commit message: fancy
Parts:
- added C1, C10, C11, C12, C13, C14, C15, C16, C8, C9: 100n, _Generic:0603_CAP, symbol Device:C_Small
- added C17, C2, C3, C5, C7: 10u, _Generic:0603_CAP, symbol Device:C_Small
- added C4, C6: 12p, _Generic:0603_CAP, symbol Device:C_Small
- added J1, J10, J11, J12, J13, J14, J15, J16, J17, J18, J19, J2, J20, J21, J22, J23, J24, J25, J26, J27, J28, J29, J3, J30, J31, J32, J33, J34, J35, J36, J37, J38, J4, J5, J6, J7, J8, J9: Conn_01x01, symbol #Connector:Conn_01x01
- added JP1, JP10, JP11, JP12, JP13, JP2, JP3, JP4, JP5, JP6, JP7, JP8, JP9: SolderJumper_2_Open, symbol #PCB_Only:SolderJumper_2_Open
- added R1, R3: 10k, _Generic:0603_RES, symbol Device:R
- added R2, R4, R5: 1k, _Generic:0603_RES, symbol Device:R
- added R6, R7: 2.2R, _Generic:0603_RES, symbol Device:R
- added SW1, SW2: 3x6mm, symbol Switch:SW_Push
- added U1: LPC1769FBD100, Package_QFP:LQFP-100_14x14mm_P0.5mm, symbol MCU_NXP_LPC:LPC1769FBD100
- added Y1: 12MHz, symbol Device:Crystal_GND24
Connections:
- new net: U1.22 (XTAL1), Y1.1
- new net: U1.23 (XTAL2), Y1.3
- new net: C6.1, Y1.2
- new net: C4.1, Y1.4
- new net: R2.2, SW1.1
- new net +3V3: C10.1, C11.1, C12.1, C13.1, C14.1, C2.1, C3.1, C5.1, C7.1, C8.1, C9.1, R1.1, R3.1, R6.1, U1.19 (VBAT), U1.28 (VDD(3V3)), U1.42 (VDD(REG)(3V3)), U1.54 (VDD(3V3)), U1.71 (VDD(3V3)), U1.84 (VDD(REG)(3V3)), U1.96 (VDD(3V3))
- new net DRV1_CS: U1.81 (P0[4])
- new net DRV1_DIAG1: J33.1 (Pin_1), JP5.1 (A), U1.66 (P2[7])
- new net DRV1_DIR: U1.94 (P1[1])
- new net DRV1_EN: U1.95 (P1[0])
- new net DRV1_STEP: U1.75 (P2[0])
- new net DRV2_CS: U1.80 (P0[5])
- new net DRV2_DIAG1: J34.1 (Pin_1), JP6.1 (A), U1.65 (P2[8])
- new net DRV2_DIR: U1.92 (P1[8])
- new net DRV2_EN: U1.93 (P1[4])
- new net DRV2_STEP: U1.74 (P2[1])
- new net DRV3_CS: U1.48 (P0[10])
- new net DRV3_DIAG1: J36.1 (Pin_1), JP7.1 (A), U1.52 (P2[11])
- new net DRV3_DIR: U1.90 (P1[10])
- new net DRV3_EN: U1.91 (P1[9])
- new net DRV3_STEP: U1.73 (P2[2])
- new net DRV4_CS: U1.49 (P0[11])
- new net DRV4_DIAG1: J37.1 (Pin_1), JP8.1 (A), U1.51 (P2[12])
- new net DRV4_DIR: U1.88 (P1[15])
- new net DRV4_EN: U1.89 (P1[14])
- new net DRV4_STEP: U1.68 (P2[5])
- new net DRV5_CS: J10.1 (Pin_1), JP12.1 (A), U1.63 (P0[16])
- new net DRV5_DIAG1: J38.1 (Pin_1), JP13.1 (A), U1.50 (P2[13])
- new net DRV5_DIR: J26.1 (Pin_1), JP10.1 (A), U1.86 (P1[17])
- new net DRV5_EN: J25.1 (Pin_1), JP9.1 (A), U1.87 (P1[16])
- new net DRV5_STEP: J32.1 (Pin_1), JP11.1 (A), U1.67 (P2[6])
- new net DRV_DIAG0: J15.1 (Pin_1), JP4.1 (A), U1.57 (P0[21])
- new net DRV_MISO: J11.1 (Pin_1), U1.61 (P0[17])
- new net DRV_MOSI: J12.1 (Pin_1), U1.60 (P0[18])
- new net DRV_SCK: J9.1 (Pin_1), U1.62 (P0[15])
- new net GND: C1.2, C10.2, C11.2, C12.2, C13.2, C14.2, C2.2, C3.2, C4.2, C5.2, C6.2, C7.2, C8.2, C9.2, R7.2, SW1.2, SW2.2, U1.31 (VSS), U1.41 (VSS), U1.55 (VSS), U1.72 (VSS), U1.83 (VSS), U1.97 (VSS)
- new net ISP_BOOT: J35.1 (Pin_1), JP3.2 (B), R1.2, R2.1, U1.53 (P2[10])
- new net Interfaces/MAX1_CS: JP2.1 (A)
- new net Interfaces/MAX2_CS: JP3.1 (A)
- new net Interfaces/SD_DETECT: JP1.1 (A)
- new net JTAG_RTCK: J18.1 (Pin_1), U1.100 (RTCK)
- new net JTAG_TCK: J23.1 (Pin_1), U1.5 (TCK/SWDCLK)
- new net JTAG_TDI: J20.1 (Pin_1), U1.2 (TDI)
- new net JTAG_TDO: J19.1 (Pin_1), U1.1 (TDO/SWO)
- new net JTAG_TMS: J21.1 (Pin_1), U1.3 (TMS/SWDIO)
- new net JTAG_TRST: J22.1 (Pin_1), U1.4 (~TRST~)
- new net MAX1_CS: J31.1 (Pin_1), JP2.2 (B), U1.43 (P1[27])
- new net P0.0_END: J1.1 (Pin_1), U1.46 (P0[0])
- new net P0.19_END: J13.1 (Pin_1), U1.59 (P0[19])
- new net P0.1_END: J2.1 (Pin_1), U1.47 (P0[1])
- new net P0.2: J3.1 (Pin_1), U1.98 (P0[2])
- new net P0.20_END: J14.1 (Pin_1), U1.58 (P0[20])
- new net P0.22_ADV: U1.56 (P0[22])
- new net P0.23_TH0: U1.9 (P0[23])
- new net P0.24_TH1: U1.8 (P0[24])
- new net P0.25_TH2: U1.7 (P0[25])
- new net P0.26_TH3: U1.6 (P0[26])
- new net P0.3: J4.1 (Pin_1), U1.99 (P0[3])
- new net P1.18_POW: U1.32 (P1[18])
- new net P1.19_POW: U1.33 (P1[19])
- new net P1.20: J27.1 (Pin_1), U1.34 (P1[20])
- new net P1.21: J28.1 (Pin_1), U1.35 (P1[21])
- new net P1.22_ADV: U1.36 (P1[22])
- new net P1.23: J29.1 (Pin_1), U1.37 (P1[23])
- new net P1.24: J30.1 (Pin_1), U1.38 (P1[24])
- new net P1.25_ADV: U1.39 (P1[25])
- new net P1.26_ADV: U1.40 (P1[26])
- new net P1.28_ADV: U1.44 (P1[28])
- new net P1.29_ADV: U1.45 (P1[29])
- new net P1.30_GEN: U1.21 (P1[30])
- new net P1.31_GEN: U1.20 (P1[31])
- new net P2.3_ADV: U1.70 (P2[3])
- new net P2.4_ADV: U1.69 (P2[4])
- new net P3.25_POW: U1.27 (P3[25])
- new net P3.26_POW: U1.26 (P3[26])
- new net P4.28_GEN: U1.82 (P4[28])
- new net P4.29_GEN: JP1.2 (B), U1.85 (P4[29])
- new net RST: C1.1, J24.1 (Pin_1), R3.2, SW2.1, U1.17 (~RESET~)
- new net SCL: J17.1 (Pin_1), U1.24 (P0[28])
- new net SDA: J16.1 (Pin_1), U1.25 (P0[27])
- new net SD_CS: J5.1 (Pin_1), U1.79 (P0[6])
- new net SD_MISO: J7.1 (Pin_1), U1.77 (P0[8])
- new net SD_MOSI: J8.1 (Pin_1), U1.76 (P0[9])
- new net SD_SCK: J6.1 (Pin_1), U1.78 (P0[7])
- new net Stepper Driver/DRV1_DIAG1: JP5.2 (B)
- new net Stepper Driver/DRV2_DIAG1: JP6.2 (B)
- new net Stepper Driver/DRV3_DIAG1: JP7.2 (B)
- new net Stepper Driver/DRV4_DIAG1: JP8.2 (B)
- new net Stepper Driver/DRV5_CS: JP12.2 (B)
- new net Stepper Driver/DRV5_DIAG1: JP13.2 (B)
- new net Stepper Driver/DRV5_DIR: JP10.2 (B)
- new net Stepper Driver/DRV5_EN: JP9.2 (B)
- new net Stepper Driver/DRV5_STEP: JP11.2 (B)
- new net Stepper Driver/DRV_DIAG0: JP4.2 (B)
- new net USB_CON: U1.64 (P2[9])
- new net USB_D+: U1.29 (P0[29])
- new net USB_D-: U1.30 (P0[30])
- new net VDDA: C16.1, C17.1, R4.1, R6.2, U1.10 (VDDA)
- new net VREFN: C15.1, R5.2, U1.15 (VREFN)
- new net VREFP: C15.2, R4.2, U1.12 (VREFP)
- new net VSSA: C16.2, C17.2, R5.1, R7.1, U1.11 (VSSA)
- no-connect marks 0 -> 3
Other:
- note added: "CAPS\n12p, 0603, 50v\n470p, 0603, 50v\n22n, 0603, 100v\n100n, 0603, 50v\n470n, 0603, 25v\n4.7u, 0805, 50v\n10u, 0603, 16v\n390u, 8x12mm, 20v\n68u, 8x10mm, 50v"
- note added: "Interfaces"
- note added: "Power"
- note added: "Power Outputs"
- note added: "Processor"
- note added: "Stepper Driver"
- note added: "|\n| SPI\n|\n|\n|"
- note removed: "buzzer\nled"
