File: hardware/kajikia/kajikia.sch (KiCad schematic (older format))
At the start: 79 parts, among them J1 Conn_01x01, J10 Conn_01x01, J11 Conn_01x01, J12 Conn_01x01, J13 Conn_01x01, J14 Conn_01x01, J15 Conn_01x01, J16 Conn_01x01, J17 Conn_01x01, J18 Conn_01x01, J19 Conn_01x01, J2 Conn_01x01, J20 Conn_01x01, J21 Conn_01x01, J22 Conn_01x01, J23 Conn_01x01, J24 Conn_01x01, J25 Conn_01x01, J26 Conn_01x01, J27 Conn_01x01, J28 Conn_01x01, J29 Conn_01x01, J3 Conn_01x01, J30 Conn_01x01, J31 Conn_01x01, J32 Conn_01x01, J33 Conn_01x01, J34 Conn_01x01, J35 Conn_01x01, J36 Conn_01x01, J37 Conn_01x01, J38 Conn_01x01, J4 Conn_01x01, J5 Conn_01x01, J6 Conn_01x01, J7 Conn_01x01, J8 Conn_01x01, J9 Conn_01x01, SW1 3x6mm, SW2 3x6mm, U1 LPC1769FBD100, Y1 12MHz

Commit message: layout test
Parts:
- J1, J10, J11, J12, J13, J14, J15, J16, J17, J18, J19, J2, J20, J21, J22, J23, J24, J25, J26, J27, J28, J29, J3, J30, J31, J32, J33, J34, J35, J36, J37, J38, J4, J5, J6, J7, J8, J9: footprint (none) -> _Generic:PinHeader_2.54mm_1P
- renumbered C4 to C3, C3 to C4, C6 to C5, C8 to C6, C5 to C7, C9 to C8, C7 to C9, R3 to R1, R1 to R2, R2 to R3, SW2 to SW1, SW1 to SW2

Commit message: fuses
Parts:
- JP1, JP10, JP11, JP12, JP13, JP2, JP3, JP4, JP5, JP6, JP7, JP8, JP9: footprint (none) -> _Generic:Solder Jumper 2P
- SW1, SW2: footprint (none) -> Button_Switch_SMD:SW_SPST_CK_RS282G05A3
Connections:
- net P1.18_POW renamed P1.18_ADV
- net P1.19_POW renamed P1.19_ADV
- net P2.3_ADV renamed P2.3_POW
- net P2.4_ADV renamed P2.4_POW
- net P3.26_POW renamed P3.26_BUZ
Other:
- note added: "MCOA0"
- note added: "MCOA1"
- note added: "MCOA2"
- note added: "MCOB0"
- note added: "MCOB2"
- note added: "PWM1[1]"
- note added: "PWM1[2]"
- note added: "PWM1[3]"
- note added: "PWM1[4]"
- note added: "PWM1[5]"
- note added: "PWM1[6]"
Changed lines of the file:
@@
 ISP_BOOT
 Text Label 6800 5350 2    50   ~ 0
-P2.3_ADV
+P2.3_POW
 Text Label 6800 5450 2    50   ~ 0
-P2.4_ADV
+P2.4_POW
 Wire Wire Line
 	6800 5450 6300 5450
@@
 	6300 5350 6800 5350
 Text Label 6800 3550 2    50   ~ 0
-P1.18_POW
+P1.18_ADV
 Wire Wire Line
 	6800 3550 6300 3550
 Text Label 6800 3650 2    50   ~ 0
-P1.19_POW
+P1.19_ADV
 Wire Wire Line
 	6800 3650 6300 3650
@@
 	6800 6550 6300 6550
 Text Label 6800 6650 2    50   ~ 0
-P3.26_POW
+P3.26_BUZ
 Wire Wire Line
 	6800 6650 6300 6650
@@
 F 0 "SW1" V 954 7348 50  0000 L CNN
 F 1 "3x6mm" V 1045 7348 50  0000 L CNN
-F 2 "" H 1000 7400 50  0001 C CNN
+F 2 "Button_Switch_SMD:SW_SPST_CK_RS282G05A3" H 1000 7400 50  0001 C CNN
 F 3 "" H 1000 7400 50  0001 C CNN
 	1    1000 7200
@@
 F 0 "SW2" V 2204 7398 50  0000 L CNN
 F 1 "3x6mm" V 2295 7398 50  0000 L CNN
-F 2 "" H 2250 7450 50  0001 C CNN
+F 2 "Button_Switch_SMD:SW_SPST_CK_RS282G05A3" H 2250 7450 50  0001 C CNN
 F 3 "" H 2250 7450 50  0001 C CNN
 	1    2250 7250
@@
 F1 "output.sch" 50
 F2 "POWER_OUT3" I L 10350 2100 50
-F3 "POWER_OUT4" I L 10350 2200 50
-F4 "POWER_OUT1" I L 10350 1900 50
-F5 "POWER_OUT2" I L 10350 2000 50
-F6 "HV_IO2" B L 10350 1100 50
-F7 "HV_IO7" B L 10350 1600 50
-F8 "HV_IO8" B L 10350 1700 50
-F9 "HV_IO1" B L 10350 1000 50
-F10 "HV_IO3" B L 10350 1200 50
-F11 "HV_IO4" B L 10350 1300 50
-F12 "HV_IO5" B L 10350 1400 50
-F13 "HV_IO6" B L 10350 1500 50
+F3 "POWER_OUT1" I L 10350 1900 50
+F4 "POWER_OUT2" I L 10350 2000 50
+F5 "HV_IO2" B L 10350 1100 50
+F6 "HV_IO7" B L 10350 1600 50
+F7 "HV_IO8" B L 10350 1700 50
+F8 "HV_IO1" B L 10350 1000 50
+F9 "HV_IO3" B L 10350 1200 50
+F10 "HV_IO4" B L 10350 1300 50
+F11 "HV_IO5" B L 10350 1400 50
+F12 "HV_IO6" B L 10350 1500 50
+F13 "BUZZER" I L 10350 2200 50
 $EndSheet
-Text Label 9850 1900 0    50   ~ 0
-P1.18_POW
-Text Label 9850 2000 0    50   ~ 0
-P1.19_POW
+Text Label 9850 1600 0    50   ~ 0
+P1.18_ADV
+Text Label 9850 1700 0    50   ~ 0
+P1.19_ADV
 Text Label 9850 2100 0    50   ~ 0
 P3.25_POW
 Text Label 9850 2200 0    50   ~ 0
-P3.26_POW
+P3.26_BUZ
 Wire Wire Line
 	9850 2200 10350 2200
@@
 	10350 2100 9850 2100
 Wire Wire Line
-	9850 2000 10350 2000
-Wire Wire Line
-	10350 1900 9850 1900
+	9850 1700 10350 1700
+Wire Wire Line
+	10350 1600 9850 1600
 Text Label 9850 1000 0    50   ~ 0
 P0.22_ADV
@@
 Text Label 9850 1500 0    50   ~ 0
 P1.29_ADV
-Text Label 9850 1600 0    50   ~ 0
-P2.3_ADV
-Text Label 9850 1700 0    50   ~ 0
-P2.4_ADV
-Wire Wire Line
-	9850 1700 10350 1700
-Wire Wire Line
-	10350 1600 9850 1600
+Text Label 9850 1900 0    50   ~ 0
+P2.3_POW
+Text Label 9850 2000 0    50   ~ 0
+P2.4_POW
+Wire Wire Line
+	9850 2000 10350 2000
+Wire Wire Line
+	10350 1900 9850 1900
 Wire Wire Line
 	9850 1500 10350 1500
@@
 U 1 1 5C3484AB
 P 10100 5900
-F 0 "JP9" H 10100 6013 50  0000 C CNN
+F 0 "JP9" H 10250 5950 50  0000 C CNN
 F 1 "SolderJumper_2_Open" H 10100 5900 50  0001 C CNN
-F 2 "" H 10100 5900 50  0001 C CNN
+F 2 "_Generic:Solder Jumper 2P" H 10100 5900 50  0001 C CNN
 F 3 "~" H 10100 5900 50  0001 C CNN
 	1    10100 5900
@@
 U 1 1 5C34857E
 P 10100 6000
-F 0 "JP10" H 10100 6113 50  0000 C CNN
+F 0 "JP10" H 10250 6050 50  0000 C CNN
 F 1 "SolderJumper_2_Open" H 10100 6000 50  0001 C CNN
-F 2 "" H 10100 6000 50  0001 C CNN
+F 2 "_Generic:Solder Jumper 2P" H 10100 6000 50  0001 C CNN
 F 3 "~" H 10100 6000 50  0001 C CNN
 	1    10100 6000
@@
 U 1 1 5C34862C
 P 10100 6100
-F 0 "JP11" H 10100 6213 50  0000 C CNN
+F 0 "JP11" H 10250 6150 50  0000 C CNN
 F 1 "SolderJumper_2_Open" H 10100 6100 50  0001 C CNN
-F 2 "" H 10100 6100 50  0001 C CNN
+F 2 "_Generic:Solder Jumper 2P" H 10100 6100 50  0001 C CNN
 F 3 "~" H 10100 6100 50  0001 C CNN
 	1    10100 6100
@@
 U 1 1 5C3486DD
 P 10100 6200
-F 0 "JP12" H 10100 6313 50  0000 C CNN
+F 0 "JP12" H 10250 6250 50  0000 C CNN
 F 1 "SolderJumper_2_Open" H 10100 6200 50  0001 C CNN
-F 2 "" H 10100 6200 50  0001 C CNN
+F 2 "_Generic:Solder Jumper 2P" H 10100 6200 50  0001 C CNN
 F 3 "~" H 10100 6200 50  0001 C CNN
 	1    10100 6200
@@
 U 1 1 5C34878D
 P 10100 6300
-F 0 "JP13" H 10100 6413 50  0000 C CNN
+F 0 "JP13" H 10250 6350 50  0000 C CNN
 F 1 "SolderJumper_2_Open" H 10100 6300 50  0001 C CNN
-F 2 "" H 10100 6300 50  0001 C CNN
+F 2 "_Generic:Solder Jumper 2P" H 10100 6300 50  0001 C CNN
 F 3 "~" H 10100 6300 50  0001 C CNN
 	1    10100 6300
@@
 F 0 "JP2" H 2050 5400 50  0000 C CNN
 F 1 "SolderJumper_2_Open" H 1900 5350 50  0001 C CNN
-F 2 "" H 1900 5350 50  0001 C CNN
+F 2 "_Generic:Solder Jumper 2P" H 1900 5350 50  0001 C CNN
 F 3 "~" H 1900 5350 50  0001 C CNN
 	1    1900 5350
@@
 F 0 "JP3" H 2050 5500 50  0000 C CNN
 F 1 "SolderJumper_2_Open" H 1900 5450 50  0001 C CNN
-F 2 "" H 1900 5450 50  0001 C CNN
+F 2 "_Generic:Solder Jumper 2P" H 1900 5450 50  0001 C CNN
 F 3 "~" H 1900 5450 50  0001 C CNN
 	1    1900 5450
@@
 U 1 1 5C43CD63
 P 10100 5750
-F 0 "JP8" H 10100 5863 50  0000 C CNN
+F 0 "JP8" H 10250 5800 50  0000 C CNN
 F 1 "SolderJumper_2_Open" H 10100 5750 50  0001 C CNN
-F 2 "" H 10100 5750 50  0001 C CNN
+F 2 "_Generic:Solder Jumper 2P" H 10100 5750 50  0001 C CNN
 F 3 "~" H 10100 5750 50  0001 C CNN
 	1    10100 5750
@@
 U 1 1 5C43CE29
 P 10100 5200
-F 0 "JP7" H 10100 5313 50  0000 C CNN
+F 0 "JP7" H 10250 5250 50  0000 C CNN
 F 1 "SolderJumper_2_Open" H 10100 5200 50  0001 C CNN
-F 2 "" H 10100 5200 50  0001 C CNN
+F 2 "_Generic:Solder Jumper 2P" H 10100 5200 50  0001 C CNN
 F 3 "~" H 10100 5200 50  0001 C CNN
 	1    10100 5200
@@
 U 1 1 5C43CEE0
 P 10100 4650
-F 0 "JP6" H 10100 4763 50  0000 C CNN
+F 0 "JP6" H 10250 4700 50  0000 C CNN
 F 1 "SolderJumper_2_Open" H 10100 4650 50  0001 C CNN
-F 2 "" H 10100 4650 50  0001 C CNN
+F 2 "_Generic:Solder Jumper 2P" H 10100 4650 50  0001 C CNN
 F 3 "~" H 10100 4650 50  0001 C CNN
 	1    10100 4650
@@
 U 1 1 5C43CF9E
 P 10100 4100
-F 0 "JP5" H 10100 4213 50  0000 C CNN
+F 0 "JP5" H 10250 4150 50  0000 C CNN
 F 1 "SolderJumper_2_Open" H 10100 4100 50  0001 C CNN
-F 2 "" H 10100 4100 50  0001 C CNN
+F 2 "_Generic:Solder Jumper 2P" H 10100 4100 50  0001 C CNN
 F 3 "~" H 10100 4100 50  0001 C CNN
 	1    10100 4100
@@
 U 1 1 5C43D06D
 P 10100 3350
-F 0 "JP4" H 10100 3463 50  0000 C CNN
+F 0 "JP4" H 10250 3400 50  0000 C CNN
 F 1 "SolderJumper_2_Open" H 10100 3350 50  0001 C CNN
-F 2 "" H 10100 3350 50  0001 C CNN
+F 2 "_Generic:Solder Jumper 2P" H 10100 3350 50  0001 C CNN
 F 3 "~" H 10100 3350 50  0001 C CNN
 	1    10100 3350
@@
 F 0 "JP1" H 2050 3900 50  0000 C CNN
 F 1 "SolderJumper_2_Open" H 1900 3850 50  0001 C CNN
-F 2 "" H 1900 3850 50  0001 C CNN
+F 2 "_Generic:Solder Jumper 2P" H 1900 3850 50  0001 C CNN
 F 3 "~" H 1900 3850 50  0001 C CNN
 	1    1900 3850
@@
 Text Notes 9100 2750 0    100  ~ 20
 Stepper Driver
+Text Notes 9400 2200 0    50   ~ 0
+PWM1[3]
+Text Notes 9400 1300 0    50   ~ 0
+PWM1[6]
+Text Notes 9400 1200 0    50   ~ 0
+MCOA1
+Text Notes 9400 1400 0    50   ~ 0
+MCOA2
+Text Notes 9400 1500 0    50   ~ 0
+MCOB2
+Text Notes 9400 2100 0    50   ~ 0
+PWM1[2]
+Text Notes 9400 2000 0    50   ~ 0
+PWM1[5]
+Text Notes 9400 1900 0    50   ~ 0
+PWM1[4]
+Text Notes 9400 1100 0    50   ~ 0
+MCOB0
+Text Notes 9400 1600 0    50   ~ 0
+PWM1[1]
+Text Notes 9400 1700 0    50   ~ 0
+MCOA0
 $EndSCHEMATC

Commit message: continue routing
Changed lines of the file:
@@
 F8 "USB_D-" B R 1750 4250 50
 F9 "USB_CON" I R 1750 4050 50
-F10 "TXD" I R 1750 4850 50
-F11 "RXD" O R 1750 4750 50
-F12 "ISP_BOOT" I R 1750 4950 50
 F13 "ENDSTOP1" O R 1750 2100 50
 F14 "ENDSTOP2" O R 1750 2200 50
@@
 Wire Wire Line
 	1750 4450 2250 4450
-Text Label 2250 4750 2    50   ~ 0
-RXD
-Text Label 2250 4850 2    50   ~ 0
-TXD
-Text Label 2250 4950 2    50   ~ 0
-ISP_BOOT
-Wire Wire Line
-	2250 4950 1750 4950
-Wire Wire Line
-	1750 4850 2250 4850
-Wire Wire Line
-	2250 4750 1750 4750
 Text Label 4000 3150 0    50   ~ 0
 SD_CS

Commit message: continue routing
Parts:
- removed Y1: 12MHz, symbol Device:Crystal_GND24
- added C80: 100p, _Generic:0603_CAP, symbol Device:C_Small
- added R80: 1k, _Generic:0603_RES, symbol Device:R
- added X1: 12MHz, Oscillator:Oscillator_SMD_EuroQuartz_XO32-4Pin_3.2x2.5mm, symbol Oscillator:XO32
- C3: value 12p -> 220p
- C5: value 12p -> 100n
Connections:
- net +3V3: now also C5.1, X1.1 (EN), X1.4 (V+)
- net GND: now also X1.2 (GND)
- net LPC_CLK: now reaches U1.22 (XTAL1)
- net LPC_CLK: now also C3.1, C80.1
- new net: C80.2, R80.2, X1.3 (OUT)
- new net DRV_CLK: R80.1
- no-connect marks 3 -> 4
Other:
- note added: "Clock"
- note removed: "|\n| SPI\n|\n|\n|"
- moved on the sheet: C1, C10, C11, C12, C13, C14, C15, C16, C17, C2, C3, C4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

Commit message: continue routing
Parts:
- added C19, C26, C31: 10u, _Generic:0603_CAP, symbol Device:C_Small
- added J104, J52, J75, J76, J77, J78: Conn_01x01, _Generic:PinHeader_2.54mm_1P, symbol #Connector:Conn_01x01
- SW1, SW2: footprint Button_Switch_SMD:SW_SPST_CK_RS282G05A3 -> _Generic:Switch_3x4mm
Connections:
- net +3V3: now also C19.1, C26.1, C31.1
- net DRV1_DIR: now also U1.95 (P1[0]); no longer U1.94 (P1[1])
- net DRV1_EN: now also U1.94 (P1[1]); no longer U1.95 (P1[0])
- net DRV2_DIR: now also U1.93 (P1[4]); no longer U1.92 (P1[8])
- net DRV2_EN: now also U1.92 (P1[8]); no longer U1.93 (P1[4])
- net DRV3_DIR: now also U1.91 (P1[9]); no longer U1.90 (P1[10])
- net DRV3_EN: now also U1.90 (P1[10]); no longer U1.91 (P1[9])
- net DRV4_DIR: now also U1.89 (P1[14]); no longer U1.88 (P1[15])
- net DRV4_EN: now also U1.88 (P1[15]); no longer U1.89 (P1[14])
- net DRV5_DIR: now also J25.1 (Pin_1), U1.87 (P1[16]); no longer J26.1 (Pin_1), U1.86 (P1[17])
- net DRV5_EN: now also J26.1 (Pin_1), U1.86 (P1[17]); no longer J25.1 (Pin_1), U1.87 (P1[16])
- net GND: now also C19.2, C26.2, C31.2
- net P1.30_GEN: now also J75.1 (Pin_1)
- net P1.31_GEN: now also J76.1 (Pin_1)
- net P3.26_BUZ: now also J104.1 (Pin_1)
- net P4.28_GEN: now also J77.1 (Pin_1)
- net P4.29_GEN: now also J78.1 (Pin_1)
- net USB_CON: now also J52.1 (Pin_1)
Other:
- moved on the sheet: C10, C11, C12, C13, C14, C2, C4, C6, C7, C8, C9

Commit message: PCB V1
Parts:
- added JP16: SolderJumper_3_Open, _Generic:Solder Jumper 3P, symbol #PCB_Only:SolderJumper_3_Open
- added R37, R42: 4.7k, _Generic:0603_RES, symbol Device:R
Connections:
- net +3V3: now also JP16.3 (B)
- net SCL: now also R37.2
- net SDA: now also R42.2
- net P1.30_GEN renamed P1.30
- net P1.31_GEN renamed P1.31
- net P4.28_GEN renamed P4.28
- net P4.29_GEN renamed P4.29
- new net: JP16.2 (C), R37.1, R42.1
- new net +5V: JP16.1 (A)
Other:
- note removed: "CAPS\n12p, 0603, 50v\n470p, 0603, 50v\n22n, 0603, 100v\n100n, 0603, 50v\n470n, 0603, 25v\n4.7u, 0805, 50v\n10u, 0603, 16v\n390u, 8x12mm, 20v\n68u, 8x10mm, 50v"
- moved on the sheet: JP1, JP2, JP3, JP4
