File: hardware/kajikia/power.sch (KiCad schematic (older format))
At the start: 0 parts

Commit message: power
Parts:
- added C162, C164, C168, C? (x5): 4.7u, symbol Device:C_Small
- added C166, C174, C? (x2): 100n, symbol Device:C_Small
- added C170, C?: 22n, symbol Device:C_Small
- added C172, C?: 100k, symbol Device:C_Small
- added C176, C?: DNP, symbol Device:C_Small
- added C178, C? (x5): 10u, symbol Device:C_Small
- added C? (x2): 390u, symbol Device:CP1_Small
- added C?: 68u, symbol Device:CP1_Small
- added D69: V25PN60, symbol Device:D_Schottky
- added D70, D?: 3.6v, symbol Device:D_Zener
- added D72, D?: SK54, symbol Device:D_Schottky
- added D?: LED, symbol Device:LED_Small
- added F5: Fuse, symbol Device:Fuse
- added J73: Conn_01x02, symbol Connector_Generic:Conn_01x02
- added J? (x20): Conn_01x01, symbol #Connector:Conn_01x01
- added JP?: SolderJumper_2_Open, symbol #PCB_Only:SolderJumper_2_Open
- added L5, L?: BCIHP0750-6R8M, symbol Device:L
- added L?: 1u, symbol Device:L
- added R121, R?: 47k, symbol Device:R
- added R123, R127, R?: 140k, symbol Device:R
- added R125, R?: 12p, symbol Device:R
- added R128, R?: 10k, symbol Device:R
- added R?: 52.3k, symbol Device:R
- added R?: 1k, symbol Device:R_Small
- added U6, U?: AOZ1284, symbol #Regulator:AOZ1284
- added U?: LM1117-3.3, symbol Regulator_Linear:LM1117-3.3
Connections:
- new net: F5.2, J73.2 (Pin_2)
- new net: C?.2, D?.1 (K), L?.1, U?.1 (LX)
- new net: C?.1, U?.2 (BST)
- new net: R?.1, U?.4 (FSW)
- new net: C?.1, U?.5 (COMP)
- new net: C?.2, R?.1, R?.2, U?.6 (FB)
- new net: C?.1, U?.7 (SS)
- new net: C?.1, D?.1 (K), R?.2, U?.8 (EN)
- new net: C?.2, R?.1
- new net: C?.2, C?.2, C?.2, C?.2, U?.1 (GND)
- new net: C?.1, L?.2, U?.3 (VI)
- new net: D?.1 (K), R?.1
- new net: C174.2, D72.1 (K), L5.1, U6.1 (LX)
- new net: C174.1, U6.2 (BST)
- new net: R121.1, U6.4 (FSW)
- new net: C172.1, U6.5 (COMP)
- new net: C176.2, R127.2, R128.1, U6.6 (FB)
- new net: C170.1, U6.7 (SS)
- new net: C166.1, D70.1 (K), R123.2, U6.8 (EN)
- new net: C172.2, R125.1
- new net +12V: C176.1, C178.1, C?.1, J?.1 (Pin_1), J?.1 (Pin_1), J?.1 (Pin_1), J?.1 (Pin_1), JP?.2 (B), L5.2, R127.1
- new net +24V: C162.1, C164.1, C168.1, C?.1, C?.1, C?.1, C?.1, C?.1, C?.1, D69.1 (K), F5.1, J?.1 (Pin_1), J?.1 (Pin_1), J?.1 (Pin_1), J?.1 (Pin_1), JP?.1 (A), R123.1, R?.1, U6.PAD (VIN), U?.PAD (VIN)
- new net +3V3: C?.1, C?.1, D?.2 (A), J?.1 (Pin_1), J?.1 (Pin_1), J?.1 (Pin_1), J?.1 (Pin_1), U?.2 (VO)
- new net +5V: C?.1, C?.1, C?.1, C?.1, J?.1 (Pin_1), J?.1 (Pin_1), J?.1 (Pin_1), J?.1 (Pin_1), L?.1, L?.2, R?.1
- new net GND: C162.2, C164.2, C166.2, C168.2, C170.2, C178.2, C?.2, C?.2, C?.2, C?.2, C?.2, C?.2, C?.2, C?.2, C?.2, C?.2, C?.2, D69.2 (A), D70.2 (A), D72.2 (A), D?.2 (A), D?.2 (A), J73.1 (Pin_1), J?.1 (Pin_1), J?.1 (Pin_1), J?.1 (Pin_1), J?.1 (Pin_1), R121.2, R125.2, R128.2, R?.2, R?.2, R?.2, R?.2, U6.3 (GND), U?.3 (GND)

Commit message: fancy
Parts:
- C155, C156, C158, C160, C164: renamed from C?; footprint (none) -> _Generic:0805_CAP
- C157: renamed from C162; footprint (none) -> _Generic:0805_CAP
- C159: renamed from C164; footprint (none) -> _Generic:0805_CAP
- C161: renamed from C166; footprint (none) -> _Generic:0603_CAP
- C162, C166, C170, C172, C174, C177, C178, C179, C180: renamed from C?; footprint (none) -> _Generic:0603_CAP
- C163: renamed from C168; footprint (none) -> _Generic:0805_CAP
- C165: renamed from C170; footprint (none) -> _Generic:0603_CAP
- C167: renamed from C172; value 100k -> 12p; footprint (none) -> _Generic:0603_CAP
- C168: renamed from C?; value 100k -> 12p; footprint (none) -> _Generic:0603_CAP
- C169: renamed from C174; footprint (none) -> _Generic:0603_CAP
- C171: renamed from C176; footprint (none) -> _Generic:0603_CAP
- C173: renamed from C178; footprint (none) -> _Generic:0603_CAP
- D66: renamed from D?; footprint (none) -> _Generic:0603_LED
- R113: renamed from R121; footprint (none) -> _Generic:0603_RES
- R114, R116, R121, R122, R123: renamed from R?; footprint (none) -> _Generic:0603_RES
- R115: renamed from R123; footprint (none) -> _Generic:0603_RES
- R117: renamed from R125; value 12p -> 100k; footprint (none) -> _Generic:0603_RES
- R118: renamed from R?; value 12p -> 100k; footprint (none) -> _Generic:0603_RES
- R119: renamed from R127; footprint (none) -> _Generic:0603_RES
- R120: renamed from R128; footprint (none) -> _Generic:0603_RES
- gave numbers to parts that had none: 30
- renumbered D70 to D61, D69 to D63, D72 to D64
Connections:
- net GND: now also C177.2, C178.2, C179.2, C180.2, U8.1 (GND)
Other:
- note added: "12V Regulator"
- note added: "3.3V Regulator"
- note added: "5V Regulator"
- note added: "Common Decoupling"
- note added: "DC Input"
- note added: "Power LED"
- note added: "Power Pins"
- moved on the sheet: C154, C155, C156, C157, C158, C159, C160, C161, C162, C163, C164, C165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
