File: hardware/kajikia/power.sch (KiCad schematic (older format))
At the start: 73 parts, among them J73 Conn_01x02, J74 Conn_01x01, J75 Conn_01x01, J76 Conn_01x01, J77 Conn_01x01, J78 Conn_01x01, J79 Conn_01x01, J80 Conn_01x01, J81 Conn_01x01, J82 Conn_01x01, J83 Conn_01x01, J84 Conn_01x01, J85 Conn_01x01, J86 Conn_01x01, J87 Conn_01x01, J88 Conn_01x01, J89 Conn_01x01, J90 Conn_01x01, J91 Conn_01x01, J92 Conn_01x01, J93 Conn_01x01, U6 AOZ1284, U7 AOZ1284, U8 LM1117-3.3

Commit message: footprints
Parts:
- removed D63: V25PN60, symbol Device:D_Schottky
- added D63: 16v, _Generic:SOD-523_DIODE, symbol Device:D_Zener
- added Q14: AON6144, _Generic:DFN5x6-8, symbol Device:Q_NMOS_SGD
- added R124: 10k, _Generic:0603_RES, symbol Device:R
- added R125: 100k, _Generic:0603_RES, symbol Device:R
- C154, C175, C176: footprint (none) -> Capacitor_SMD:CP_Elec_8x10
- D61, D62: footprint (none) -> _Generic:SOD-523_DIODE
- D64, D65: footprint (none) -> Diode_SMD:D_SMB
- L5, L6: footprint (none) -> _Generic:7x7mm_IND
- L7: footprint (none) -> _Generic:0805_IND
- U6, U7: footprint (none) -> _Generic:SO-8-EP1
- U8: footprint (none) -> Package_TO_SOT_SMD:SOT-223-3_TabPin2
Connections:
- net +24V: now also R124.1
- net GND: now also D63.2 (A), Q14.1 (S), R125.2; no longer J73.1 (Pin_1)
- new net: J73.1 (Pin_1), Q14.3 (D)
- new net: D63.1 (K), Q14.2 (G), R124.2, R125.1
Other:
- note added: "Replace with DMT40M9LPS for\nhigher current application > 25A"
- moved on the sheet: F5, J73
Changed lines of the file:
@@
 F 0 "U6" H 6500 2300 50  0000 C CNN
 F 1 "AOZ1284" H 5850 2300 50  0000 C CNN
-F 2 "" H 6150 1350 50  0001 C CIN
+F 2 "_Generic:SO-8-EP1" H 6150 1350 50  0001 C CIN
 F 3 "" H 5750 2300 50  0001 C CNN
 	1    6150 1850
@@
 F 0 "L5" V 7640 1750 50  0000 C CNN
 F 1 "BCIHP0750-6R8M" V 7549 1750 50  0000 C CNN
-F 2 "" H 7450 1750 50  0001 C CNN
+F 2 "_Generic:7x7mm_IND" H 7450 1750 50  0001 C CNN
 F 3 "~" H 7450 1750 50  0001 C CNN
 	1    7450 1750
@@
 F 0 "D64" V 7154 2029 50  0000 L CNN
 F 1 "SK54" V 7245 2029 50  0000 L CNN
-F 2 "" H 7200 1950 50  0001 C CNN
+F 2 "Diode_SMD:D_SMB" H 7200 1950 50  0001 C CNN
 F 3 "~" H 7200 1950 50  0001 C CNN
 	1    7200 1950
@@
 F 0 "D61" V 4204 2279 50  0000 L CNN
 F 1 "3.6v" V 4295 2279 50  0000 L CNN
-F 2 "" H 4250 2200 50  0001 C CNN
+F 2 "_Generic:SOD-523_DIODE" H 4250 2200 50  0001 C CNN
 F 3 "~" H 4250 2200 50  0001 C CNN
 	1    4250 2200
@@
 	8100 2150 7700 2150
 $Comp
-L Device:D_Schottky D63
-U 1 1 5C32C9D8
-P 2050 1500
-F 0 "D63" V 2004 1579 50  0000 L CNN
-F 1 "V25PN60" V 2095 1579 50  0000 L CNN
-F 2 "" H 2050 1500 50  0001 C CNN
-F 3 "~" H 2050 1500 50  0001 C CNN
-	1    2050 1500
-	0    1    1    0
-$EndComp
-$Comp
 L Connector_Generic:Conn_01x02 J73
 U 1 1 5C330DAD
-P 1050 1550
-F 0 "J73" H 970 1225 50  0000 C CNN
-F 1 "Conn_01x02" H 970 1316 50  0000 C CNN
-F 2 "" H 1050 1550 50  0001 C CNN
-F 3 "~" H 1050 1550 50  0001 C CNN
-	1    1050 1550
+P 1050 1500
+F 0 "J73" H 970 1175 50  0000 C CNN
+F 1 "Conn_01x02" H 970 1266 50  0000 C CNN
+F 2 "" H 1050 1500 50  0001 C CNN
+F 3 "~" H 1050 1500 50  0001 C CNN
+	1    1050 1500
 	-1   0    0    1
 $EndComp
@@
 L power:+24V #PWR0174
 U 1 1 5C334E02
-P 2050 1200
-F 0 "#PWR0174" H 2050 1050 50  0001 C CNN
-F 1 "+24V" H 2065 1373 50  0000 C CNN
-F 2 "" H 2050 1200 50  0001 C CNN
-F 3 "" H 2050 1200 50  0001 C CNN
-	1    2050 1200
-	1    0    0    -1
-$EndComp
-Wire Wire Line
-	1250 1550 1400 1550
-Wire Wire Line
-	1400 1550 1400 1700
-Wire Wire Line
-	2050 1700 2050 1650
-Wire Wire Line
-	2050 1350 2050 1300
-Wire Wire Line
-	1250 1450 1400 1450
-Wire Wire Line
-	1400 1450 1400 1300
+P 2400 1050
+F 0 "#PWR0174" H 2400 900 50  0001 C CNN
+F 1 "+24V" H 2415 1223 50  0000 C CNN
+F 2 "" H 2400 1050 50  0001 C CNN
+F 3 "" H 2400 1050 50  0001 C CNN
+	1    2400 1050
+	1    0    0    -1
+$EndComp
+Wire Wire Line
+	1250 1500 1400 1500
+Wire Wire Line
+	1400 1500 1400 1950
+Wire Wire Line
+	1250 1400 1400 1400
+Wire Wire Line
+	1400 1400 1400 1150
 $Comp
 L #Power:GND #PWR0175
 U 1 1 5C34B6E8
-P 2050 1800
-F 0 "#PWR0175" H 2050 1550 50  0001 C CNN
-F 1 "GND" H 2050 1650 50  0001 C CNN
-F 2 "" H 2050 1800 50  0001 C CNN
-F 3 "" H 2050 1800 50  0001 C CNN
-	1    2050 1800
-	1    0    0    -1
-$EndComp
-Wire Wire Line
-	2050 1700 2050 1800
-Wire Wire Line
-	2050 1200 2050 1300
-Connection ~ 2050 1300
-Connection ~ 2050 1700
-Wire Wire Line
-	1400 1700 1700 1700
-Wire Wire Line
-	1400 1300 1450 1300
+P 2400 2050
+F 0 "#PWR0175" H 2400 1800 50  0001 C CNN
+F 1 "GND" H 2400 1900 50  0001 C CNN
+F 2 "" H 2400 2050 50  0001 C CNN
+F 3 "" H 2400 2050 50  0001 C CNN
+	1    2400 2050
+	1    0    0    -1
+$EndComp
+Wire Wire Line
+	2400 1950 2400 2050
+Wire Wire Line
+	2400 1050 2400 1150
+Wire Wire Line
+	1400 1150 1500 1150
 $Comp
 L Device:Fuse F5
 U 1 1 5C35C7B9
-P 1600 1300
-F 0 "F5" V 1403 1300 50  0000 C CNN
-F 1 "Fuse" V 1494 1300 50  0000 C CNN
-F 2 "" V 1530 1300 50  0001 C CNN
-F 3 "~" H 1600 1300 50  0001 C CNN
-	1    1600 1300
+P 1650 1150
+F 0 "F5" V 1453 1150 50  0000 C CNN
+F 1 "Fuse" V 1544 1150 50  0000 C CNN
+F 2 "" V 1580 1150 50  0001 C CNN
+F 3 "~" H 1650 1150 50  0001 C CNN
+	1    1650 1150
 	0    1    1    0
 $EndComp
-Wire Wire Line
-	1750 1300 2050 1300
 $Comp
 L power:+12V #PWR0185
@@
 F 0 "C175" H 9041 1996 50  0000 L CNN
 F 1 "390u" H 9041 1905 50  0000 L CNN
-F 2 "" H 8950 1950 50  0001 C CNN
+F 2 "Capacitor_SMD:CP_Elec_8x10" H 8950 1950 50  0001 C CNN
 F 3 "~" H 8950 1950 50  0001 C CNN
 	1    8950 1950
@@
 F 0 "U7" H 6500 4950 50  0000 C CNN
 F 1 "AOZ1284" H 5850 4950 50  0000 C CNN
-F 2 "" H 6150 4000 50  0001 C CIN
+F 2 "_Generic:SO-8-EP1" H 6150 4000 50  0001 C CIN
 F 3 "" H 5750 4950 50  0001 C CNN
 	1    6150 4500
@@
 F 0 "L6" V 7640 4400 50  0000 C CNN
 F 1 "BCIHP0750-6R8M" V 7549 4400 50  0000 C CNN
-F 2 "" H 7450 4400 50  0001 C CNN
+F 2 "_Generic:7x7mm_IND" H 7450 4400 50  0001 C CNN
 F 3 "~" H 7450 4400 50  0001 C CNN
 	1    7450 4400
@@
 F 0 "D65" V 7154 4679 50  0000 L CNN
 F 1 "SK54" V 7245 4679 50  0000 L CNN
-F 2 "" H 7200 4600 50  0001 C CNN
+F 2 "Diode_SMD:D_SMB" H 7200 4600 50  0001 C CNN
 F 3 "~" H 7200 4600 50  0001 C CNN
 	1    7200 4600
@@
 F 0 "D62" V 4204 4929 50  0000 L CNN
 F 1 "3.6v" V 4295 4929 50  0000 L CNN
-F 2 "" H 4250 4850 50  0001 C CNN
+F 2 "_Generic:SOD-523_DIODE" H 4250 4850 50  0001 C CNN
 F 3 "~" H 4250 4850 50  0001 C CNN
 	1    4250 4850
@@
 F 0 "C176" H 9041 4646 50  0000 L CNN
 F 1 "390u" H 9041 4555 50  0000 L CNN
-F 2 "" H 8950 4600 50  0001 C CNN
+F 2 "Capacitor_SMD:CP_Elec_8x10" H 8950 4600 50  0001 C CNN
 F 3 "~" H 8950 4600 50  0001 C CNN
 	1    8950 4600
@@
 F 0 "C154" H 1791 4196 50  0000 L CNN
 F 1 "68u" H 1791 4105 50  0000 L CNN
-F 2 "" H 1700 4150 50  0001 C CNN
+F 2 "Capacitor_SMD:CP_Elec_8x10" H 1700 4150 50  0001 C CNN
 F 3 "~" H 1700 4150 50  0001 C CNN
 	1    1700 4150
@@
 F 0 "U8" H 2450 6992 50  0000 C CNN
 F 1 "LM1117-3.3" H 2450 6901 50  0000 C CNN
-F 2 "" H 2450 6750 50  0001 C CNN
+F 2 "Package_TO_SOT_SMD:SOT-223-3_TabPin2" H 2450 6750 50  0001 C CNN
 F 3 "http://www.ti.com/lit/ds/symlink/lm1117.pdf" H 2450 6750 50  0001 C CNN
 	1    2450 6750
@@
 F 0 "L7" V 1940 6750 50  0000 C CNN
 F 1 "1u" V 1849 6750 50  0000 C CNN
-F 2 "" H 1750 6750 50  0001 C CNN
+F 2 "_Generic:0805_IND" H 1750 6750 50  0001 C CNN
 F 3 "~" H 1750 6750 50  0001 C CNN
 	1    1750 6750
@@
 Wire Wire Line
 	8550 4400 8950 4400
-$Comp
-L power:PWR_FLAG #FLG012
-U 1 1 5C51A64E
-P 2500 1200
-F 0 "#FLG012" H 2500 1275 50  0001 C CNN
-F 1 "PWR_FLAG" H 2500 1374 50  0000 C CNN
-F 2 "" H 2500 1200 50  0001 C CNN
-F 3 "~" H 2500 1200 50  0001 C CNN
-	1    2500 1200
-	1    0    0    -1
-$EndComp
-Wire Wire Line
-	2500 1200 2500 1300
-Wire Wire Line
-	2500 1300 2050 1300
-$Comp
-L power:PWR_FLAG #FLG011
-U 1 1 5C5471E7
-P 1700 1700
-F 0 "#FLG011" H 1700 1775 50  0001 C CNN
-F 1 "PWR_FLAG" H 1700 1874 50  0000 C CNN
-F 2 "" H 1700 1700 50  0001 C CNN
-F 3 "~" H 1700 1700 50  0001 C CNN
-	1    1700 1700
-	1    0    0    -1
-$EndComp
-Connection ~ 1700 1700
-Wire Wire Line
-	1700 1700 2050 1700
 $Comp
 L power:PWR_FLAG #FLG013
@@
 Text Notes 4450 6000 0    100  ~ 20
 Power LED
+Wire Wire Line
+	1400 1950 1450 1950
+$Comp
+L Device:Q_NMOS_SGD Q14
+U 1 1 5C3AA6BF
+P 1650 1850
+F 0 "Q14" V 1900 1850 50  0000 C CNN
+F 1 "AON6144" V 1991 1850 50  0000 C CNN
+F 2 "_Generic:DFN5x6-8" H 1850 1950 50  0001 C CNN
+F 3 "~" H 1650 1850 50  0001 C CNN
+	1    1650 1850
+	0    -1   1    0
+$EndComp
+Wire Wire Line
+	1850 1950 2000 1950
+$Comp
+L Device:R R124
+U 1 1 5C407302
+P 2000 1350
+F 0 "R124" H 2070 1396 50  0000 L CNN
+F 1 "10k" H 2070 1305 50  0000 L CNN
+F 2 "_Generic:0603_RES" V 1930 1350 50  0001 C CNN
+F 3 "~" H 2000 1350 50  0001 C CNN
+	1    2000 1350
+	1    0    0    -1
+$EndComp
+$Comp
+L Device:D_Zener D63
+U 1 1 5C407892
+P 2400 1750
+F 0 "D63" V 2354 1829 50  0000 L CNN
+F 1 "16v" V 2445 1829 50  0000 L CNN
+F 2 "_Generic:SOD-523_DIODE" H 2400 1750 50  0001 C CNN
+F 3 "~" H 2400 1750 50  0001 C CNN
+	1    2400 1750
+	0    1    1    0
+$EndComp
+Wire Wire Line
+	2400 1600 2400 1550
+Wire Wire Line
+	2400 1550 2000 1550
+Wire Wire Line
+	1650 1550 1650 1650
+Wire Wire Line
+	2000 1550 2000 1500
+Wire Wire Line
+	2400 1900 2400 1950
+Connection ~ 2400 1950
+$Comp
+L Device:R R125
+U 1 1 5C479547
+P 2000 1750
+F 0 "R125" H 2070 1796 50  0000 L CNN
+F 1 "100k" H 2070 1705 50  0000 L CNN
+F 2 "_Generic:0603_RES" V 1930 1750 50  0001 C CNN
+F 3 "~" H 2000 1750 50  0001 C CNN
+	1    2000 1750
+	1    0    0    -1
+$EndComp
+Wire Wire Line
+	2000 1900 2000 1950
+Connection ~ 2000 1950
+Wire Wire Line
+	2000 1950 2100 1950
+Wire Wire Line
+	2000 1600 2000 1550
+Connection ~ 2000 1550
+Wire Wire Line
+	2000 1550 1650 1550
+Text Notes 850  2100 0    25   ~ 0
+Replace with DMT40M9LPS for\nhigher current application > 25A
+$Comp
+L power:PWR_FLAG #FLG0101
+U 1 1 5C5382D5
+P 2100 2000
+F 0 "#FLG0101" H 2100 2075 50  0001 C CNN
+F 1 "PWR_FLAG" H 2100 2173 50  0000 C CNN
+F 2 "" H 2100 2000 50  0001 C CNN
+F 3 "~" H 2100 2000 50  0001 C CNN
+	1    2100 2000
+	-1   0    0    1
+$EndComp
+Wire Wire Line
+	2100 2000 2100 1950
+Connection ~ 2100 1950
+Wire Wire Line
+	2100 1950 2400 1950
+$Comp
+L power:PWR_FLAG #FLG0102
+U 1 1 5C5499F4
+P 2100 1100
+F 0 "#FLG0102" H 2100 1175 50  0001 C CNN
+F 1 "PWR_FLAG" H 2100 1274 50  0000 C CNN
+F 2 "" H 2100 1100 50  0001 C CNN
+F 3 "~" H 2100 1100 50  0001 C CNN
+	1    2100 1100
+	1    0    0    -1
+$EndComp
+Wire Wire Line
+	2100 1100 2100 1150
+Connection ~ 2100 1150
+Wire Wire Line
+	2100 1150 2400 1150
+Wire Wire Line
+	2000 1200 2000 1150
+Connection ~ 2000 1150
+Wire Wire Line
+	2000 1150 2100 1150
+Wire Wire Line
+	1800 1150 2000 1150
 $EndSCHEMATC

Commit message: layout test
Parts:
- removed J73: Conn_01x02, symbol Connector_Generic:Conn_01x02
- added J39: Screw_Terminal_01x02, _Generic:KF635-2P, symbol Connector:Screw_Terminal_01x02
- D5: renamed from D64; footprint Diode_SMD:D_SMB -> _Generic:SMB_DIODE
- D6: renamed from D65; footprint Diode_SMD:D_SMB -> _Generic:SMB_DIODE
- F1: renamed from F5; value Fuse -> FUSE; footprint (none) -> _Generic:SMD_Fuseholder
- J40: renamed from J90; footprint (none) -> _Generic:PinHeader_2.54mm_1P
- J41: renamed from J91; footprint (none) -> _Generic:PinHeader_2.54mm_1P
- J42: renamed from J92; footprint (none) -> _Generic:PinHeader_2.54mm_1P
- J43: renamed from J93; footprint (none) -> _Generic:PinHeader_2.54mm_1P
- J44: renamed from J86; footprint (none) -> _Generic:PinHeader_2.54mm_1P
- J45: renamed from J87; footprint (none) -> _Generic:PinHeader_2.54mm_1P
- J46: renamed from J88; footprint (none) -> _Generic:PinHeader_2.54mm_1P
- J47: renamed from J89; footprint (none) -> _Generic:PinHeader_2.54mm_1P
- J48: renamed from J82; footprint (none) -> _Generic:PinHeader_2.54mm_1P
- J49: renamed from J83; footprint (none) -> _Generic:PinHeader_2.54mm_1P
- J50: renamed from J84; footprint (none) -> _Generic:PinHeader_2.54mm_1P
- J51: renamed from J85; footprint (none) -> _Generic:PinHeader_2.54mm_1P
- J52: renamed from J78; footprint (none) -> _Generic:PinHeader_2.54mm_1P
- J53: renamed from J79; footprint (none) -> _Generic:PinHeader_2.54mm_1P
- J54: renamed from J80; footprint (none) -> _Generic:PinHeader_2.54mm_1P
- J55: renamed from J81; footprint (none) -> _Generic:PinHeader_2.54mm_1P
- J56: renamed from J74; footprint (none) -> _Generic:PinHeader_2.54mm_1P
- J57: renamed from J75; footprint (none) -> _Generic:PinHeader_2.54mm_1P
- J58: renamed from J76; footprint (none) -> _Generic:PinHeader_2.54mm_1P
- J59: renamed from J77; footprint (none) -> _Generic:PinHeader_2.54mm_1P
- renumbered C177 to C18, C154 to C19, C178 to C20, C179 to C21, C180 to C22, C155 to C23, C156 to C24, C157 to C25, C158 to C26, C159 to C27, C160 to C28, C161 to C29, C162 to C30, C163 to C31, C164 to C32, C165 to C33, C166 to C34, C167 to C35, C168 to C36, C169 to C37, C170 to C38, C171 to C39, C172 to C40, C173 to C41, C174 to C42, C175 to C43, C176 to C44, D63 to D1, D61 to D2, D62 to D3, D66 to D4, JP42 to JP14, L7 to L1, L5 to L2, L6 to L3, Q14 to Q1, R113 to R10, R114 to R11, R115 to R12, R116 to R13, R123 to R14, R117 to R15, R118 to R16, R119 to R17, R120 to R18, R121 to R19, R122 to R20, R124 to R8, R125 to R9, U8 to U2, U6 to U3, U7 to U4
Connections:
- net at Q1.3 (D): now also J39.1 (Pin_1)
- net at F1.2: now also J39.2 (Pin_2)

Commit message: tmc layout
Parts:
- added H1, H2, H3, H4: M3, MountingHole:MountingHole_3.2mm_M3_ISO14580_Pad, symbol Mechanical:MountingHole_Pad
Connections:
- net GND: now also H1.1, H2.1, H3.1, H4.1
Changed lines of the file:
@@
 	-1   0    0    1
 $EndComp
+$Comp
+L Mechanical:MountingHole_Pad H1
+U 1 1 5C3850E4
+P 7800 6100
+F 0 "H1" H 7900 6151 50  0000 L CNN
+F 1 "M3" H 7900 6060 50  0000 L CNN
+F 2 "MountingHole:MountingHole_3.2mm_M3_ISO14580_Pad" H 7800 6100 50  0001 C CNN
+F 3 "~" H 7800 6100 50  0001 C CNN
+	1    7800 6100
+	1    0    0    -1
+$EndComp
+$Comp
+L Mechanical:MountingHole_Pad H2
+U 1 1 5C3852A7
+P 8200 6100
+F 0 "H2" H 8300 6151 50  0000 L CNN
+F 1 "M3" H 8300 6060 50  0000 L CNN
+F 2 "MountingHole:MountingHole_3.2mm_M3_ISO14580_Pad" H 8200 6100 50  0001 C CNN
+F 3 "~" H 8200 6100 50  0001 C CNN
+	1    8200 6100
+	1    0    0    -1
+$EndComp
+$Comp
+L Mechanical:MountingHole_Pad H3
+U 1 1 5C38532F
+P 8600 6100
+F 0 "H3" H 8700 6151 50  0000 L CNN
+F 1 "M3" H 8700 6060 50  0000 L CNN
+F 2 "MountingHole:MountingHole_3.2mm_M3_ISO14580_Pad" H 8600 6100 50  0001 C CNN
+F 3 "~" H 8600 6100 50  0001 C CNN
+	1    8600 6100
+	1    0    0    -1
+$EndComp
+$Comp
+L Mechanical:MountingHole_Pad H4
+U 1 1 5C3853B9
+P 9000 6100
+F 0 "H4" H 9100 6151 50  0000 L CNN
+F 1 "M3" H 9100 6060 50  0000 L CNN
+F 2 "MountingHole:MountingHole_3.2mm_M3_ISO14580_Pad" H 9000 6100 50  0001 C CNN
+F 3 "~" H 9000 6100 50  0001 C CNN
+	1    9000 6100
+	1    0    0    -1
+$EndComp
+$Comp
+L #Power:GND #PWR0201
+U 1 1 5C385548
+P 8400 6350
+F 0 "#PWR0201" H 8400 6100 50  0001 C CNN
+F 1 "GND" H 8400 6200 50  0001 C CNN
+F 2 "" H 8400 6350 50  0001 C CNN
+F 3 "" H 8400 6350 50  0001 C CNN
+	1    8400 6350
+	1    0    0    -1
+$EndComp
+Wire Wire Line
+	7800 6200 7800 6300
+Wire Wire Line
+	7800 6300 8200 6300
+Wire Wire Line
+	9000 6300 9000 6200
+Wire Wire Line
+	8600 6200 8600 6300
+Connection ~ 8600 6300
+Wire Wire Line
+	8600 6300 9000 6300
+Wire Wire Line
+	8200 6300 8200 6200
+Connection ~ 8200 6300
+Wire Wire Line
+	8200 6300 8400 6300
+Wire Wire Line
+	8400 6350 8400 6300
+Connection ~ 8400 6300
+Wire Wire Line
+	8400 6300 8600 6300
 $EndSCHEMATC

Commit message: driver polys
Connections:
- net DCIN+: now reaches F1.2, J39.2 (Pin_2)
- net DCIN-: now reaches J39.1 (Pin_1), Q1.3 (D)
Changed lines of the file:
@@
 Wire Wire Line
 	2000 1550 1650 1550
-Text Notes 850  2100 0    25   ~ 0
+Text Notes 700  2200 0    25   ~ 0
 Replace with DMT40M9LPS for\nhigher current application > 25A
 $Comp
@@
 Wire Wire Line
 	8400 6300 8600 6300
+Text GLabel 1350 1150 0    50   Input ~ 0
+DCIN+
+Wire Wire Line
+	1400 1150 1350 1150
+Connection ~ 1400 1150
+Text GLabel 1350 1950 0    50   Input ~ 0
+DCIN-
+Wire Wire Line
+	1400 1950 1350 1950
+Connection ~ 1400 1950
 $EndSCHEMATC
