File: hardware/kajikia/power.sch (KiCad schematic (older format))
At the start: 80 parts, among them J39 Screw_Terminal_01x02, J40 Conn_01x01, J41 Conn_01x01, J42 Conn_01x01, J43 Conn_01x01, J44 Conn_01x01, J45 Conn_01x01, J46 Conn_01x01, J47 Conn_01x01, J48 Conn_01x01, J49 Conn_01x01, J50 Conn_01x01, J51 Conn_01x01, J52 Conn_01x01, J53 Conn_01x01, J54 Conn_01x01, J55 Conn_01x01, J56 Conn_01x01, J57 Conn_01x01, J58 Conn_01x01, J59 Conn_01x01, Q1 AON6144, U2 LM1117-3.3, U3 AOZ1284, U4 AOZ1284

Commit message: fuses
Parts:
- added C191, C78: 220u, Capacitor_SMD:CP_Elec_6.3x7.7, symbol Device:CP1_Small
- F1: value FUSE -> Fuse
- JP14: footprint (none) -> _Generic:Solder Jumper 2P
Connections:
- net +24V: now also J39.2 (Pin_2), C191.1, C78.1; no longer F1.1
- net DCIN-: now also F1.2, C191.2, C78.2; no longer Q1.3 (D)
- removed net DCIN+: F1.2, J39.2 (Pin_2)
- new net: F1.1, Q1.3 (D)
Other:
- moved on the sheet: D1, J39, Q1, R8, R9
Changed lines of the file:
@@
 L power:+24V #PWR017
 U 1 1 5C334E02
-P 2400 1050
-F 0 "#PWR017" H 2400 900 50  0001 C CNN
-F 1 "+24V" H 2415 1223 50  0000 C CNN
-F 2 "" H 2400 1050 50  0001 C CNN
-F 3 "" H 2400 1050 50  0001 C CNN
-	1    2400 1050
-	1    0    0    -1
-$EndComp
-Wire Wire Line
-	1250 1500 1400 1500
-Wire Wire Line
-	1400 1500 1400 1950
-Wire Wire Line
-	1250 1400 1400 1400
-Wire Wire Line
-	1400 1400 1400 1150
+P 2650 1050
+F 0 "#PWR017" H 2650 900 50  0001 C CNN
+F 1 "+24V" H 2665 1223 50  0000 C CNN
+F 2 "" H 2650 1050 50  0001 C CNN
+F 3 "" H 2650 1050 50  0001 C CNN
+	1    2650 1050
+	1    0    0    -1
+$EndComp
+Wire Wire Line
+	1200 1500 1350 1500
+Wire Wire Line
+	1200 1400 1350 1400
 $Comp
 L #Power:GND #PWR018
 U 1 1 5C34B6E8
-P 2400 2050
-F 0 "#PWR018" H 2400 1800 50  0001 C CNN
-F 1 "GND" H 2400 1900 50  0001 C CNN
-F 2 "" H 2400 2050 50  0001 C CNN
-F 3 "" H 2400 2050 50  0001 C CNN
-	1    2400 2050
-	1    0    0    -1
-$EndComp
-Wire Wire Line
-	2400 1950 2400 2050
-Wire Wire Line
-	2400 1050 2400 1150
-Wire Wire Line
-	1400 1150 1500 1150
-$Comp
-L Device:Fuse F1
-U 1 1 5C35C7B9
-P 1650 1150
-F 0 "F1" V 1453 1150 50  0000 C CNN
-F 1 "FUSE" V 1544 1150 50  0000 C CNN
-F 2 "_Generic:SMD_Fuseholder" V 1580 1150 50  0001 C CNN
-F 3 "~" H 1650 1150 50  0001 C CNN
-	1    1650 1150
-	0    1    1    0
-$EndComp
+P 2650 2050
+F 0 "#PWR018" H 2650 1800 50  0001 C CNN
+F 1 "GND" H 2650 1900 50  0001 C CNN
+F 2 "" H 2650 2050 50  0001 C CNN
+F 3 "" H 2650 2050 50  0001 C CNN
+	1    2650 2050
+	1    0    0    -1
+$EndComp
+Wire Wire Line
+	2650 1950 2650 2050
+Wire Wire Line
+	2650 1050 2650 1150
 $Comp
 L power:+12V #PWR034
@@
 F 0 "JP14" H 8300 1363 50  0000 C CNN
 F 1 "SolderJumper_2_Open" H 8300 1250 50  0001 C CNN
-F 2 "" H 8300 1250 50  0001 C CNN
+F 2 "_Generic:Solder Jumper 2P" H 8300 1250 50  0001 C CNN
 F 3 "~" H 8300 1250 50  0001 C CNN
 	1    8300 1250
@@
 Power LED
 Wire Wire Line
-	1400 1950 1450 1950
+	1350 1950 1400 1950
 $Comp
 L Device:Q_NMOS_SGD Q1
 U 1 1 5C3AA6BF
-P 1650 1850
-F 0 "Q1" V 1900 1850 50  0000 C CNN
-F 1 "AON6144" V 1991 1850 50  0000 C CNN
-F 2 "_Generic:DFN5x6-8" H 1850 1950 50  0001 C CNN
-F 3 "~" H 1650 1850 50  0001 C CNN
-	1    1650 1850
+P 1950 1850
+F 0 "Q1" V 2200 1850 50  0000 C CNN
+F 1 "AON6144" V 2291 1850 50  0000 C CNN
+F 2 "_Generic:DFN5x6-8" H 2150 1950 50  0001 C CNN
+F 3 "~" H 1950 1850 50  0001 C CNN
+	1    1950 1850
 	0    -1   1    0
 $EndComp
 Wire Wire Line
-	1850 1950 2000 1950
+	2150 1950 2250 1950
 $Comp
 L Device:R R8
 U 1 1 5C407302
-P 2000 1350
-F 0 "R8" H 2070 1396 50  0000 L CNN
-F 1 "10k" H 2070 1305 50  0000 L CNN
-F 2 "_Generic:0603_RES" V 1930 1350 50  0001 C CNN
-F 3 "~" H 2000 1350 50  0001 C CNN
-	1    2000 1350
+P 2250 1350
+F 0 "R8" H 2320 1396 50  0000 L CNN
+F 1 "10k" H 2320 1305 50  0000 L CNN
+F 2 "_Generic:0603_RES" V 2180 1350 50  0001 C CNN
+F 3 "~" H 2250 1350 50  0001 C CNN
+	1    2250 1350
 	1    0    0    -1
 $EndComp
@@
 L Device:D_Zener D1
 U 1 1 5C407892
-P 2400 1750
-F 0 "D1" V 2354 1829 50  0000 L CNN
-F 1 "16v" V 2445 1829 50  0000 L CNN
-F 2 "_Generic:SOD-523_DIODE" H 2400 1750 50  0001 C CNN
-F 3 "~" H 2400 1750 50  0001 C CNN
-	1    2400 1750
+P 2650 1750
+F 0 "D1" V 2604 1829 50  0000 L CNN
+F 1 "16v" V 2695 1829 50  0000 L CNN
+F 2 "_Generic:SOD-523_DIODE" H 2650 1750 50  0001 C CNN
+F 3 "~" H 2650 1750 50  0001 C CNN
+	1    2650 1750
 	0    1    1    0
 $EndComp
 Wire Wire Line
-	2400 1600 2400 1550
-Wire Wire Line
-	2400 1550 2000 1550
-Wire Wire Line
-	1650 1550 1650 1650
-Wire Wire Line
-	2000 1550 2000 1500
-Wire Wire Line
-	2400 1900 2400 1950
-Connection ~ 2400 1950
+	2650 1600 2650 1550
+Wire Wire Line
+	2650 1550 2250 1550
+Wire Wire Line
+	1950 1550 1950 1650
+Wire Wire Line
+	2250 1550 2250 1500
+Wire Wire Line
+	2650 1900 2650 1950
+Connection ~ 2650 1950
 $Comp
 L Device:R R9
 U 1 1 5C479547
-P 2000 1750
-F 0 "R9" H 2070 1796 50  0000 L CNN
-F 1 "100k" H 2070 1705 50  0000 L CNN
-F 2 "_Generic:0603_RES" V 1930 1750 50  0001 C CNN
-F 3 "~" H 2000 1750 50  0001 C CNN
-	1    2000 1750
-	1    0    0    -1
-$EndComp
-Wire Wire Line
-	2000 1900 2000 1950
-Connection ~ 2000 1950
-Wire Wire Line
-	2000 1950 2100 1950
-Wire Wire Line
-	2000 1600 2000 1550
-Connection ~ 2000 1550
-Wire Wire Line
-	2000 1550 1650 1550
+P 2250 1750
+F 0 "R9" H 2320 1796 50  0000 L CNN
+F 1 "100k" H 2320 1705 50  0000 L CNN
+F 2 "_Generic:0603_RES" V 2180 1750 50  0001 C CNN
+F 3 "~" H 2250 1750 50  0001 C CNN
+	1    2250 1750
+	1    0    0    -1
+$EndComp
+Wire Wire Line
+	2250 1900 2250 1950
+Connection ~ 2250 1950
+Wire Wire Line
+	2250 1600 2250 1550
+Connection ~ 2250 1550
+Wire Wire Line
+	2250 1550 1950 1550
 Text Notes 700  2200 0    25   ~ 0
 Replace with DMT40M9LPS for\nhigher current application > 25A
@@
 L power:PWR_FLAG #FLG07
 U 1 1 5C5382D5
-P 2100 2000
-F 0 "#FLG07" H 2100 2075 50  0001 C CNN
-F 1 "PWR_FLAG" H 2100 2173 50  0000 C CNN
-F 2 "" H 2100 2000 50  0001 C CNN
-F 3 "~" H 2100 2000 50  0001 C CNN
-	1    2100 2000
+P 2400 2000
+F 0 "#FLG07" H 2400 2075 50  0001 C CNN
+F 1 "PWR_FLAG" H 2400 2173 50  0000 C CNN
+F 2 "" H 2400 2000 50  0001 C CNN
+F 3 "~" H 2400 2000 50  0001 C CNN
+	1    2400 2000
 	-1   0    0    1
 $EndComp
 Wire Wire Line
-	2100 2000 2100 1950
-Connection ~ 2100 1950
-Wire Wire Line
-	2100 1950 2400 1950
+	2400 2000 2400 1950
 $Comp
 L power:PWR_FLAG #FLG06
 U 1 1 5C5499F4
-P 2100 1100
-F 0 "#FLG06" H 2100 1175 50  0001 C CNN
-F 1 "PWR_FLAG" H 2100 1274 50  0000 C CNN
-F 2 "" H 2100 1100 50  0001 C CNN
-F 3 "~" H 2100 1100 50  0001 C CNN
-	1    2100 1100
-	1    0    0    -1
-$EndComp
-Wire Wire Line
-	2100 1100 2100 1150
-Connection ~ 2100 1150
-Wire Wire Line
-	2100 1150 2400 1150
-Wire Wire Line
-	2000 1200 2000 1150
-Connection ~ 2000 1150
-Wire Wire Line
-	2000 1150 2100 1150
-Wire Wire Line
-	1800 1150 2000 1150
+P 2400 1100
+F 0 "#FLG06" H 2400 1175 50  0001 C CNN
+F 1 "PWR_FLAG" H 2400 1274 50  0000 C CNN
+F 2 "" H 2400 1100 50  0001 C CNN
+F 3 "~" H 2400 1100 50  0001 C CNN
+	1    2400 1100
+	1    0    0    -1
+$EndComp
+Wire Wire Line
+	2400 1100 2400 1150
+Wire Wire Line
+	2250 1200 2250 1150
+Connection ~ 2250 1150
 $Comp
 L Connector:Screw_Terminal_01x02 J39
 U 1 1 5C365574
-P 1050 1500
-F 0 "J39" H 970 1267 50  0000 C CNN
-F 1 "Screw_Terminal_01x02" H 970 1266 50  0001 C CNN
-F 2 "_Generic:KF635-2P" H 1050 1500 50  0001 C CNN
-F 3 "~" H 1050 1500 50  0001 C CNN
-	1    1050 1500
+P 1000 1500
+F 0 "J39" H 920 1267 50  0000 C CNN
+F 1 "Screw_Terminal_01x02" H 920 1266 50  0001 C CNN
+F 2 "_Generic:KF635-2P" H 1000 1500 50  0001 C CNN
+F 3 "~" H 1000 1500 50  0001 C CNN
+	1    1000 1500
 	-1   0    0    1
 $EndComp
@@
 Wire Wire Line
 	8400 6300 8600 6300
-Text GLabel 1350 1150 0    50   Input ~ 0
-DCIN+
-Wire Wire Line
-	1400 1150 1350 1150
-Connection ~ 1400 1150
-Text GLabel 1350 1950 0    50   Input ~ 0
+Text GLabel 1300 1950 0    50   Input ~ 0
 DCIN-
 Wire Wire Line
-	1400 1950 1350 1950
-Connection ~ 1400 1950
+	1350 1950 1300 1950
+Connection ~ 1350 1950
+Wire Wire Line
+	1350 1150 1500 1150
+$Comp
+L Device:Fuse F1
+U 1 1 5C420B0B
+P 1550 1950
+F 0 "F1" V 1353 1950 50  0000 C CNN
+F 1 "Fuse" V 1444 1950 50  0000 C CNN
+F 2 "_Generic:SMD_Fuseholder" V 1480 1950 50  0001 C CNN
+F 3 "~" H 1550 1950 50  0001 C CNN
+	1    1550 1950
+	0    1    1    0
+$EndComp
+Wire Wire Line
+	1700 1950 1750 1950
+Connection ~ 2400 1950
+Wire Wire Line
+	2400 1950 2650 1950
+Wire Wire Line
+	2250 1950 2400 1950
+Connection ~ 2400 1150
+Wire Wire Line
+	2400 1150 2650 1150
+Wire Wire Line
+	2250 1150 2400 1150
+$Comp
+L Device:CP1_Small C78
+U 1 1 5C8D0CF9
+P 1500 1300
+F 0 "C78" H 1591 1346 50  0000 L CNN
+F 1 "220u" H 1591 1255 50  0000 L CNN
+F 2 "Capacitor_SMD:CP_Elec_6.3x7.7" H 1500 1300 50  0001 C CNN
+F 3 "~" H 1500 1300 50  0001 C CNN
+	1    1500 1300
+	1    0    0    -1
+$EndComp
+Wire Wire Line
+	1500 1400 1500 1500
+Wire Wire Line
+	1500 1500 1350 1500
+Connection ~ 1350 1500
+Wire Wire Line
+	1350 1500 1350 1950
+$Comp
+L Device:CP1_Small C191
+U 1 1 5C910F5C
+P 1850 1300
+F 0 "C191" H 1941 1346 50  0000 L CNN
+F 1 "220u" H 1941 1255 50  0000 L CNN
+F 2 "Capacitor_SMD:CP_Elec_6.3x7.7" H 1850 1300 50  0001 C CNN
+F 3 "~" H 1850 1300 50  0001 C CNN
+	1    1850 1300
+	1    0    0    -1
+$EndComp
+Wire Wire Line
+	1850 1400 1850 1500
+Wire Wire Line
+	1500 1500 1850 1500
+Connection ~ 1500 1500
+Wire Wire Line
+	1350 1150 1350 1400
+Wire Wire Line
+	1500 1150 1500 1200
+Connection ~ 1500 1150
+Wire Wire Line
+	1500 1150 1850 1150
+Wire Wire Line
+	1850 1150 1850 1200
+Connection ~ 1850 1150
+Wire Wire Line
+	1850 1150 2250 1150
 $EndSCHEMATC

Commit message: continue routing
Parts:
- removed J46, J47, J49, J50, J52, J53: Conn_01x01, _Generic:PinHeader_2.54mm_1P, symbol #Connector:Conn_01x01
- added C193: 220u, Capacitor_SMD:CP_Elec_6.3x7.7, symbol Device:CP1_Small
- added C194, C195, C196, C197, C198, C199: 4.7u, _Generic:1210_CAP, symbol Device:C_Small
- C23, C24, C25, C26, C27, C28, C31, C32: footprint _Generic:0805_CAP -> _Generic:1210_CAP
- C41, C42: value 10u -> 4.7u; footprint _Generic:0603_CAP -> _Generic:1210_CAP
- C43, C44: value 390u -> 220u; footprint Capacitor_SMD:CP_Elec_8x10 -> Capacitor_SMD:CP_Elec_6.3x7.7
Connections:
- net +12V: now also C194.1, C196.1, C198.1
- net +24V: now also C193.1
- net +5V: now also C195.1, C197.1, C199.1
- net GND: now also C193.2, C194.2, C195.2, C196.2, C197.2, C198.2, C199.2
Other:
- moved on the sheet: C23, C25, C27, C29, C31, C33, C35, C37, C39, C41, D2, D5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

Commit message: continue routing
Parts:
- removed C19: 68u, Capacitor_SMD:CP_Elec_8x10, symbol Device:CP1_Small
- removed C198, C199, C26, C31: 4.7u, _Generic:1210_CAP, symbol Device:C_Small
Other:
- moved on the sheet: C23, C24, C25, C27
Changed lines of the file:
@@
 	1    0    0    -1
 $EndComp
-$Comp
-L Device:C_Small C31
-U 1 1 5E9998E5
+Wire Wire Line
+	5100 2100 5100 2050
+Wire Wire Line
+	5100 2050 5350 2050
+Wire Wire Line
+	4750 2350 4750 2400
+Wire Wire Line
+	4750 2400 5100 2400
+Wire Wire Line
+	5850 2400 5850 2350
+Wire Wire Line
+	5100 2300 5100 2400
+Connection ~ 5100 2400
+Wire Wire Line
+	5100 2400 5850 2400
+Connection ~ 4750 2400
+$Comp
+L Device:C_Small C27
+U 1 1 5E999D70
 P 4550 1250
-F 0 "C31" H 4642 1296 50  0000 L CNN
+F 0 "C27" H 4642 1296 50  0000 L CNN
 F 1 "4.7u" H 4642 1205 50  0000 L CNN
 F 2 "_Generic:1210_CAP" H 4550 1250 50  0001 C CNN
@@
 	1    0    0    -1
 $EndComp
-Wire Wire Line
-	5100 2100 5100 2050
-Wire Wire Line
-	5100 2050 5350 2050
-Wire Wire Line
-	4750 2350 4750 2400
-Wire Wire Line
-	4750 2400 5100 2400
-Wire Wire Line
-	5850 2400 5850 2350
-Wire Wire Line
-	5100 2300 5100 2400
-Connection ~ 5100 2400
-Wire Wire Line
-	5100 2400 5850 2400
-Connection ~ 4750 2400
-$Comp
-L Device:C_Small C27
-U 1 1 5E999D70
+$Comp
+L Device:C_Small C25
+U 1 1 5E999DED
 P 4150 1250
-F 0 "C27" H 4242 1296 50  0000 L CNN
+F 0 "C25" H 4242 1296 50  0000 L CNN
 F 1 "4.7u" H 4242 1205 50  0000 L CNN
 F 2 "_Generic:1210_CAP" H 4150 1250 50  0001 C CNN
@@
 	1    0    0    -1
 $EndComp
-$Comp
-L Device:C_Small C25
-U 1 1 5E999DED
-P 3750 1250
-F 0 "C25" H 3842 1296 50  0000 L CNN
-F 1 "4.7u" H 3842 1205 50  0000 L CNN
-F 2 "_Generic:1210_CAP" H 3750 1250 50  0001 C CNN
-F 3 "~" H 3750 1250 50  0001 C CNN
-	1    3750 1250
-	1    0    0    -1
-$EndComp
-Wire Wire Line
-	3750 1050 3750 1150
-Wire Wire Line
-	4150 1150 4150 1050
+Wire Wire Line
+	4150 1050 4150 1150
 Wire Wire Line
 	4550 1150 4550 1050
-Connection ~ 4550 1050
-Wire Wire Line
-	3750 1350 3750 1450
+Wire Wire Line
+	4150 1350 4150 1450
 Wire Wire Line
 	4550 1350 4550 1450
-Wire Wire Line
-	4550 1450 4150 1450
-Wire Wire Line
-	4150 1350 4150 1450
-Connection ~ 4150 1450
 $Comp
 L Device:C_Small C37
@@
 Wire Wire Line
 	4350 1650 5050 1650
-Connection ~ 4150 1050
-Wire Wire Line
-	4150 1050 4550 1050
+Connection ~ 4550 1050
 Wire Wire Line
 	6600 2150 7400 2150
@@
 Wire Wire Line
 	5850 1050 5850 1350
-Wire Wire Line
-	4550 1050 5050 1050
 Connection ~ 5050 1050
 $Comp
 L Device:C_Small C23
 U 1 1 5C49B960
-P 3350 1250
-F 0 "C23" H 3442 1296 50  0000 L CNN
-F 1 "4.7u" H 3442 1205 50  0000 L CNN
-F 2 "_Generic:1210_CAP" H 3350 1250 50  0001 C CNN
-F 3 "~" H 3350 1250 50  0001 C CNN
-	1    3350 1250
-	1    0    0    -1
-$EndComp
-Wire Wire Line
-	3350 1050 3350 1150
-Wire Wire Line
-	3350 1350 3350 1450
+P 3750 1250
+F 0 "C23" H 3842 1296 50  0000 L CNN
+F 1 "4.7u" H 3842 1205 50  0000 L CNN
+F 2 "_Generic:1210_CAP" H 3750 1250 50  0001 C CNN
+F 3 "~" H 3750 1250 50  0001 C CNN
+	1    3750 1250
+	1    0    0    -1
+$EndComp
+Wire Wire Line
+	3750 1050 3750 1150
+Wire Wire Line
+	3750 1350 3750 1450
 $Comp
 L #Power:GND #PWR021
 U 1 1 5C4A3EED
-P 3350 1500
-F 0 "#PWR021" H 3350 1250 50  0001 C CNN
-F 1 "GND" H 3350 1350 50  0001 C CNN
-F 2 "" H 3350 1500 50  0001 C CNN
-F 3 "" H 3350 1500 50  0001 C CNN
-	1    3350 1500
-	1    0    0    -1
-$EndComp
-Wire Wire Line
-	3350 1500 3350 1450
-Connection ~ 3350 1450
-Wire Wire Line
-	3350 1450 3750 1450
-Wire Wire Line
-	3350 1050 3750 1050
-Connection ~ 3750 1050
+P 3750 1500
+F 0 "#PWR021" H 3750 1250 50  0001 C CNN
+F 1 "GND" H 3750 1350 50  0001 C CNN
+F 2 "" H 3750 1500 50  0001 C CNN
+F 3 "" H 3750 1500 50  0001 C CNN
+	1    3750 1500
+	1    0    0    -1
+$EndComp
+Wire Wire Line
+	3750 1500 3750 1450
+Connection ~ 3750 1450
+Wire Wire Line
+	3750 1450 4150 1450
 Wire Wire Line
 	3750 1050 4150 1050
-Connection ~ 3750 1450
-Wire Wire Line
-	3750 1450 4150 1450
+Connection ~ 4150 1050
+Wire Wire Line
+	4150 1050 4550 1050
+Connection ~ 4150 1450
+Wire Wire Line
+	4150 1450 4550 1450
 $Comp
 L #Regulator:AOZ1284 U4
@@
 Connection ~ 5050 5050
 Wire Wire Line
-	4050 3700 4050 3800
-Wire Wire Line
 	4450 3800 4450 3700
 Wire Wire Line
 	4850 3800 4850 3700
 Connection ~ 4850 3700
-Wire Wire Line
-	4050 4000 4050 4100
 Wire Wire Line
 	4850 4000 4850 4100
@@
 Connection ~ 5350 3700
 Wire Wire Line
-	3650 3700 3650 3800
-Wire Wire Line
-	3650 4000 3650 4100
+	4050 3700 4050 3800
+Wire Wire Line
+	4050 4000 4050 4100
 $Comp
 L #Power:GND #PWR022
 U 1 1 5C4EC56F
-P 3650 4150
-F 0 "#PWR022" H 3650 3900 50  0001 C CNN
-F 1 "GND" H 3650 4000 50  0001 C CNN
-F 2 "" H 3650 4150 50  0001 C CNN
-F 3 "" H 3650 4150 50  0001 C CNN
-	1    3650 4150
-	1    0    0    -1
-$EndComp
-Wire Wire Line
-	3650 4150 3650 4100
-Connection ~ 3650 4100
-Wire Wire Line
-	3650 4100 4050 4100
-Wire Wire Line
-	3650 3700 4050 3700
-Connection ~ 4050 3700
-Wire Wire Line
-	4050 3700 4450 3700
+P 4050 4150
+F 0 "#PWR022" H 4050 3900 50  0001 C CNN
+F 1 "GND" H 4050 4000 50  0001 C CNN
+F 2 "" H 4050 4150 50  0001 C CNN
+F 3 "" H 4050 4150 50  0001 C CNN
+	1    4050 4150
+	1    0    0    -1
+$EndComp
+Wire Wire Line
+	4050 4150 4050 4100
 Connection ~ 4050 4100
-Wire Wire Line
-	4050 4100 4450 4100
 Wire Wire Line
 	8100 3750 8100 3900
@@
 $EndComp
 $Comp
-L Device:CP1_Small C19
-U 1 1 5C573F79
-P 1700 4150
-F 0 "C19" H 1791 4196 50  0000 L CNN
-F 1 "68u" H 1791 4105 50  0000 L CNN
-F 2 "Capacitor_SMD:CP_Elec_8x10" H 1700 4150 50  0001 C CNN
-F 3 "~" H 1700 4150 50  0001 C CNN
-	1    1700 4150
-	1    0    0    -1
-$EndComp
-$Comp
 L power:+24V #PWR015
 U 1 1 5C574053
-P 1700 3950
-F 0 "#PWR015" H 1700 3800 50  0001 C CNN
-F 1 "+24V" H 1715 4123 50  0000 C CNN
-F 2 "" H 1700 3950 50  0001 C CNN
-F 3 "" H 1700 3950 50  0001 C CNN
-	1    1700 3950
+P 2100 3900
+F 0 "#PWR015" H 2100 3750 50  0001 C CNN
+F 1 "+24V" H 2115 4073 50  0000 C CNN
+F 2 "" H 2100 3900 50  0001 C CNN
+F 3 "" H 2100 3900 50  0001 C CNN
+	1    2100 3900
 	1    0    0    -1
 $EndComp
@@
 L #Power:GND #PWR016
 U 1 1 5C574142
-P 1700 4350
-F 0 "#PWR016" H 1700 4100 50  0001 C CNN
-F 1 "GND" H 1700 4200 50  0001 C CNN
-F 2 "" H 1700 4350 50  0001 C CNN
-F 3 "" H 1700 4350 50  0001 C CNN
-	1    1700 4350
-	1    0    0    -1
-$EndComp
-Wire Wire Line
-	1700 4350 1700 4300
-Wire Wire Line
-	1700 4050 1700 4000
+P 2100 4350
+F 0 "#PWR016" H 2100 4100 50  0001 C CNN
+F 1 "GND" H 2100 4200 50  0001 C CNN
+F 2 "" H 2100 4350 50  0001 C CNN
+F 3 "" H 2100 4350 50  0001 C CNN
+	1    2100 4350
+	1    0    0    -1
+$EndComp
 $Comp
 L Regulator_Linear:LM1117-3.3 U2
@@
 	1    0    0    -1
 $EndComp
-Wire Wire Line
-	1700 4300 2100 4300
-Wire Wire Line
-	2100 4300 2100 4250
-Connection ~ 1700 4300
-Wire Wire Line
-	1700 4300 1700 4250
-Wire Wire Line
-	2100 4050 2100 4000
-Wire Wire Line
-	2100 4000 1700 4000
-Connection ~ 1700 4000
-Wire Wire Line
-	1700 4000 1700 3950
 $Comp
 L Device:CP1_Small C43
@@
 $EndComp
 $Comp
-L Device:C_Small C26
-U 1 1 5C5FFB0B
+L Device:C_Small C24
+U 1 1 5C5FFB11
 P 4050 3900
-F 0 "C26" H 4142 3946 50  0000 L CNN
+F 0 "C24" H 4142 3946 50  0000 L CNN
 F 1 "4.7u" H 4142 3855 50  0000 L CNN
 F 2 "_Generic:1210_CAP" H 4050 3900 50  0001 C CNN
 F 3 "~" H 4050 3900 50  0001 C CNN
 	1    4050 3900
-	1    0    0    -1
-$EndComp
-$Comp
-L Device:C_Small C24
-U 1 1 5C5FFB11
-P 3650 3900
-F 0 "C24" H 3742 3946 50  0000 L CNN
-F 1 "4.7u" H 3742 3855 50  0000 L CNN
-F 2 "_Generic:1210_CAP" H 3650 3900 50  0001 C CNN
-F 3 "~" H 3650 3900 50  0001 C CNN
-	1    3650 3900
 	1    0    0    -1
 $EndComp
@@
 	1    0    0    -1
 $EndComp
-$Comp
-L Device:C_Small C198
-U 1 1 5C6AA1C9
-P 8250 1450
-F 0 "C198" H 8342 1496 50  0000 L CNN
-F 1 "4.7u" H 8342 1405 50  0000 L CNN
-F 2 "_Generic:1210_CAP" H 8250 1450 50  0001 C CNN
-F 3 "~" H 8250 1450 50  0001 C CNN
-	1    8250 1450
-	1    0    0    -1
-$EndComp
-Wire Wire Line
-	7800 1250 8250 1250
-Wire Wire Line
-	8250 1250 8250 1350
-Connection ~ 8250 1250
-Wire Wire Line
-	8250 1250 8650 1250
-Wire Wire Line
-	8250 1550 8250 1650
-Wire Wire Line
-	8250 1650 8650 1650
-Connection ~ 8650 1650
-$Comp
-L Device:C_Small C199
-U 1 1 5C70C82E
-P 8550 4100
-F 0 "C199" H 8642 4146 50  0000 L CNN
-F 1 "4.7u" H 8642 4055 50  0000 L CNN
-F 2 "_Generic:1210_CAP" H 8550 4100 50  0001 C CNN
-F 3 "~" H 8550 4100 50  0001 C CNN
-	1    8550 4100
-	1    0    0    -1
-$EndComp
-Wire Wire Line
-	8100 3900 8550 3900
-Wire Wire Line
-	8550 3900 8550 4000
-Connection ~ 8550 3900
-Wire Wire Line
-	8550 3900 8950 3900
-Wire Wire Line
-	8550 4200 8550 4300
-Wire Wire Line
-	8550 4300 8950 4300
-Connection ~ 8950 4300
 Wire Wire Line
 	10300 4250 10300 4650
+Wire Wire Line
+	2100 4250 2100 4350
+Wire Wire Line
+	2100 3900 2100 4050
+Wire Wire Line
+	4550 1050 5050 1050
+Wire Wire Line
+	7800 1250 8650 1250
+Wire Wire Line
+	4050 4100 4450 4100
+Wire Wire Line
+	4050 3700 4450 3700
+Wire Wire Line
+	8100 3900 8950 3900
 $EndSCHEMATC

Commit message: continue routing
Parts:
- added J100, J101, J102, J103, J49, J50, J53, J68, J69, J70, J94, J95, J96, J97, J98, J99: Conn_01x01, _Generic:PinHeader_2.54mm_1P, symbol #Connector:Conn_01x01
Connections:
- net +3V3: now also J100.1 (Pin_1), J101.1 (Pin_1), J102.1 (Pin_1), J103.1 (Pin_1), J94.1 (Pin_1), J95.1 (Pin_1)
- net GND: now also J49.1 (Pin_1), J50.1 (Pin_1), J53.1 (Pin_1), J68.1 (Pin_1), J69.1 (Pin_1), J70.1 (Pin_1), J96.1 (Pin_1), J97.1 (Pin_1), J98.1 (Pin_1), J99.1 (Pin_1)
