File: hardware/kajikia/power.sch (KiCad schematic (older format))
At the start: 90 parts, among them J100 Conn_01x01, J101 Conn_01x01, J102 Conn_01x01, J39 Screw_Terminal_01x02, J44 Conn_01x01, J45 Conn_01x01, J48 Conn_01x01, J49 Conn_01x01, J50 Conn_01x01, J51 Conn_01x01, J53 Conn_01x01, J54 Conn_01x01, J55 Conn_01x01, J56 Conn_01x01, J57 Conn_01x01, J58 Conn_01x01, J59 Conn_01x01, J68 Conn_01x01, J69 Conn_01x01, J70 Conn_01x01, J94 Conn_01x01, J95 Conn_01x01, J96 Conn_01x01, J98 Conn_01x01, J99 Conn_01x01, Q1 AON6144, U2 LM1117-3.3, U3 AOZ1284, U4 AOZ1284

Commit message: PCB V1
Parts:
- H5, H6: renamed from H?; footprint (none) -> MountingHole:MountingHole_2.2mm_M2_DIN965
Other:
- note added: "Mounting Holes"
- note removed: "Common Decoupling"
- note removed: "Replace with DMT40M9LPS for\nhigher current application > 25A"
- moved on the sheet: C191, C193, C194, C196, C23, C25, C27, C29, C33, C35, C37, C39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
