File: hardware/kajikia/driver.sch (KiCad schematic (older format))
At the start: 9 parts, among them J68 Conn_01x04, J69 Conn_01x04, J70 Conn_01x04, J71 Conn_01x04, J72 Conn_01x04, X1 12MHz

Commit message: layout test
Parts:
- J89: renamed from J68; footprint (none) -> _Generic:JST_XH_4P
- J90: renamed from J69; footprint (none) -> _Generic:JST_XH_4P
- J91: renamed from J70; footprint (none) -> _Generic:JST_XH_4P
- J92: renamed from J71; footprint (none) -> _Generic:JST_XH_4P
- J93: renamed from J72; footprint (none) -> _Generic:JST_XH_4P
- renumbered C53 to C80, R66 to R79, R67 to R80
Connections:
- net Driver1/OA1: now also J89.2 (Pin_2); no longer J89.1 (Pin_1)
- net Driver1/OA2: now also J89.1 (Pin_1); no longer J89.2 (Pin_2)
- net Driver1/OB1: now also J89.4 (Pin_4); no longer J89.3 (Pin_3)
- net Driver1/OB2: now also J89.3 (Pin_3); no longer J89.4 (Pin_4)
- net Driver2/OA1: now also J91.2 (Pin_2); no longer J91.1 (Pin_1)
- net Driver2/OA2: now also J91.1 (Pin_1); no longer J91.2 (Pin_2)
- net Driver2/OB1: now also J91.4 (Pin_4); no longer J91.3 (Pin_3)
- net Driver2/OB2: now also J91.3 (Pin_3); no longer J91.4 (Pin_4)
- net Driver3/OA1: now also J93.2 (Pin_2); no longer J93.1 (Pin_1)
- net Driver3/OA2: now also J93.1 (Pin_1); no longer J93.2 (Pin_2)
- net Driver3/OB1: now also J93.4 (Pin_4); no longer J93.3 (Pin_3)
- net Driver3/OB2: now also J93.3 (Pin_3); no longer J93.4 (Pin_4)
- net Driver4/OA1: now also J90.2 (Pin_2); no longer J90.1 (Pin_1)
- net Driver4/OA2: now also J90.1 (Pin_1); no longer J90.2 (Pin_2)
- net Driver4/OB1: now also J90.4 (Pin_4); no longer J90.3 (Pin_3)
- net Driver4/OB2: now also J90.3 (Pin_3); no longer J90.4 (Pin_4)
- net Driver5/OA1: now also J92.2 (Pin_2); no longer J92.1 (Pin_1)
- net Driver5/OA2: now also J92.1 (Pin_1); no longer J92.2 (Pin_2)
- net Driver5/OB1: now also J92.4 (Pin_4); no longer J92.3 (Pin_3)
- net Driver5/OB2: now also J92.3 (Pin_3); no longer J92.4 (Pin_4)
Changed lines of the file:
@@
 F10 "DIAG0" O L 4150 3000 50
 F11 "DIAG1" O L 4150 3100 50
-F12 "OA1" O R 4850 2050 50
-F13 "OA2" O R 4850 2150 50
-F14 "OB1" O R 4850 2250 50
-F15 "OB2" O R 4850 2350 50
+F12 "OA1" O R 4850 2250 50
+F13 "OA2" O R 4850 2350 50
+F14 "OB1" O R 4850 2050 50
+F15 "OB2" O R 4850 2150 50
 $EndSheet
 Wire Wire Line
@@
 L Connector_Generic:Conn_01x04 J?
 U 1 1 60EA0743
-P 5100 2150
+P 5100 2250
 AR Path="/5AF7E834/60C2EDFB/60EA0743" Ref="J?"  Part="1"
 AR Path="/5B406A82/60EA0743" Ref="J?"  Part="1"
-AR Path="/60C2EDFB/60EA0743" Ref="J68"  Part="1"
-F 0 "J68" H 5180 2142 50  0000 L CNN
-F 1 "Conn_01x04" H 5180 2051 50  0001 L CNN
-F 2 "" H 5100 2150 50  0001 C CNN
-F 3 "~" H 5100 2150 50  0001 C CNN
-	1    5100 2150
-	1    0    0    -1
-$EndComp
-Wire Wire Line
-	4850 2050 4900 2050
-Wire Wire Line
-	4850 2150 4900 2150
-Wire Wire Line
-	4850 2250 4900 2250
-Wire Wire Line
-	4850 2350 4900 2350
+AR Path="/60C2EDFB/60EA0743" Ref="J89"  Part="1"
+F 0 "J89" H 5180 2242 50  0000 L CNN
+F 1 "Conn_01x04" H 5180 2151 50  0001 L CNN
+F 2 "_Generic:JST_XH_4P" H 5100 2250 50  0001 C CNN
+F 3 "~" H 5100 2250 50  0001 C CNN
+	1    5100 2250
+	1    0    0    1
+$EndComp
 $Sheet
 S 6650 1950 700  1250
@@
 F10 "DIAG0" O L 6650 3000 50
 F11 "DIAG1" O L 6650 3100 50
-F12 "OA1" O R 7350 2050 50
-F13 "OA2" O R 7350 2150 50
-F14 "OB1" O R 7350 2250 50
-F15 "OB2" O R 7350 2350 50
+F12 "OA1" O R 7350 2250 50
+F13 "OA2" O R 7350 2350 50
+F14 "OB1" O R 7350 2050 50
+F15 "OB2" O R 7350 2150 50
 $EndSheet
 Wire Wire Line
@@
 L Connector_Generic:Conn_01x04 J?
 U 1 1 60ECA914
-P 7600 2150
+P 7600 2250
 AR Path="/5AF7E834/60C2EDFB/60ECA914" Ref="J?"  Part="1"
 AR Path="/5B406A82/60ECA914" Ref="J?"  Part="1"
-AR Path="/60C2EDFB/60ECA914" Ref="J70"  Part="1"
-F 0 "J70" H 7680 2142 50  0000 L CNN
-F 1 "Conn_01x04" H 7680 2051 50  0001 L CNN
-F 2 "" H 7600 2150 50  0001 C CNN
-F 3 "~" H 7600 2150 50  0001 C CNN
-	1    7600 2150
-	1    0    0    -1
+AR Path="/60C2EDFB/60ECA914" Ref="J91"  Part="1"
+F 0 "J91" H 7680 2242 50  0000 L CNN
+F 1 "Conn_01x04" H 7680 2151 50  0001 L CNN
+F 2 "_Generic:JST_XH_4P" H 7600 2250 50  0001 C CNN
+F 3 "~" H 7600 2250 50  0001 C CNN
+	1    7600 2250
+	1    0    0    1
 $EndComp
 Wire Wire Line
@@
 F10 "DIAG0" O L 9150 3000 50
 F11 "DIAG1" O L 9150 3100 50
-F12 "OA1" O R 9850 2050 50
-F13 "OA2" O R 9850 2150 50
-F14 "OB1" O R 9850 2250 50
-F15 "OB2" O R 9850 2350 50
+F12 "OA1" O R 9850 2250 50
+F13 "OA2" O R 9850 2350 50
+F14 "OB1" O R 9850 2050 50
+F15 "OB2" O R 9850 2150 50
 $EndSheet
 Wire Wire Line
@@
 L Connector_Generic:Conn_01x04 J?
 U 1 1 60ECD6EE
-P 10100 2150
+P 10100 2250
 AR Path="/5AF7E834/60C2EDFB/60ECD6EE" Ref="J?"  Part="1"
 AR Path="/5B406A82/60ECD6EE" Ref="J?"  Part="1"
-AR Path="/60C2EDFB/60ECD6EE" Ref="J72"  Part="1"
-F 0 "J72" H 10180 2142 50  0000 L CNN
-F 1 "Conn_01x04" H 10180 2051 50  0001 L CNN
-F 2 "" H 10100 2150 50  0001 C CNN
-F 3 "~" H 10100 2150 50  0001 C CNN
-	1    10100 2150
-	1    0    0    -1
+AR Path="/60C2EDFB/60ECD6EE" Ref="J93"  Part="1"
+F 0 "J93" H 10180 2242 50  0000 L CNN
+F 1 "Conn_01x04" H 10180 2151 50  0001 L CNN
+F 2 "_Generic:JST_XH_4P" H 10100 2250 50  0001 C CNN
+F 3 "~" H 10100 2250 50  0001 C CNN
+	1    10100 2250
+	1    0    0    1
 $EndComp
 Wire Wire Line
@@
 F10 "DIAG0" O L 4150 5700 50
 F11 "DIAG1" O L 4150 5800 50
-F12 "OA1" O R 4850 4750 50
-F13 "OA2" O R 4850 4850 50
-F14 "OB1" O R 4850 4950 50
-F15 "OB2" O R 4850 5050 50
+F12 "OA1" O R 4850 4950 50
+F13 "OA2" O R 4850 5050 50
+F14 "OB1" O R 4850 4750 50
+F15 "OB2" O R 4850 4850 50
 $EndSheet
 Wire Wire Line
@@
 L Connector_Generic:Conn_01x04 J?
 U 1 1 60ED5884
-P 5100 4850
+P 5100 4950
 AR Path="/5AF7E834/60C2EDFB/60ED5884" Ref="J?"  Part="1"
 AR Path="/5B406A82/60ED5884" Ref="J?"  Part="1"
-AR Path="/60C2EDFB/60ED5884" Ref="J69"  Part="1"
-F 0 "J69" H 5180 4842 50  0000 L CNN
-F 1 "Conn_01x04" H 5180 4751 50  0001 L CNN
-F 2 "" H 5100 4850 50  0001 C CNN
-F 3 "~" H 5100 4850 50  0001 C CNN
-	1    5100 4850
-	1    0    0    -1
+AR Path="/60C2EDFB/60ED5884" Ref="J90"  Part="1"
+F 0 "J90" H 5180 4942 50  0000 L CNN
+F 1 "Conn_01x04" H 5180 4851 50  0001 L CNN
+F 2 "_Generic:JST_XH_4P" H 5100 4950 50  0001 C CNN
+F 3 "~" H 5100 4950 50  0001 C CNN
+	1    5100 4950
+	1    0    0    1
 $EndComp
 Wire Wire Line
@@
 F10 "DIAG0" O L 6650 5700 50
 F11 "DIAG1" O L 6650 5800 50
-F12 "OA1" O R 7350 4750 50
-F13 "OA2" O R 7350 4850 50
-F14 "OB1" O R 7350 4950 50
-F15 "OB2" O R 7350 5050 50
+F12 "OA1" O R 7350 4950 50
+F13 "OA2" O R 7350 5050 50
+F14 "OB1" O R 7350 4750 50
+F15 "OB2" O R 7350 4850 50
 $EndSheet
 Wire Wire Line
@@
 L Connector_Generic:Conn_01x04 J?
 U 1 1 60ED8656
-P 7600 4850
+P 7600 4950
 AR Path="/5AF7E834/60C2EDFB/60ED8656" Ref="J?"  Part="1"
 AR Path="/5B406A82/60ED8656" Ref="J?"  Part="1"
-AR Path="/60C2EDFB/60ED8656" Ref="J71"  Part="1"
-F 0 "J71" H 7680 4842 50  0000 L CNN
-F 1 "Conn_01x04" H 7680 4751 50  0001 L CNN
-F 2 "" H 7600 4850 50  0001 C CNN
-F 3 "~" H 7600 4850 50  0001 C CNN
-	1    7600 4850
-	1    0    0    -1
+AR Path="/60C2EDFB/60ED8656" Ref="J92"  Part="1"
+F 0 "J92" H 7680 4942 50  0000 L CNN
+F 1 "Conn_01x04" H 7680 4851 50  0001 L CNN
+F 2 "_Generic:JST_XH_4P" H 7600 4950 50  0001 C CNN
+F 3 "~" H 7600 4950 50  0001 C CNN
+	1    7600 4950
+	1    0    0    1
 $EndComp
 Wire Wire Line
@@
 AR Path="/5AF7E834/60C2EDFB/60EF0E90" Ref="#PWR?"  Part="1"
 AR Path="/5B406A82/60EF0E90" Ref="#PWR?"  Part="1"
-AR Path="/60C2EDFB/60EF0E90" Ref="#PWR094"  Part="1"
-F 0 "#PWR094" H 2650 4750 50  0001 C CNN
+AR Path="/60C2EDFB/60EF0E90" Ref="#PWR0125"  Part="1"
+F 0 "#PWR0125" H 2650 4750 50  0001 C CNN
 F 1 "+3.3V" H 2665 5073 50  0000 C CNN
 F 2 "" H 2650 4900 50  0001 C CNN
@@
 AR Path="/5AF7E834/60C2EDFB/60EF0ED6" Ref="R?"  Part="1"
 AR Path="/5B406A82/60EF0ED6" Ref="R?"  Part="1"
-AR Path="/60C2EDFB/60EF0ED6" Ref="R66"  Part="1"
-F 0 "R66" H 2720 5146 50  0000 L CNN
+AR Path="/60C2EDFB/60EF0ED6" Ref="R79"  Part="1"
+F 0 "R79" H 2720 5146 50  0000 L CNN
 F 1 "10k" H 2720 5055 50  0000 L CNN
 F 2 "_Generic:0603_RES" V 2580 5100 50  0001 C CNN
@@
 AR Path="/5AF7E834/60C2EDFB/60F01F7D" Ref="C?"  Part="1"
 AR Path="/5B406A82/60F01F7D" Ref="C?"  Part="1"
-AR Path="/60C2EDFB/60F01F7D" Ref="C53"  Part="1"
-F 0 "C53" H 1542 2096 50  0000 L CNN
+AR Path="/60C2EDFB/60F01F7D" Ref="C80"  Part="1"
+F 0 "C80" H 1542 2096 50  0000 L CNN
 F 1 "100n" H 1542 2005 50  0000 L CNN
 F 2 "_Generic:0603_CAP" H 1450 2050 50  0001 C CNN
@@
 AR Path="/5AF7E834/60C2EDFB/60F1567A" Ref="#PWR?"  Part="1"
 AR Path="/5B406A82/60F1567A" Ref="#PWR?"  Part="1"
-AR Path="/60C2EDFB/60F1567A" Ref="#PWR092"  Part="1"
-F 0 "#PWR092" H 1450 1400 50  0001 C CNN
+AR Path="/60C2EDFB/60F1567A" Ref="#PWR0123"  Part="1"
+F 0 "#PWR0123" H 1450 1400 50  0001 C CNN
 F 1 "+3.3V" H 1465 1723 50  0000 C CNN
 F 2 "" H 1450 1550 50  0001 C CNN
@@
 AR Path="/5AF7E834/60C2EDFB/60F38F1C" Ref="R?"  Part="1"
 AR Path="/5B406A82/60F38F1C" Ref="R?"  Part="1"
-AR Path="/60C2EDFB/60F38F1C" Ref="R67"  Part="1"
-F 0 "R67" V 2793 2050 50  0000 C CNN
+AR Path="/60C2EDFB/60F38F1C" Ref="R80"  Part="1"
+F 0 "R80" V 2793 2050 50  0000 C CNN
 F 1 "0R" V 2884 2050 50  0000 C CNN
 F 2 "_Generic:0603_RES" V 2930 2050 50  0001 C CNN
@@
 	3150 2050 3400 2050
 $Comp
-L #Power:GND #PWR093
+L #Power:GND #PWR0124
 U 1 1 5C5C4BD5
 P 1450 2550
-F 0 "#PWR093" H 1450 2300 50  0001 C CNN
+F 0 "#PWR0124" H 1450 2300 50  0001 C CNN
 F 1 "GND" H 1455 2377 50  0000 C CNN
 F 2 "" H 1450 2550 50  0001 C CNN
@@
 Text Notes 550  750  0    100  ~ 20
 Stepper Driver Connection
+Wire Wire Line
+	4850 2050 4900 2050
+Wire Wire Line
+	4850 2150 4900 2150
+Wire Wire Line
+	4850 2350 4900 2350
+Wire Wire Line
+	4850 2250 4900 2250
 $EndSCHEMATC

Commit message: continue routing
Parts:
- removed C80: 100n, _Generic:0603_CAP, symbol Device:C_Small
- removed R80: 0R, _Generic:0603_RES, symbol Device:R
- removed X1: 12MHz, Oscillator:Oscillator_SMD_EuroQuartz_XO32-4Pin_3.2x2.5mm, symbol Oscillator:XO32
Changed lines of the file:
@@
 Wire Wire Line
 	3000 3000 3000 4350
-$Comp
-L Oscillator:XO32 X?
-U 1 1 60F01ECC
-P 2200 2050
-AR Path="/5AF7E834/60C2EDFB/60F01ECC" Ref="X?"  Part="1"
-AR Path="/5B406A82/60F01ECC" Ref="X?"  Part="1"
-AR Path="/60C2EDFB/60F01ECC" Ref="X1"  Part="1"
-F 0 "X1" H 2541 2096 50  0000 L CNN
-F 1 "12MHz" H 2541 2005 50  0000 L CNN
-F 2 "Oscillator:Oscillator_SMD_EuroQuartz_XO32-4Pin_3.2x2.5mm" H 2900 1700 50  0001 C CNN
-F 3 "http://cdn-reichelt.de/documents/datenblatt/B400/XO32.pdf" H 2100 2050 50  0001 C CNN
-	1    2200 2050
-	1    0    0    -1
-$EndComp
-$Comp
-L Device:C_Small C?
-U 1 1 60F01F7D
-P 1450 2050
-AR Path="/5AF7E834/60C2EDFB/60F01F7D" Ref="C?"  Part="1"
-AR Path="/5B406A82/60F01F7D" Ref="C?"  Part="1"
-AR Path="/60C2EDFB/60F01F7D" Ref="C80"  Part="1"
-F 0 "C80" H 1542 2096 50  0000 L CNN
-F 1 "100n" H 1542 2005 50  0000 L CNN
-F 2 "_Generic:0603_CAP" H 1450 2050 50  0001 C CNN
-F 3 "~" H 1450 2050 50  0001 C CNN
-	1    1450 2050
-	1    0    0    -1
-$EndComp
-Wire Wire Line
-	1900 2050 1800 2050
-Wire Wire Line
-	1800 2050 1800 1650
-Wire Wire Line
-	1800 1650 2200 1650
-Wire Wire Line
-	2200 1650 2200 1750
-Wire Wire Line
-	1450 1950 1450 1650
-Wire Wire Line
-	1450 1650 1800 1650
-Connection ~ 1800 1650
-Wire Wire Line
-	1450 2150 1450 2450
-Wire Wire Line
-	1450 2450 2200 2450
-Wire Wire Line
-	2200 2450 2200 2350
-Wire Wire Line
-	1450 2550 1450 2450
-Connection ~ 1450 2450
-$Comp
-L power:+3.3V #PWR?
-U 1 1 60F1567A
-P 1450 1550
-AR Path="/5AF7E834/60C2EDFB/60F1567A" Ref="#PWR?"  Part="1"
-AR Path="/5B406A82/60F1567A" Ref="#PWR?"  Part="1"
-AR Path="/60C2EDFB/60F1567A" Ref="#PWR0123"  Part="1"
-F 0 "#PWR0123" H 1450 1400 50  0001 C CNN
-F 1 "+3.3V" H 1465 1723 50  0000 C CNN
-F 2 "" H 1450 1550 50  0001 C CNN
-F 3 "" H 1450 1550 50  0001 C CNN
-	1    1450 1550
-	1    0    0    -1
-$EndComp
-Wire Wire Line
-	1450 1550 1450 1650
-Connection ~ 1450 1650
-Wire Wire Line
-	2500 2050 2850 2050
-Connection ~ 3400 2050
-$Comp
-L Device:R R?
-U 1 1 60F38F1C
-P 3000 2050
-AR Path="/5AF7E834/60C2EDFB/60F38F1C" Ref="R?"  Part="1"
-AR Path="/5B406A82/60F38F1C" Ref="R?"  Part="1"
-AR Path="/60C2EDFB/60F38F1C" Ref="R80"  Part="1"
-F 0 "R80" V 2793 2050 50  0000 C CNN
-F 1 "0R" V 2884 2050 50  0000 C CNN
-F 2 "_Generic:0603_RES" V 2930 2050 50  0001 C CNN
-F 3 "~" H 3000 2050 50  0001 C CNN
-	1    3000 2050
-	0    1    1    0
-$EndComp
-Wire Wire Line
-	3150 2050 3400 2050
-$Comp
-L #Power:GND #PWR0124
-U 1 1 5C5C4BD5
-P 1450 2550
-F 0 "#PWR0124" H 1450 2300 50  0001 C CNN
-F 1 "GND" H 1455 2377 50  0000 C CNN
-F 2 "" H 1450 2550 50  0001 C CNN
-F 3 "" H 1450 2550 50  0001 C CNN
-	1    1450 2550
-	1    0    0    -1
-$EndComp
 Text Notes 550  750  0    100  ~ 20
 Stepper Driver Connection
@@
 Wire Wire Line
 	4850 2250 4900 2250
+Text HLabel 2450 3950 0    50   Input ~ 0
+DRV_CLK
+Wire Wire Line
+	2450 3950 3400 3950
 $EndSCHEMATC
