File: hardware/kajikia/kajikia.kicad_pcb (KiCad board)
At the start: 2 copper layers, 100 x 75 mm, 43 parts, among them IC1 TMC5161, J39 Screw_Terminal_01x02, J82 Screw_Terminal_01x04, J88 Screw_Terminal_01x04, J89 Conn_01x04

Commit message: tmc layout
Parts:
- added C1: 100n, _Generic:0603_CAP, F.Cu at (170.0, 188.9)
- added C10: 100n, _Generic:0603_CAP, F.Cu at (185.2, 173.0)
- added C102: 10u, _Generic:0603_CAP, F.Cu at (210.2, 140.6)
- added C103: 100n, _Generic:0603_CAP, F.Cu at (214.2, 140.7)
- added C104: 10u, _Generic:0603_CAP, F.Cu at (212.2, 142.5)
- added C105: 470n, _Generic:0603_CAP, F.Cu at (214.2, 139.8)
- added C106: 100n, _Generic:0603_CAP, F.Cu at (208.2, 144.2)
- added C107: 22n, _Generic:0603_CAP, F.Cu at (212.2, 143.4)
- added C108: 100n, _Generic:0603_CAP, F.Cu at (214.2, 141.6)
- added C109: 100n, _Generic:0603_CAP, F.Cu at (210.2, 142.4)
- added C11: 100n, _Generic:0603_CAP, F.Cu at (185.2, 174.8)
- added C110: 470n, _Generic:0603_CAP, F.Cu at (204.2, 145.0)
- added C111: 470n, _Generic:0603_CAP, F.Cu at (212.2, 139.8)
- added C112: 4.7u, _Generic:1210_CAP, F.Cu at (205.2, 139.8)
- added C113: 470n, _Generic:0603_CAP, F.Cu at (212.2, 140.7)
- added C114: 470n, _Generic:0603_CAP, F.Cu at (217.9, 136.3)
- added C115: 4.7u, _Generic:1210_CAP, F.Cu at (209.2, 137.2)
- added C116: 4.7u, _Generic:1210_CAP, F.Cu at (205.2, 137.2)
- added C117: 470p, _Generic:0603_CAP, F.Cu at (212.2, 141.6)
- added C118: 470p, _Generic:0603_CAP, F.Cu at (210.2, 144.2)
- added C119: 470p, _Generic:0603_CAP, F.Cu at (210.2, 143.3)
- added C12: 100n, _Generic:0603_CAP, F.Cu at (185.2, 173.9)
- added C120: 470p, _Generic:0603_CAP, F.Cu at (216.2, 137.2)
- added C121: 470n, _Generic:0603_CAP, F.Cu at (213.9, 138.9)
- added C122: 470n, _Generic:0603_CAP, F.Cu at (211.9, 138.9)
- added C123: 10u, _Generic:0603_CAP, F.Cu at (163.5, 197.5)
- added C124: 100n, _Generic:0603_CAP, F.Cu at (165.5, 194.9)
- added C125: 10u, _Generic:0603_CAP, F.Cu at (159.5, 201.1)
- added C126: 470n, _Generic:0603_CAP, F.Cu at (161.5, 199.3)
- added C127: 100n, _Generic:0603_CAP, F.Cu at (155.5, 201.9)
- added C128: 22n, _Generic:0603_CAP, F.Cu at (161.5, 198.4)
- added C129: 100n, _Generic:0603_CAP, F.Cu at (159.5, 200.2)
- added C13: 100n, _Generic:0603_CAP, F.Cu at (184.5, 175.7)
- added C130: 100n, _Generic:0603_CAP, F.Cu at (157.5, 201.9)
- added C131: 470n, _Generic:0603_CAP, F.Cu at (153.5, 202.7)
- added C132: 470n, _Generic:0603_CAP, F.Cu at (163.5, 194.9)
- added C133: 4.7u, _Generic:1210_CAP, F.Cu at (152.5, 194.9)
- added C134: 470n, _Generic:0603_CAP, F.Cu at (161.5, 197.5)
- added C135: 470n, _Generic:0603_CAP, F.Cu at (159.5, 199.3)
- added C136: 4.7u, _Generic:1210_CAP, F.Cu at (156.5, 194.9)
- added C137: 4.7u, _Generic:1210_CAP, F.Cu at (152.5, 200.1)
- added C138: 470p, _Generic:0603_CAP, F.Cu at (155.5, 200.1)
- added C139: 470p, _Generic:0603_CAP, F.Cu at (159.5, 198.4)
- added C14: 100n, _Generic:0603_CAP, F.Cu at (170.0, 189.8)
- added C140: 470p, _Generic:0603_CAP, F.Cu at (157.5, 200.1)
- added C141: 470p, _Generic:0603_CAP, F.Cu at (159.5, 197.5)
- added C142: 470n, _Generic:0603_CAP, F.Cu at (165.2, 194.0)
- added C143: 470n, _Generic:0603_CAP, F.Cu at (157.5, 201.0)
- added C144: 10u, _Generic:0603_CAP, F.Cu at (205.2, 185.7)
- added C145: 100n, _Generic:0603_CAP, F.Cu at (195.2, 189.1)
- added C146: 10u, _Generic:0603_CAP, F.Cu at (205.0, 186.6)
- added C147: 470n, _Generic:0603_CAP, F.Cu at (197.2, 192.7)
- added C148: 100n, _Generic:0603_CAP, F.Cu at (191.2, 192.6)
- added C149: 22n, _Generic:0603_CAP, F.Cu at (195.2, 190.9)
- added C15: 100n, _Generic:0603_CAP, F.Cu at (172.6, 188.0)
- added C150: 100n, _Generic:0603_CAP, F.Cu at (191.2, 193.5)
- added C151: 100n, _Generic:0603_CAP, F.Cu at (197.2, 190.0)
- added C152: 470n, _Generic:0603_CAP, F.Cu at (193.2, 193.5)
- added C153: 470n, _Generic:0603_CAP, F.Cu at (195.2, 191.8)
- added C154: 4.7u, _Generic:1210_CAP, F.Cu at (192.2, 185.7)
- added C155: 470n, _Generic:0603_CAP, F.Cu at (201.0, 187.4)
- added C156: 470n, _Generic:0603_CAP, F.Cu at (193.2, 192.6)
- added C157: 4.7u, _Generic:1210_CAP, F.Cu at (192.2, 190.9)
- added C158: 4.7u, _Generic:1210_CAP, F.Cu at (192.2, 188.3)
- added C159: 470p, _Generic:0603_CAP, F.Cu at (195.2, 192.7)
- added C16: 100n, _Generic:0603_CAP, F.Cu at (174.6, 186.2)
- added C160: 470p, _Generic:0603_CAP, F.Cu at (195.2, 190.0)
- added C161: 470p, _Generic:0603_CAP, F.Cu at (199.2, 191.9)
- added C162: 470p, _Generic:0603_CAP, F.Cu at (199.0, 187.4)
- added C163: 470n, _Generic:0603_CAP, F.Cu at (197.2, 190.9)
- added C164: 470n, _Generic:0603_CAP, F.Cu at (197.2, 189.1)
- added C165: 10u, _Generic:0603_CAP, F.Cu at (215.9, 151.6)
- added C166: 100n, _Generic:0603_CAP, F.Cu at (216.2, 149.9)
- added C167: 10u, _Generic:0603_CAP, F.Cu at (210.2, 156.0)
- added C168: 470n, _Generic:0603_CAP, F.Cu at (214.2, 152.5)
- added C169: 100n, _Generic:0603_CAP, F.Cu at (212.2, 154.3)
- added C17: 10u, _Generic:0603_CAP, F.Cu at (172.6, 187.1)
- added C170: 22n, _Generic:0603_CAP, F.Cu at (217.9, 149.0)
- added C171: 100n, _Generic:0603_CAP, F.Cu at (212.2, 153.4)
- added C172: 100n, _Generic:0603_CAP, F.Cu at (212.2, 152.5)
- added C173: 470n, _Generic:0603_CAP, F.Cu at (218.2, 149.9)
- added C174: 470n, _Generic:0603_CAP, F.Cu at (206.2, 156.8)
- added C175: 4.7u, _Generic:1210_CAP, F.Cu at (205.2, 149.8)
- added C176: 470n, _Generic:0603_CAP, F.Cu at (208.2, 156.9)
- added C177: 470n, _Generic:0603_CAP, F.Cu at (213.9, 151.6)
- added C178: 4.7u, _Generic:1210_CAP, F.Cu at (205.2, 152.4)
- added C179: 4.7u, _Generic:1210_CAP, F.Cu at (205.2, 155.0)
- added C18: 10u, _Generic:0603_CAP, F.Cu at (193.6, 148.1)
- added C180: 470p, _Generic:0603_CAP, F.Cu at (210.2, 155.1)
- added C181: 470p, _Generic:0603_CAP, F.Cu at (212.2, 155.2)
- added C182: 470p, _Generic:0603_CAP, F.Cu at (214.2, 150.7)
- added C183: 470p, _Generic:0603_CAP, F.Cu at (204.2, 157.7)
- added C184: 470n, _Generic:0603_CAP, F.Cu at (208.2, 153.3)
- added C185: 470n, _Generic:0603_CAP, F.Cu at (210.2, 156.9)
- added C186: 4.7u, _Generic:1210_CAP, B.Cu at (145.5, 64.0)
- added C187: 4.7u, _Generic:1210_CAP, F.Cu at (205.2, 142.4)
- added C188: 4.7u, _Generic:1210_CAP, F.Cu at (152.5, 197.5)
- added C189: 4.7u, _Generic:1210_CAP, F.Cu at (196.2, 185.7)
- added C19: 68u, Capacitor_SMD:CP_Elec_8x10, F.Cu at (161.7, 145.4)
- added C190: 4.7u, _Generic:1210_CAP, F.Cu at (209.2, 149.8)
- added C2: 10u, _Generic:0603_CAP, F.Cu at (172.6, 186.2)
- added C20: 10u, _Generic:0603_CAP, F.Cu at (198.6, 141.6)
- added C21: 10u, _Generic:0603_CAP, F.Cu at (169.2, 159.5)
- added C22: 10u, _Generic:0603_CAP, F.Cu at (193.6, 149.0)
- added C23: 4.7u, _Generic:0805_CAP, F.Cu at (177.1, 151.0)
- added C24: 4.7u, _Generic:0805_CAP, F.Cu at (198.9, 140.5)
- added C25: 4.7u, _Generic:0805_CAP, F.Cu at (159.9, 159.4)
- added C26: 4.7u, _Generic:0805_CAP, F.Cu at (179.6, 151.0)
- added C27: 4.7u, _Generic:0805_CAP, F.Cu at (186.9, 141.7)
- added C28: 4.7u, _Generic:0805_CAP, F.Cu at (157.4, 159.4)
- added C29: 100n, _Generic:0603_CAP, F.Cu at (181.6, 143.4)
- added C3: 12p, _Generic:0603_CAP, F.Cu at (182.5, 175.7)
- added C30: 100n, _Generic:0603_CAP, F.Cu at (167.2, 160.2)
- added C31: 4.7u, _Generic:0805_CAP, F.Cu at (179.3, 143.7)
- added C32: 4.7u, _Generic:0805_CAP, F.Cu at (162.4, 159.8)
- added C33: 22n, _Generic:0603_CAP, F.Cu at (197.8, 144.7)
- added C34: 22n, _Generic:0603_CAP, F.Cu at (191.6, 148.1)
- added C35: 12p, _Generic:0603_CAP, F.Cu at (171.2, 159.5)
- added C36: 12p, _Generic:0603_CAP, F.Cu at (173.2, 159.5)
- added C37: 100n, _Generic:0603_CAP, F.Cu at (175.2, 160.2)
- added C38: 100n, _Generic:0603_CAP, F.Cu at (177.2, 160.2)
- added C39: DNP, _Generic:0603_CAP, F.Cu at (179.2, 160.2)
- added C4: 10u, _Generic:0603_CAP, F.Cu at (182.5, 178.4)
- added C40: DNP, _Generic:0603_CAP, F.Cu at (180.9, 158.7)
- added C41: 10u, _Generic:0603_CAP, F.Cu at (197.8, 142.9)
- added C42: 10u, _Generic:0603_CAP, F.Cu at (192.2, 150.8)
- added C43: 390u, Capacitor_SMD:CP_Elec_8x10, F.Cu at (161.7, 154.3)
- added C44: 390u, Capacitor_SMD:CP_Elec_8x10, F.Cu at (172.8, 140.3)
- added C45: 100n, _Generic:0603_CAP, F.Cu at (143.7, 177.2)
- added C46: 10u, _Generic:0603_CAP, F.Cu at (138.8, 182.1)
- added C47: 100n, _Generic:0603_CAP, F.Cu at (128.9, 192.6)
- added C48: 22n, _Generic:0603_CAP, F.Cu at (124.3, 194.8)
- added C49: 10u, _Generic:0603_CAP, F.Cu at (126.3, 196.2)
- added C5: 12p, _Generic:0603_CAP, F.Cu at (174.6, 187.1)
- added C50: 12p, _Generic:0603_CAP, F.Cu at (131.9, 189.1)
- added C51: 12p, _Generic:0603_CAP, F.Cu at (138.0, 185.0)
- added C52: 100n, _Generic:0603_CAP, F.Cu at (124.3, 196.6)
- added C53: 22n, _Generic:0603_CAP, F.Cu at (136.0, 183.6)
- added C54: 4.7u, _Generic:0805_CAP, F.Cu at (132.1, 182.5)
- added C55: 4.7u, _Generic:0805_CAP, F.Cu at (138.7, 180.0)
- added C56: 4.7u, _Generic:0805_CAP, F.Cu at (124.6, 193.6)
- added C57: 4.7u, _Generic:0805_CAP, F.Cu at (134.6, 182.5)
- added C58: 10u, _Generic:0603_CAP, F.Cu at (136.0, 186.3)
- added C59: 10u, _Generic:0603_CAP, F.Cu at (141.0, 179.8)
- added C6: 100n, _Generic:0603_CAP, F.Cu at (179.9, 180.9)
- added C60: 10u, _Generic:0603_CAP, F.Cu at (136.0, 184.5)
- added C61: 10u, _Generic:0603_CAP, F.Cu at (126.8, 193.5)
- added C62: 10u, _Generic:0603_CAP, F.Cu at (143.4, 153.7)
- added C63: 100n, _Generic:0603_CAP, F.Cu at (134.3, 162.6)
- added C64: 4.7u, _Generic:0805_CAP, F.Cu at (124.5, 164.6)
- added C65: 4.7u, _Generic:0805_CAP, F.Cu at (138.9, 155.4)
- added C66: 4.7u, _Generic:0805_CAP, F.Cu at (106.7, 165.5)
- added C67: 68u, Capacitor_SMD:CP_Elec_8x10, F.Cu at (125.6, 153.9)
- added C68: 4.7u, _Generic:0805_CAP, F.Cu at (119.3, 166.0)
- added C69: 4.7u, _Generic:0805_CAP, F.Cu at (121.8, 166.0)
- added C7: 10u, _Generic:0603_CAP, F.Cu at (177.3, 183.6)
- added C70: 4.7u, _Generic:0805_CAP, F.Cu at (124.3, 166.0)
- added C71: 4.7u, _Generic:0805_CAP, F.Cu at (122.0, 164.6)
- added C72: 4.7u, _Generic:0805_CAP, F.Cu at (119.5, 164.6)
- added C73: 10u, _Generic:0603_CAP, F.Cu at (141.2, 156.1)
- added C74: 100n, _Generic:0603_CAP, F.Cu at (149.6, 145.9)
- added C75: 4.7u, _Generic:0805_CAP, F.Cu at (116.8, 165.3)
- added C76: 4.7u, _Generic:0805_CAP, F.Cu at (99.2, 165.5)
- added C77: 68u, Capacitor_SMD:CP_Elec_8x10, F.Cu at (136.5, 147.1)
- added C78: 4.7u, _Generic:0805_CAP, F.Cu at (101.7, 165.5)
- added C79: 4.7u, _Generic:0805_CAP, F.Cu at (104.2, 165.5)
- added C8: 100n, _Generic:0603_CAP, F.Cu at (182.5, 177.5)
- added C80: 100n, _Generic:0603_CAP, F.Cu at (195.1, 177.7)
- added C9: 10u, _Generic:0603_CAP, F.Cu at (182.5, 176.6)
- added D1: 16v, _Generic:SOD-523_DIODE, F.Cu at (181.2, 159.6)
- added D10: 3.6v, _Generic:SOD-523_DIODE, F.Cu at (126.8, 194.4)
- added D11: DNP, _Generic:SOD-523_DIODE, F.Cu at (145.3, 176.3)
- added D12: DNP, _Generic:SOD-523_DIODE, F.Cu at (140.5, 181.2)
- added D13: DNP, _Generic:SOD-523_DIODE, F.Cu at (136.0, 185.4)
- added D14: DNP, _Generic:SOD-523_DIODE, F.Cu at (130.9, 191.7)
- added D15: 3.6v, _Generic:SOD-523_DIODE, F.Cu at (141.4, 152.0)
- added D16: 3.6v, _Generic:SOD-523_DIODE, F.Cu at (147.1, 141.9)
- added D17: 3.6v, _Generic:SOD-523_DIODE, F.Cu at (145.1, 141.9)
- added D18: LED, _Generic:0603_LED, F.Cu at (151.6, 145.9)
- added D19: LED, _Generic:0603_LED, F.Cu at (141.2, 155.2)
- added D2: 3.6v, _Generic:SOD-523_DIODE, F.Cu at (195.1, 146.4)
- added D20: 3.6v, _Generic:SOD-523_DIODE, F.Cu at (131.8, 157.6)
- added D21: 3.6v, _Generic:SOD-523_DIODE, F.Cu at (143.1, 141.9)
- added D22: 3.6v, _Generic:SOD-523_DIODE, F.Cu at (143.4, 152.8)
- added D23: 3.6v, _Generic:SOD-523_DIODE, F.Cu at (141.0, 157.0)
- added D24: 3.6v, _Generic:SOD-523_DIODE, F.Cu at (143.2, 154.7)
- added D25: LED, _Generic:0603_LED, F.Cu at (147.5, 149.6)
- added D26: LED, _Generic:0603_LED, F.Cu at (134.3, 161.7)
- added D3: 3.6v, _Generic:SOD-523_DIODE, F.Cu at (197.8, 143.8)
- added D35: MSK4010, _Generic:SOD-523_DIODE, F.Cu at (208.2, 143.3)
- added D36: MSK4010, _Generic:SOD-523_DIODE, F.Cu at (208.2, 142.4)
- added D37: MSK4010, _Generic:SOD-523_DIODE, F.Cu at (206.2, 145.0)
- added D38: MSK4010, _Generic:SOD-523_DIODE, F.Cu at (214.2, 138.0)
- added D39: MSK4010, _Generic:SOD-523_DIODE, F.Cu at (215.9, 136.3)
- added D4: LED, _Generic:0603_LED, F.Cu at (182.9, 158.7)
- added D40: MSK4010, _Generic:SOD-523_DIODE, F.Cu at (212.2, 138.0)
- added D41: MSK4010, _Generic:SOD-523_DIODE, F.Cu at (218.2, 137.2)
- added D42: MSK4010, _Generic:SOD-523_DIODE, F.Cu at (215.9, 138.9)
- added D43: MSK4010, _Generic:SOD-523_DIODE, F.Cu at (165.2, 195.8)
- added D44: MSK4010, _Generic:SOD-523_DIODE, F.Cu at (153.5, 201.8)
- added D45: MSK4010, _Generic:SOD-523_DIODE, F.Cu at (163.2, 196.6)
- added D46: MSK4010, _Generic:SOD-523_DIODE, F.Cu at (157.5, 199.2)
- added D47: MSK4010, _Generic:SOD-523_DIODE, F.Cu at (159.2, 196.6)
- added D48: MSK4010, _Generic:SOD-523_DIODE, F.Cu at (161.2, 196.6)
- added D49: MSK4010, _Generic:SOD-523_DIODE, F.Cu at (161.5, 195.7)
- added D5: SK54, _Generic:SMB_DIODE, F.Cu at (185.8, 144.9)
- added D50: MSK4010, _Generic:SOD-523_DIODE, F.Cu at (155.5, 201.0)
- added D51: MSK4010, _Generic:SOD-523_DIODE, F.Cu at (199.2, 190.1)
- added D52: MSK4010, _Generic:SOD-523_DIODE, F.Cu at (203.2, 188.3)
- added D53: MSK4010, _Generic:SOD-523_DIODE, F.Cu at (199.2, 188.3)
- added D54: MSK4010, _Generic:SOD-523_DIODE, F.Cu at (199.2, 189.2)
- added D55: MSK4010, _Generic:SOD-523_DIODE, F.Cu at (201.2, 188.3)
- added D56: MSK4010, _Generic:SOD-523_DIODE, F.Cu at (197.2, 191.8)
- added D57: MSK4010, _Generic:SOD-523_DIODE, F.Cu at (203.2, 185.7)
- added D58: MSK4010, _Generic:SOD-523_DIODE, F.Cu at (203.0, 187.4)
- added D59: MSK4010, _Generic:SOD-523_DIODE, F.Cu at (210.2, 153.3)
- added D6: SK54, _Generic:SMB_DIODE, F.Cu at (195.4, 137.8)
- added D60: MSK4010, _Generic:SOD-523_DIODE, F.Cu at (208.2, 155.1)
- added D61: MSK4010, _Generic:SOD-523_DIODE, F.Cu at (215.9, 149.0)
- added D62: MSK4010, _Generic:SOD-523_DIODE, F.Cu at (204.2, 156.8)
- added D63: MSK4010, _Generic:SOD-523_DIODE, F.Cu at (214.2, 153.4)
- added D64: MSK4010, _Generic:SOD-523_DIODE, F.Cu at (210.2, 154.2)
- added D65: MSK4010, _Generic:SOD-523_DIODE, F.Cu at (214.2, 154.3)
- added D66: MSK4010, _Generic:SOD-523_DIODE, F.Cu at (208.2, 154.2)
- added D7: 3.6v, _Generic:SOD-523_DIODE, F.Cu at (126.9, 191.7)
- added D8: 3.6v, _Generic:SOD-523_DIODE, F.Cu at (126.9, 192.6)
- added D9: 3.6v, _Generic:SOD-523_DIODE, F.Cu at (138.0, 183.2)
- added F1: FUSE, _Generic:SMD_Fuseholder, F.Cu at (161.7, 138.4)
- added F2: FUSE, _Generic:SMD_Fuseholder, F.Cu at (114.6, 138.4)
- added F3: FUSE, _Generic:SMD_Fuseholder, F.Cu at (103.5, 143.5)
- added F4: FUSE, _Generic:SMD_Fuseholder, F.Cu at (103.5, 138.4)
- added F5: FUSE, _Generic:SMD_Fuseholder, F.Cu at (103.5, 148.6)
- added H1: M3, MountingHole:MountingHole_3.2mm_M3_ISO14580_Pad, F.Cu at (103.0, 53.0)
- added H2: M3, MountingHole:MountingHole_3.2mm_M3_ISO14580_Pad, F.Cu at (197.0, 53.0)
- added H3: M3, MountingHole:MountingHole_3.2mm_M3_ISO14580_Pad, F.Cu at (197.0, 122.0)
- added H4: M3, MountingHole:MountingHole_3.2mm_M3_ISO14580_Pad, F.Cu at (103.0, 122.0)
- added IC2, IC3, IC4, IC5: TMC5161, footprints:QFN42L, F.Cu at (110.5, 195.8)
- added J1: Conn_01x01, _Generic:PinHeader_2.54mm_1P, F.Cu at (182.9, 173.9)
- added J10: Conn_01x01, _Generic:PinHeader_2.54mm_1P, F.Cu at (165.0, 189.1)
- added J11: Conn_01x01, _Generic:PinHeader_2.54mm_1P, F.Cu at (174.9, 176.5)
- added J12: Conn_01x01, _Generic:PinHeader_2.54mm_1P, F.Cu at (177.6, 179.2)
- added J13: Conn_01x01, _Generic:PinHeader_2.54mm_1P, F.Cu at (177.6, 173.9)
- added J14: Conn_01x01, _Generic:PinHeader_2.54mm_1P, F.Cu at (180.2, 176.5)
- added J15: Conn_01x01, _Generic:PinHeader_2.54mm_1P, F.Cu at (169.7, 171.2)
- added J16: Conn_01x01, _Generic:PinHeader_2.54mm_1P, F.Cu at (169.7, 184.4)
- added J17: Conn_01x01, _Generic:PinHeader_2.54mm_1P, F.Cu at (172.3, 181.8)
- added J18: Conn_01x01, _Generic:PinHeader_2.54mm_1P, F.Cu at (174.9, 179.2)
- added J19: Conn_01x01, _Generic:PinHeader_2.54mm_1P, F.Cu at (177.6, 176.5)
- added J2: Conn_01x01, _Generic:PinHeader_2.54mm_1P, F.Cu at (185.5, 171.2)
- added J20: Conn_01x01, _Generic:PinHeader_2.54mm_1P, F.Cu at (180.2, 173.9)
- added J21: Conn_01x01, _Generic:PinHeader_2.54mm_1P, F.Cu at (182.9, 171.2)
- added J22: Conn_01x01, _Generic:PinHeader_2.54mm_1P, F.Cu at (167.7, 189.1)
- added J23: Conn_01x01, _Generic:PinHeader_2.54mm_1P, F.Cu at (172.3, 184.4)
- added J24: Conn_01x01, _Generic:PinHeader_2.54mm_1P, F.Cu at (174.9, 181.8)
- added J25: Conn_01x01, _Generic:PinHeader_2.54mm_1P, F.Cu at (162.4, 189.1)
- added J26: Conn_01x01, _Generic:PinHeader_2.54mm_1P, F.Cu at (157.1, 189.1)
- added J27: Conn_01x01, _Generic:PinHeader_2.54mm_1P, F.Cu at (169.7, 176.5)
- added J28: Conn_01x01, _Generic:PinHeader_2.54mm_1P, F.Cu at (169.7, 181.8)
- added J29: Conn_01x01, _Generic:PinHeader_2.54mm_1P, F.Cu at (177.6, 171.2)
- added J3: Conn_01x01, _Generic:PinHeader_2.54mm_1P, F.Cu at (177.6, 181.8)
- added J30: Conn_01x01, _Generic:PinHeader_2.54mm_1P, F.Cu at (172.3, 179.2)
- added J31: Conn_01x01, _Generic:PinHeader_2.54mm_1P, F.Cu at (174.9, 173.9)
- added J32: Conn_01x01, _Generic:PinHeader_2.54mm_1P, F.Cu at (170.3, 187.1)
- added J33: Conn_01x01, _Generic:PinHeader_2.54mm_1P, F.Cu at (172.3, 176.5)
- added J34: Conn_01x01, _Generic:PinHeader_2.54mm_1P, F.Cu at (169.7, 179.2)
- added J35: Conn_01x01, _Generic:PinHeader_2.54mm_1P, F.Cu at (174.9, 171.2)
- added J36: Conn_01x01, _Generic:PinHeader_2.54mm_1P, F.Cu at (159.7, 189.1)
- added J37: Conn_01x01, _Generic:PinHeader_2.54mm_1P, F.Cu at (172.3, 171.2)
- added J38: Conn_01x01, _Generic:PinHeader_2.54mm_1P, F.Cu at (172.3, 173.9)
- added J4: Conn_01x01, _Generic:PinHeader_2.54mm_1P, F.Cu at (180.2, 179.2)
- added J40: Conn_01x01, _Generic:PinHeader_2.54mm_1P, F.Cu at (182.6, 156.9)
- added J41: Conn_01x01, _Generic:PinHeader_2.54mm_1P, F.Cu at (196.3, 141.1)
- added J42: Conn_01x01, _Generic:PinHeader_2.54mm_1P, F.Cu at (185.2, 156.1)
- added J43: Conn_01x01, _Generic:PinHeader_2.54mm_1P, F.Cu at (187.8, 150.8)
- added J44: Conn_01x01, _Generic:PinHeader_2.54mm_1P, F.Cu at (195.5, 143.7)
- added J45: Conn_01x01, _Generic:PinHeader_2.54mm_1P, F.Cu at (185.2, 153.5)
- added J46: Conn_01x01, _Generic:PinHeader_2.54mm_1P, F.Cu at (184.0, 148.2)
- added J47: Conn_01x01, _Generic:PinHeader_2.54mm_1P, F.Cu at (192.8, 143.7)
- added J48: Conn_01x01, _Generic:PinHeader_2.54mm_1P, F.Cu at (175.9, 158.4)
- added J49: Conn_01x01, _Generic:PinHeader_2.54mm_1P, F.Cu at (178.5, 158.4)
- added J5: Conn_01x01, _Generic:PinHeader_2.54mm_1P, F.Cu at (180.2, 171.2)
- added J50: Conn_01x01, _Generic:PinHeader_2.54mm_1P, F.Cu at (182.6, 154.3)
- added J51: Conn_01x01, _Generic:PinHeader_2.54mm_1P, F.Cu at (185.2, 150.8)
- added J52: Conn_01x01, _Generic:PinHeader_2.54mm_1P, F.Cu at (190.2, 144.9)
- added J53: Conn_01x01, _Generic:PinHeader_2.54mm_1P, F.Cu at (190.2, 142.3)
- added J54: Conn_01x01, _Generic:PinHeader_2.54mm_1P, F.Cu at (193.7, 141.1)
- added J55: Conn_01x01, _Generic:PinHeader_2.54mm_1P, F.Cu at (189.3, 148.2)
- added J56: Conn_01x01, _Generic:PinHeader_2.54mm_1P, F.Cu at (182.6, 151.6)
- added J57: Conn_01x01, _Generic:PinHeader_2.54mm_1P, F.Cu at (186.6, 148.2)
- added J58: Conn_01x01, _Generic:PinHeader_2.54mm_1P, F.Cu at (192.8, 146.4)
- added J59: Conn_01x01, _Generic:PinHeader_2.54mm_1P, F.Cu at (187.8, 153.5)
- added J6: Conn_01x01, _Generic:PinHeader_2.54mm_1P, F.Cu at (174.9, 184.4)
- added J62: Conn_01x02, _Generic:JST_XH_2P, F.Cu at (126.6, 179.6)
- added J63: Conn_01x02, _Generic:JST_XH_2P, F.Cu at (119.1, 193.2)
- added J64: Conn_01x04, _Generic:JST_XH_4P, F.Cu at (104.7, 179.6)
- added J65: Conn_01x04, _Generic:JST_XH_4P, F.Cu at (118.2, 172.8)
- added J66: Conn_01x03, _Generic:JST_XH_3P, F.Cu at (114.4, 186.4)
- added J67: Conn_01x03, _Generic:JST_XH_3P, F.Cu at (130.4, 172.8)
- added J68: Conn_01x03, _Generic:JST_XH_3P, F.Cu at (103.5, 186.4)
- added J69: Conn_01x03, _Generic:JST_XH_3P, F.Cu at (116.9, 179.6)
- added J7: Conn_01x01, _Generic:PinHeader_2.54mm_1P, F.Cu at (151.8, 189.1)
- added J70: Conn_01x04, _Generic:JST_XH_4P, F.Cu at (104.7, 172.8)
- added J71: Conn_01x02, _Generic:JST_XH_2P, F.Cu at (140.0, 172.8)
- added J72: Conn_01x02, _Generic:JST_XH_2P, F.Cu at (102.2, 193.2)
- added J73: Conn_01x02, _Generic:JST_XH_2P, F.Cu at (110.6, 193.2)
- added J74: Conn_01x02, _Generic:JST_XH_2P, F.Cu at (124.1, 186.4)
- added J75: Conn_01x01, _Generic:PinHeader_2.54mm_1P, F.Cu at (124.6, 191.6)
- added J76: Conn_01x01, _Generic:PinHeader_2.54mm_1P, F.Cu at (138.8, 178.0)
- added J77: Conn_01x01, _Generic:PinHeader_2.54mm_1P, F.Cu at (129.6, 189.9)
- added J78: Conn_01x01, _Generic:PinHeader_2.54mm_1P, F.Cu at (141.4, 178.0)
- added J79: Conn_01x03, _Generic:JST_XH_3P, F.Cu at (114.6, 143.9)
- added J8: Conn_01x01, _Generic:PinHeader_2.54mm_1P, F.Cu at (154.5, 189.1)
- added J80: Conn_01x03, _Generic:JST_XH_3P, F.Cu at (103.5, 154.1)
- added J81: Conn_01x03, _Generic:JST_XH_3P, F.Cu at (114.4, 157.5)
- added J83: Conn_01x03, _Generic:JST_XH_3P, F.Cu at (125.7, 138.8)
- added J84: Conn_01x03, _Generic:JST_XH_3P, F.Cu at (103.5, 160.9)
- added J85: Conn_01x03, _Generic:JST_XH_3P, F.Cu at (125.5, 145.6)
- added J86: Conn_01x03, _Generic:JST_XH_3P, F.Cu at (136.6, 138.8)
- added J87: Conn_01x03, _Generic:JST_XH_3P, F.Cu at (114.6, 150.7)
- added J9: Conn_01x01, _Generic:PinHeader_2.54mm_1P, F.Cu at (169.7, 173.9)
- added J90: Conn_01x04, _Generic:JST_XH_4P, F.Cu at (210.4, 166.5)
- added J91: Conn_01x04, _Generic:JST_XH_4P, F.Cu at (197.0, 173.3)
- added J92: Conn_01x04, _Generic:JST_XH_4P, F.Cu at (197.0, 166.5)
- added J93: Conn_01x04, _Generic:JST_XH_4P, F.Cu at (210.4, 173.3)
- added L1: 1u, _Generic:0805_IND, F.Cu at (164.9, 159.4)
- added L2: BCIHP0750-6R8M, _Generic:7x7mm_IND, F.Cu at (181.9, 139.4)
- added L3: BCIHP0750-6R8M, _Generic:7x7mm_IND, F.Cu at (170.8, 155.5)
- added L4: 470, _Generic:0603_IND, F.Cu at (131.9, 190.0)
- added L5: 470, _Generic:0603_IND, F.Cu at (138.0, 184.1)
- added L6: 470, _Generic:0603_IND, F.Cu at (143.0, 179.8)
- added L7: 470, _Generic:0603_IND, F.Cu at (133.9, 189.1)
- added Q1: AON6144, _Generic:DFN5x6-8, F.Cu at (179.3, 147.5)
- added Q10: AO3400, _Generic:SOT-23, F.Cu at (134.7, 158.7)
- added Q11: AON6144, _Generic:DFN5x6-8, F.Cu at (134.3, 154.3)
- added Q12: AO3400, _Generic:SOT-23, F.Cu at (139.0, 153.1)
- added Q13: AO3400, _Generic:SOT-23, F.Cu at (150.2, 137.5)
- added Q14: AON6144, _Generic:DFN5x6-8, F.Cu at (145.5, 138.7)
- added Q2: AO3401, _Generic:SOT-23, F.Cu at (145.6, 171.5)
- added Q3: AO3400, _Generic:SOT-23, F.Cu at (116.9, 163.0)
- added Q4: AO3400, _Generic:SOT-23, F.Cu at (150.2, 140.7)
- added Q5: AO3400, _Generic:SOT-23, F.Cu at (143.1, 149.9)
- added Q6: AON6144, _Generic:DFN5x6-8, F.Cu at (145.2, 145.5)
- added Q7: AON6144, _Generic:DFN5x6-8, F.Cu at (123.3, 161.1)
- added Q8: AO3400, _Generic:SOT-23, F.Cu at (150.0, 143.9)
- added Q9: AO3400, _Generic:SOT-23, F.Cu at (128.0, 165.0)
- added R1: 10k, _Generic:0603_RES, F.Cu at (182.5, 179.3)
- added R10: 47k, _Generic:0603_RES, F.Cu at (197.1, 146.5)
- added R100: 2.2R, _Generic:0603_RES, F.Cu at (155.5, 198.3)
- added R101: 1k, _Generic:0603_RES, F.Cu at (163.2, 194.0)
- added R102: 47R, _Generic:0603_RES, F.Cu at (159.5, 195.7)
- added R103: 47R, _Generic:0603_RES, F.Cu at (151.5, 201.8)
- added R104: 47R, _Generic:0603_RES, F.Cu at (155.5, 199.2)
- added R105: 47R, _Generic:0603_RES, F.Cu at (157.5, 198.3)
- added R106: 100m, _Generic:1206_RES, F.Cu at (156.4, 197.0)
- added R107: 100m, _Generic:1206_RES, F.Cu at (160.4, 194.4)
- added R108: 0R, _Generic:0603_RES, F.Cu at (205.0, 184.8)
- added R109: 2.2R, _Generic:0603_RES, F.Cu at (201.2, 190.1)
- added R11: 47k, _Generic:0603_RES, F.Cu at (197.1, 145.6)
- added R110: 1k, _Generic:0603_RES, F.Cu at (201.2, 186.5)
- added R111: 47R, _Generic:0603_RES, F.Cu at (203.0, 184.8)
- added R112: 47R, _Generic:0603_RES, F.Cu at (199.2, 186.5)
- added R113: 47R, _Generic:0603_RES, F.Cu at (199.2, 191.0)
- added R114: 47R, _Generic:0603_RES, F.Cu at (201.2, 189.2)
- added R115: 100m, _Generic:1206_RES, F.Cu at (200.1, 185.2)
- added R116: 100m, _Generic:1206_RES, F.Cu at (196.1, 187.8)
- added R117: 0R, _Generic:0603_RES, F.Cu at (208.2, 156.0)
- added R118: 2.2R, _Generic:0603_RES, F.Cu at (206.2, 157.7)
- added R119: 1k, _Generic:0603_RES, F.Cu at (211.9, 151.6)
- added R12: 140k, _Generic:0603_RES, F.Cu at (190.2, 152.7)
- added R120: 47R, _Generic:0603_RES, F.Cu at (217.9, 150.8)
- added R121: 47R, _Generic:0603_RES, F.Cu at (216.2, 152.5)
- added R122: 47R, _Generic:0603_RES, F.Cu at (212.2, 150.7)
- added R123: 47R, _Generic:0603_RES, F.Cu at (212.2, 156.1)
- added R124: 100m, _Generic:1206_RES, F.Cu at (209.0, 152.0)
- added R125: 100m, _Generic:1206_RES, F.Cu at (213.0, 149.4)
- added R13: 140k, _Generic:0603_RES, F.Cu at (187.5, 155.2)
- added R14: 1k, _Generic:0603_RES, F.Cu at (190.2, 151.8)
- added R15: 100k, _Generic:0603_RES, F.Cu at (195.1, 145.5)
- added R16: 100k, _Generic:0603_RES, F.Cu at (192.2, 149.9)
- added R17: 140k, _Generic:0603_RES, F.Cu at (183.2, 159.6)
- added R18: 10k, _Generic:0603_RES, F.Cu at (190.2, 150.0)
- added R19: 52.3k, _Generic:0603_RES, F.Cu at (191.6, 149.0)
- added R2: 10k, _Generic:0603_RES, F.Cu at (184.5, 176.6)
- added R20: 10k, _Generic:0603_RES, F.Cu at (184.9, 157.9)
- added R21: 4.7k, _Generic:0603_RES, F.Cu at (136.0, 187.2)
- added R22: 4.7k, _Generic:0603_RES, F.Cu at (138.0, 186.8)
- added R23: 0R, _Generic:0603_RES, F.Cu at (126.3, 197.1)
- added R24: 47R, _Generic:0603_RES, F.Cu at (130.9, 192.6)
- added R25: 47R, _Generic:0603_RES, F.Cu at (126.3, 195.3)
- added R26: 1.5k, _Generic:0603_RES, F.Cu at (132.9, 190.9)
- added R27: 10k, _Generic:0603_RES, F.Cu at (136.8, 182.3)
- added R28: 50k, _Generic:0603_RES, F.Cu at (128.3, 195.3)
- added R29: 10k, _Generic:0603_RES, F.Cu at (140.0, 183.0)
- added R3: 1k, _Generic:0603_RES, F.Cu at (172.0, 188.9)
- added R30: 10k, _Generic:0603_RES, F.Cu at (136.0, 188.1)
- added R31: 10k, _Generic:0603_RES, F.Cu at (140.0, 183.9)
- added R32: 47k, _Generic:0603_RES, F.Cu at (138.0, 185.9)
- added R33: 47k, _Generic:0603_RES, F.Cu at (133.9, 190.0)
- added R34: 0R, _Generic:0603_RES, F.Cu at (145.7, 178.1)
- added R35: 47k, _Generic:0603_RES, F.Cu at (145.0, 179.0)
- added R36: 47k, _Generic:0603_RES, F.Cu at (130.8, 193.5)
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Connections:
- C83 pad 1: Net-(C83-Pad1) -> /Stepper Driver/Driver1/5V_out
- IC1 pad 11: Net-(IC1-Pad11) -> /Stepper Driver/Driver1/SRBH
- IC1 pad 3: GND -> Net-(IC1-Pad3)
- IC1 pad 5: GND -> /Stepper Driver/Driver1/5V_out
- IC1 pad 6: Net-(C83-Pad1) -> /Stepper Driver/Driver1/5V_out
- IC1 pad 9: GND -> Net-(IC1-Pad9)
- IC1 pad BL: Net-(IC1-PadBL) -> /Stepper Driver/Driver1/SRBH
- R82 pad 2: Net-(C83-Pad1) -> /Stepper Driver/Driver1/5V_out
- R86 pad 2: Net-(IC1-Pad11) -> /Stepper Driver/Driver1/SRBH
Routing:
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- added copper zone on B.Cu, net +24V
- added copper zone on F.Cu, net +24V
- added copper zone on B.Cu, net /Stepper Driver/Driver1/OA1
- added copper zone on F.Cu, net /Stepper Driver/Driver1/OA1
- added copper zone on In1.Cu, net /Stepper Driver/Driver1/OA1
- added copper zone on In2.Cu, net /Stepper Driver/Driver1/OA1
- added copper zone on B.Cu, net /Stepper Driver/Driver1/OA2
- added copper zone on F.Cu, net /Stepper Driver/Driver1/OA2
- added copper zone on In1.Cu, net /Stepper Driver/Driver1/OA2
- added copper zone on In2.Cu, net /Stepper Driver/Driver1/OA2
- added copper zone on B.Cu, net /Stepper Driver/Driver1/OB1
- added copper zone on F.Cu, net /Stepper Driver/Driver1/OB1
- added copper zone on In1.Cu, net /Stepper Driver/Driver1/OB1
- added copper zone on In2.Cu, net /Stepper Driver/Driver1/OB1
- added copper zone on B.Cu, net /Stepper Driver/Driver1/OB2
- added copper zone on F.Cu, net /Stepper Driver/Driver1/OB2
- added copper zone on In1.Cu, net /Stepper Driver/Driver1/OB2
- added copper zone on In2.Cu, net /Stepper Driver/Driver1/OB2
- added copper zone on F.Cu, net /Stepper Driver/Driver1/RSA
- added copper zone on F.Cu, net /Stepper Driver/Driver1/RSB
- added copper zone on B.Cu, net GND
- added copper zone on F.Cu, net GND
Other:
- copper layers 2 -> 4

Commit message: before copy
Routing:
- net GND: track 32.0 -> 37.5 mm, vias 78 -> 79
- net Net-(IC1-Pad3): track 0.94 -> 0.00 mm, vias 1 -> 0

Commit message: all driver
Parts:
- C112, C115, C116, C133, C136, C137, C154, C157, C158, C175, C178, C179, C187, C188, C189, C190: moved to B.Cu
- moved IC5 151.0 mm to (184.0, 63.9)
- moved D44 149.2 mm to (157.2, 52.7), turned to 90 degrees
- moved D50 148.9 mm to (142.8, 52.7), turned to 90 degrees
- moved C138 145.0 mm to (157.2, 55.1), turned to 270 degrees
- moved C143 144.3 mm to (142.8, 57.5), turned to 90 degrees
- moved IC4 143.5 mm to (167.0, 63.9)
- moved C141 143.4 mm to (142.8, 55.1), turned to 270 degrees
- moved C140 142.7 mm to (153.6, 57.5), turned to 270 degrees
- moved D46 142.1 mm to (147.6, 57.5), turned to 270 degrees
- moved C139 141.5 mm to (146.4, 57.5), turned to 270 degrees
- moved D58 141.5 mm to (159.8, 52.7), turned to 90 degrees
- moved C134 140.4 mm to (150.6, 57.5), turned to 270 degrees
- moved D45 140.3 mm to (145.2, 57.5), turned to 90 degrees
- moved D48 139.4 mm to (152.4, 57.5), turned to 270 degrees
- moved D49 139.3 mm to (144.0, 57.5), turned to 90 degrees
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Routing:
- net GND: track 37.5 -> 155.0 mm, vias 79 -> 395
- net +24V: track 18.1 -> 90.4 mm, vias 61 -> 305
- net /Stepper Driver/Driver5/RSB: track 0.00 -> 17.7 mm
- net /Stepper Driver/Driver4/RSB: track 0.00 -> 17.7 mm
- net /Stepper Driver/Driver3/RSB: track 0.00 -> 17.7 mm
- net /Stepper Driver/Driver2/RSB: track 0.00 -> 17.7 mm
- net /Stepper Driver/Driver5/RSA: track 0.00 -> 16.8 mm
- net /Stepper Driver/Driver4/RSA: track 0.00 -> 16.8 mm
- net /Stepper Driver/Driver3/RSA: track 0.00 -> 16.8 mm
- net /Stepper Driver/Driver2/RSA: track 0.00 -> 16.8 mm
- net /Stepper Driver/Driver2/OB1: track 0.00 -> 16.7 mm, vias 0 -> 59
- net /Stepper Driver/Driver5/OB1: track 0.00 -> 16.7 mm, vias 0 -> 59
- net /Stepper Driver/Driver4/OB1: track 0.00 -> 16.7 mm, vias 0 -> 59
- net /Stepper Driver/Driver3/OB1: track 0.00 -> 16.7 mm, vias 0 -> 59
- net /Stepper Driver/Driver5/OA2: track 0.00 -> 15.6 mm, vias 0 -> 59
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- added copper zone on B.Cu, net /Stepper Driver/Driver2/OA1
- added copper zone on F.Cu, net /Stepper Driver/Driver2/OA1
- added copper zone on In1.Cu, net /Stepper Driver/Driver2/OA1
- added copper zone on In2.Cu, net /Stepper Driver/Driver2/OA1
- added copper zone on B.Cu, net /Stepper Driver/Driver2/OA2
- added copper zone on F.Cu, net /Stepper Driver/Driver2/OA2
- added copper zone on In1.Cu, net /Stepper Driver/Driver2/OA2
- added copper zone on In2.Cu, net /Stepper Driver/Driver2/OA2
- added copper zone on B.Cu, net /Stepper Driver/Driver2/OB1
- added copper zone on F.Cu, net /Stepper Driver/Driver2/OB1
- added copper zone on In1.Cu, net /Stepper Driver/Driver2/OB1
- added copper zone on In2.Cu, net /Stepper Driver/Driver2/OB1
- added copper zone on B.Cu, net /Stepper Driver/Driver2/OB2
- added copper zone on F.Cu, net /Stepper Driver/Driver2/OB2
- added copper zone on In1.Cu, net /Stepper Driver/Driver2/OB2
- added copper zone on In2.Cu, net /Stepper Driver/Driver2/OB2
- added copper zone on F.Cu, net /Stepper Driver/Driver2/RSA
- added copper zone on F.Cu, net /Stepper Driver/Driver2/RSB
- added copper zone on B.Cu, net /Stepper Driver/Driver3/OA1
- added copper zone on F.Cu, net /Stepper Driver/Driver3/OA1
- added copper zone on In1.Cu, net /Stepper Driver/Driver3/OA1
- added copper zone on In2.Cu, net /Stepper Driver/Driver3/OA1
- added copper zone on B.Cu, net /Stepper Driver/Driver3/OA2
- added copper zone on F.Cu, net /Stepper Driver/Driver3/OA2
- added copper zone on In1.Cu, net /Stepper Driver/Driver3/OA2
- added copper zone on In2.Cu, net /Stepper Driver/Driver3/OA2
- added copper zone on B.Cu, net /Stepper Driver/Driver3/OB1
- added copper zone on F.Cu, net /Stepper Driver/Driver3/OB1
- added copper zone on In1.Cu, net /Stepper Driver/Driver3/OB1
- added copper zone on In2.Cu, net /Stepper Driver/Driver3/OB1
- added copper zone on B.Cu, net /Stepper Driver/Driver3/OB2
- added copper zone on F.Cu, net /Stepper Driver/Driver3/OB2
- added copper zone on In1.Cu, net /Stepper Driver/Driver3/OB2
- added copper zone on In2.Cu, net /Stepper Driver/Driver3/OB2
- added copper zone on F.Cu, net /Stepper Driver/Driver3/RSA
- added copper zone on F.Cu, net /Stepper Driver/Driver3/RSB
- added copper zone on B.Cu, net /Stepper Driver/Driver4/OA1
- added copper zone on F.Cu, net /Stepper Driver/Driver4/OA1
- added copper zone on In1.Cu, net /Stepper Driver/Driver4/OA1
- added copper zone on In2.Cu, net /Stepper Driver/Driver4/OA1
- added copper zone on B.Cu, net /Stepper Driver/Driver4/OA2
- added copper zone on F.Cu, net /Stepper Driver/Driver4/OA2
- added copper zone on In1.Cu, net /Stepper Driver/Driver4/OA2
- added copper zone on In2.Cu, net /Stepper Driver/Driver4/OA2
- added copper zone on B.Cu, net /Stepper Driver/Driver4/OB1
- added copper zone on F.Cu, net /Stepper Driver/Driver4/OB1
- added copper zone on In1.Cu, net /Stepper Driver/Driver4/OB1
- added copper zone on In2.Cu, net /Stepper Driver/Driver4/OB1
- added copper zone on B.Cu, net /Stepper Driver/Driver4/OB2
- added copper zone on F.Cu, net /Stepper Driver/Driver4/OB2
- added copper zone on In1.Cu, net /Stepper Driver/Driver4/OB2
- added copper zone on In2.Cu, net /Stepper Driver/Driver4/OB2
- added copper zone on F.Cu, net /Stepper Driver/Driver4/RSA
- added copper zone on F.Cu, net /Stepper Driver/Driver4/RSB
- added copper zone on B.Cu, net /Stepper Driver/Driver5/OA1
- added copper zone on F.Cu, net /Stepper Driver/Driver5/OA1
- added copper zone on In1.Cu, net /Stepper Driver/Driver5/OA1
- added copper zone on In2.Cu, net /Stepper Driver/Driver5/OA1
- added copper zone on B.Cu, net /Stepper Driver/Driver5/OA2
- added copper zone on F.Cu, net /Stepper Driver/Driver5/OA2
- added copper zone on In1.Cu, net /Stepper Driver/Driver5/OA2
- added copper zone on In2.Cu, net /Stepper Driver/Driver5/OA2
- added copper zone on B.Cu, net /Stepper Driver/Driver5/OB1
- added copper zone on F.Cu, net /Stepper Driver/Driver5/OB1
- added copper zone on In1.Cu, net /Stepper Driver/Driver5/OB1
- added copper zone on In2.Cu, net /Stepper Driver/Driver5/OB1
- added copper zone on B.Cu, net /Stepper Driver/Driver5/OB2
- added copper zone on F.Cu, net /Stepper Driver/Driver5/OB2
- added copper zone on In1.Cu, net /Stepper Driver/Driver5/OB2
- added copper zone on In2.Cu, net /Stepper Driver/Driver5/OB2
- added copper zone on F.Cu, net /Stepper Driver/Driver5/RSA
- added copper zone on F.Cu, net /Stepper Driver/Driver5/RSB

Commit message: driver polys
Parts:
- moved U1 180.5 mm to (232.8, 13.9)
- moved C13 178.5 mm to (259.5, 13.7)
- moved C3 178.5 mm to (257.5, 13.7)
- moved C33 178.5 mm to (272.8, -17.3)
- moved C4 178.5 mm to (257.5, 16.4)
- moved C41 178.5 mm to (272.8, -19.1)
- moved C8 178.5 mm to (257.5, 15.5)
- moved C9 178.5 mm to (257.5, 14.6)
- moved D3 178.5 mm to (272.8, -18.2)
- moved J54 178.5 mm to (268.7, -20.9)
- moved R1 178.5 mm to (257.5, 17.3)
- moved R2 178.5 mm to (259.5, 14.6)
- moved R5 178.5 mm to (259.5, 15.5)
- moved C1 178.5 mm to (245.0, 26.9)
- moved C10 178.5 mm to (260.2, 11.0)
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Connections:
- C67 pad 1: +24V -> DCIN+
- C67 pad 2: GND -> DCIN-
- C68 pad 2: GND -> DCIN-
- C69 pad 2: GND -> DCIN-
- C77 pad 1: +24V -> DCIN+
- C77 pad 2: GND -> DCIN-
- C78 pad 2: GND -> DCIN-
- C79 pad 2: GND -> DCIN-
- F1 pad 2: Net-(F1-Pad2) -> DCIN+
- F2 pad 1: +24V -> DCIN+
- F3 pad 1: +24V -> DCIN+
- F4 pad 1: +24V -> DCIN+
- F5 pad 1: +24V -> DCIN+
- J39 pad 1: Net-(J39-Pad1) -> DCIN-
- J39 pad 2: Net-(F1-Pad2) -> DCIN+
- Q1 pad 3: Net-(J39-Pad1) -> DCIN-
- Q11 pad 1: GND -> DCIN-
- Q14 pad 1: GND -> DCIN-
- Q6 pad 1: GND -> DCIN-
- Q7 pad 1: GND -> DCIN-
Routing:
- net GND: track 155.0 -> 179.8 mm, vias 395 -> 383
- net /Stepper Driver/Driver1/OB1: track 16.7 -> 39.7 mm
- net +24V: track 90.4 -> 96.6 mm, vias 305 -> 301
- net /Stepper Driver/Driver5/OB1: vias 59 -> 58
- net /Stepper Driver/Driver4/OB1: vias 59 -> 58
- net /Stepper Driver/Driver4/OA2: vias 59 -> 58
- net /Stepper Driver/Driver3/OB1: vias 59 -> 58
- net /Stepper Driver/Driver3/OA2: vias 59 -> 58
- net /Stepper Driver/Driver2/OB1: vias 59 -> 58
- net /Stepper Driver/Driver2/OA2: vias 59 -> 58
- net /Stepper Driver/Driver1/OA2: vias 59 -> 58
- added copper zone on In1.Cu, net GND
Other:
- outline, holes or cut-outs redrawn
- board text added: "DRV1"
- board text added: "DRV2"
- board text added: "DRV3"
- board text added: "DRV4"
- board text added: "DRV5"

Commit message: fuses
Parts:
- removed C1, C10, C11, C12, C13, C14, C15, C16, C45, C47, C52, C6, C8, C80: 100n, _Generic:0603_CAP
- removed C17, C2, C4, C46, C49, C58, C59, C60, C61, C7, C9: 10u, _Generic:0603_CAP
- removed C3, C5, C50, C51: 12p, _Generic:0603_CAP
- removed C48, C53: 22n, _Generic:0603_CAP
- removed C54, C55, C56, C57, C64, C65, C66, C70, C71, C72, C75, C76, C78: 4.7u, _Generic:0805_CAP
- removed D10, D15, D16, D17, D20, D21, D22, D23, D24, D7, D8, D9: 3.6v, _Generic:SOD-523_DIODE
- removed D11, D12, D13, D14: DNP, _Generic:SOD-523_DIODE
- removed D26: LED, _Generic:0603_LED
- removed F1, F2, F3, F4, F5: FUSE, _Generic:SMD_Fuseholder
- removed J1, J10, J11, J12, J13, J14, J15, J16, J17, J18, J19, J2, J20, J21, J22, J23, J24, J25, J26, J27, J28, J29, J3, J30, J31, J32, J33, J34, J35, J36, J37, J38, J4, J5, J6, J7, J75, J76, J77, J78, J8, J9: Conn_01x01, _Generic:PinHeader_2.54mm_1P
- removed J62, J63, J71, J72, J73, J74: Conn_01x02, _Generic:JST_XH_2P
- removed J64, J65, J70: Conn_01x04, _Generic:JST_XH_4P
- removed J66, J67, J68, J69, J79, J80, J81, J83, J84, J85, J86, J87: Conn_01x03, _Generic:JST_XH_3P
- removed L4, L5, L6, L7: 470, _Generic:0603_IND
- removed Q10, Q12, Q13, Q3, Q4, Q5, Q8, Q9: AO3400, _Generic:SOT-23
- removed Q14: AON6144, _Generic:DFN5x6-8
- removed Q2: AO3401, _Generic:SOT-23
- removed R1, R2, R27, R29, R30, R31, R79: 10k, _Generic:0603_RES
- removed R21, R22, R37, R38, R39, R40, R41, R42, R44, R46, R48, R50: 4.7k, _Generic:0603_RES
- removed R23, R34, R51, R52, R53, R54, R80: 0R, _Generic:0603_RES
- removed R24, R25: 47R, _Generic:0603_RES
- removed R26: 1.5k, _Generic:0603_RES
- removed R28, R56, R58, R60, R66, R68, R70, R72, R74: 50k, _Generic:0603_RES
- removed R3, R4, R5, R55, R57, R59, R65, R67, R69, R71, R73, R78: 1k, _Generic:0603_RES
- removed R32, R33, R35, R36: 47k, _Generic:0603_RES
- removed R43, R45, R47, R49: DNP, _Generic:0603_RES
- removed R6, R7: 2.2R, _Generic:0603_RES
- removed U5, U6: MAX6675, _Generic:SO-8
- removed X1: 12MHz, Oscillator:Oscillator_SMD_EuroQuartz_XO32-4Pin_3.2x2.5mm
- C67, C77: value 68u -> 220u; footprint Capacitor_SMD:CP_Elec_8x10 -> Capacitor_SMD:CP_Elec_6.3x7.7
- C68, C69: footprint _Generic:0805_CAP -> _Generic:1210_CAP; moved to B.Cu
- C79: footprint _Generic:0805_CAP -> _Generic:1210_CAP
- J88: value Screw_Terminal_01x04 -> Screw_Terminal_01x02; footprint _Generic:KF635-4P -> _Generic:KF635-2P
- moved C44 185.8 mm to (145.8, 133.6)
- moved C33 181.2 mm to (180.2, 138.5)
- moved C41 181.2 mm to (180.2, 136.7)
- moved J41 181.2 mm to (178.7, 134.9)
- moved J46 181.2 mm to (166.4, 142.0)
- moved J49 181.2 mm to (160.9, 152.2)
- moved J54 181.2 mm to (176.1, 134.9)
- moved C18 181.2 mm to (176.0, 141.9)
- moved C20 181.2 mm to (181.0, 135.4)
- moved C21 181.2 mm to (151.6, 153.3)
- moved C23 181.2 mm to (159.5, 144.8)
- moved C24 181.2 mm to (181.3, 134.3)
- moved C25 181.2 mm to (142.3, 153.2)
- moved C26 181.2 mm to (162.0, 144.8)
- moved C27 181.2 mm to (169.3, 135.5)
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Connections:
- net /P3.26_POW renamed /P3.26_BUZ
- C67 pad 1: DCIN+ -> +24V
- C68 pad 1: Net-(C68-Pad1) -> +24V
- C69 pad 1: Net-(C69-Pad1) -> +24V
- C77 pad 1: DCIN+ -> Net-(C77-Pad1)
- C79 pad 1: Net-(C79-Pad1) -> +24V
- D25 pad 1: Net-(D25-Pad1) -> Net-(C77-Pad1)
- J39 pad 2: DCIN+ -> +24V
- J82 pad 1: Net-(C69-Pad1) -> Net-(D18-Pad1)
- J82 pad 2: Net-(D18-Pad1) -> +24V
- J82 pad 3: Net-(C68-Pad1) -> Net-(D19-Pad1)
- J82 pad 4: Net-(D19-Pad1) -> +24V
- J88 pad 1: Net-(C79-Pad1) -> Net-(C77-Pad1)
- J88 pad 2: Net-(D25-Pad1) -> +24V
- Q11 pad 3: Net-(D25-Pad1) -> Net-(C77-Pad1)
- R61 pad 1: Net-(Q6-Pad2) -> Net-(Q7-Pad2)
- R62 pad 1: Net-(Q7-Pad2) -> Net-(Q6-Pad2)
- U1 pad 32: /P1.18_POW -> /P1.18_ADV
- U1 pad 33: /P1.19_POW -> /P1.19_ADV
- U1 pad 69: /P2.4_ADV -> /P2.4_POW
- U1 pad 70: /P2.3_ADV -> /P2.3_POW
- U7 pad 2: /P1.18_POW -> /P2.3_POW
- U7 pad 4: /P1.19_POW -> /P2.4_POW
Routing:
- net +24V: track 96.6 -> 96.2 mm, vias 301 -> 300
- added copper zone on In1.Cu, net +24V
- added copper zone on In2.Cu, net +24V
- added copper zone on F.Cu, net Net-(C77-Pad1)
- added copper zone on F.Cu, net Net-(D18-Pad1)
- added copper zone on F.Cu, net Net-(D19-Pad1)
- removed copper zone on B.Cu, net GND
