File: hardware/kajikia/kajikia.kicad_pcb (KiCad board)
At the start: 4 copper layers, 100 x 75 mm, 310 parts, among them IC1 TMC5161, IC2 TMC5161, IC3 TMC5161, IC4 TMC5161, IC5 TMC5161, J39 Screw_Terminal_01x02, J40 Conn_01x01, J41 Conn_01x01, J42 Conn_01x01, J43 Conn_01x01, J44 Conn_01x01, J45 Conn_01x01, J46 Conn_01x01, J47 Conn_01x01, J48 Conn_01x01, J49 Conn_01x01, J50 Conn_01x01, J51 Conn_01x01, J52 Conn_01x01, J53 Conn_01x01, J54 Conn_01x01, J55 Conn_01x01, J56 Conn_01x01, J57 Conn_01x01, J58 Conn_01x01, J59 Conn_01x01, J82 Screw_Terminal_01x04, J88 Screw_Terminal_01x02, J89 Conn_01x04, J90 Conn_01x04, J91 Conn_01x04, J92 Conn_01x04, J93 Conn_01x04, Q1 AON6144, Q11 AON6144, Q6 AON6144, Q7 AON6144, U1 LPC1769FBD100, U2 LM1117-3.3, U3 AOZ1284, U4 AOZ1284, U7 IR4427S, U8 IR4427S

Commit message: continue routing
Parts:
- removed J46, J47, J49, J50, J52, J53: Conn_01x01, _Generic:PinHeader_2.54mm_1P
- added C1: 100n, _Generic:0603_CAP, F.Cu at (327.0, 185.2)
- added C10: 100n, _Generic:0603_CAP, F.Cu at (266.6, 103.6)
- added C11: 100n, _Generic:0603_CAP, F.Cu at (266.6, 102.7)
- added C12: 100n, _Generic:0603_CAP, F.Cu at (269.2, 100.1)
- added C13: 100n, _Generic:0603_CAP, F.Cu at (269.2, 99.2)
- added C14: 100n, _Generic:0603_CAP, F.Cu at (323.0, 184.8)
- added C15: 100n, _Generic:0603_CAP, F.Cu at (274.5, 95.7)
- added C16: 100n, _Generic:0603_CAP, F.Cu at (325.0, 184.3)
- added C17: 10u, _Generic:0603_CAP, F.Cu at (271.2, 99.2)
- added C191: 220u, Capacitor_SMD:CP_Elec_6.3x7.7, F.Cu at (127.5, 81.9)
- added C192: 4.7u, _Generic:1210_CAP, B.Cu at (118.7, 108.8)
- added C193: 220u, Capacitor_SMD:CP_Elec_6.3x7.7, F.Cu at (127.5, 120.0)
- added C194: 4.7u, _Generic:1210_CAP, B.Cu at (138.9, 114.3)
- added C195: 4.7u, _Generic:1210_CAP, B.Cu at (144.9, 95.3)
- added C196: 4.7u, _Generic:1210_CAP, B.Cu at (141.9, 114.3)
- added C197: 4.7u, _Generic:1210_CAP, B.Cu at (138.9, 95.3)
- added C198: 4.7u, _Generic:1210_CAP, F.Cu at (281.8, 94.7)
- added C199: 4.7u, _Generic:1210_CAP, F.Cu at (285.8, 92.1)
- added C2: 10u, _Generic:0603_CAP, F.Cu at (273.9, 96.6)
- added C3: 12p, _Generic:0603_CAP, F.Cu at (270.6, 101.0)
- added C4: 10u, _Generic:0603_CAP, F.Cu at (330.2, 183.5)
- added C45: 100n, _Generic:0603_CAP, F.Cu at (189.2, 78.6)
- added C46: 10u, _Generic:0603_CAP, F.Cu at (310.6, 139.2)
- added C47: 100n, _Generic:0603_CAP, F.Cu at (291.2, 158.1)
- added C48: 22n, _Generic:0603_CAP, F.Cu at (191.4, 73.8)
- added C49: 10u, _Generic:0603_CAP, F.Cu at (295.6, 152.9)
- added C5: 12p, _Generic:0603_CAP, F.Cu at (268.6, 101.8)
- added C50: 12p, _Generic:0603_CAP, F.Cu at (310.9, 136.5)
- added C51: 12p, _Generic:0603_CAP, F.Cu at (295.6, 152.0)
- added C52: 100n, _Generic:0603_CAP, F.Cu at (189.2, 80.2)
- added C53: 22n, _Generic:0603_CAP, F.Cu at (191.4, 82.2)
- added C54: 4.7u, _Generic:0805_CAP, F.Cu at (277.5, 159.8)
- added C55: 4.7u, _Generic:0805_CAP, F.Cu at (275.0, 159.8)
- added C56: 4.7u, _Generic:0805_CAP, F.Cu at (280.0, 159.8)
- added C57: 4.7u, _Generic:0805_CAP, F.Cu at (272.5, 159.8)
- added C58: 10u, _Generic:0603_CAP, F.Cu at (297.6, 151.1)
- added C59: 10u, _Generic:0603_CAP, F.Cu at (299.6, 150.4)
- added C6: 100n, _Generic:0603_CAP, F.Cu at (271.9, 96.5)
- added C60: 10u, _Generic:0603_CAP, F.Cu at (302.3, 147.0)
- added C61: 10u, _Generic:0603_CAP, F.Cu at (293.8, 155.6)
- added C64: 4.7u, _Generic:0805_CAP, F.Cu at (133.8, 151.4)
- added C65: 4.7u, _Generic:0805_CAP, F.Cu at (131.3, 151.4)
- added C66: 4.7u, _Generic:0805_CAP, F.Cu at (126.3, 151.4)
- added C7: 10u, _Generic:0603_CAP, F.Cu at (274.5, 93.9)
- added C70: 4.7u, _Generic:0805_CAP, F.Cu at (128.8, 151.4)
- added C71: 4.7u, _Generic:0805_CAP, F.Cu at (136.3, 151.4)
- added C72: 4.7u, _Generic:0805_CAP, F.Cu at (138.8, 151.4)
- added C75: 4.7u, _Generic:0805_CAP, F.Cu at (141.3, 151.4)
- added C76: 4.7u, _Generic:0805_CAP, F.Cu at (143.8, 151.4)
- added C78: 220u, Capacitor_SMD:CP_Elec_6.3x7.7, F.Cu at (118.1, 81.9)
- added C8: 100n, _Generic:0603_CAP, F.Cu at (271.9, 97.4)
- added C80: 100n, _Generic:0603_CAP, F.Cu at (353.3, 158.1)
- added C9: 10u, _Generic:0603_CAP, F.Cu at (274.5, 94.8)
- added D10: 3.6v, _Generic:SOD-523_DIODE, F.Cu at (291.8, 154.6)
- added D11: DNP, _Generic:SOD-523_DIODE, F.Cu at (308.9, 137.4)
- added D12: DNP, _Generic:SOD-523_DIODE, F.Cu at (289.2, 158.1)
- added D13: DNP, _Generic:SOD-523_DIODE, F.Cu at (308.9, 138.3)
- added D14: DNP, _Generic:SOD-523_DIODE, F.Cu at (295.6, 151.1)
- added D15: 3.6v, _Generic:SOD-523_DIODE, F.Cu at (158.9, 140.4)
- added D16: 3.6v, _Generic:SOD-523_DIODE, F.Cu at (164.3, 133.5)
- added D17: 3.6v, _Generic:SOD-523_DIODE, F.Cu at (148.0, 150.8)
- added D20: 3.6v, _Generic:SOD-523_DIODE, F.Cu at (153.3, 144.4)
- added D21: 3.6v, _Generic:SOD-523_DIODE, F.Cu at (144.0, 152.6)
- added D22: 3.6v, _Generic:SOD-523_DIODE, F.Cu at (164.3, 131.7)
- added D23: 3.6v, _Generic:SOD-523_DIODE, F.Cu at (164.3, 132.6)
- added D24: 3.6v, _Generic:SOD-523_DIODE, F.Cu at (146.0, 151.2)
- added D26: MSK4010, _Generic:SOD-523_DIODE, F.Cu at (146.0, 152.1)
- added D7: 3.6v, _Generic:SOD-523_DIODE, F.Cu at (310.9, 138.3)
- added D8: 3.6v, _Generic:SOD-523_DIODE, F.Cu at (291.8, 153.7)
- added D9: 3.6v, _Generic:SOD-523_DIODE, F.Cu at (311.6, 134.2)
- added F1: Fuse, _Generic:SMD_Fuseholder, F.Cu at (118.9, 75.6)
- added F2: Fuse, _Generic:SMD_Fuseholder, F.Cu at (118.9, 88.3)
- added F3: Fuse, _Generic:SMD_Fuseholder, F.Cu at (118.9, 101.0)
- added F4: Fuse, _Generic:SMD_Fuseholder, F.Cu at (118.9, 113.7)
- added J1: Conn_01x01, _Generic:PinHeader_2.54mm_1P, F.Cu at (261.6, 92.1)
- added J10: Conn_01x01, _Generic:PinHeader_2.54mm_1P, F.Cu at (319.9, 183.0)
- added J11: Conn_01x01, _Generic:PinHeader_2.54mm_1P, F.Cu at (261.6, 102.7)
- added J12: Conn_01x01, _Generic:PinHeader_2.54mm_1P, F.Cu at (264.3, 94.8)
- added J13: Conn_01x01, _Generic:PinHeader_2.54mm_1P, F.Cu at (266.9, 92.1)
- added J14: Conn_01x01, _Generic:PinHeader_2.54mm_1P, F.Cu at (259.0, 102.7)
- added J15: Conn_01x01, _Generic:PinHeader_2.54mm_1P, F.Cu at (261.6, 100.0)
- added J16: Conn_01x01, _Generic:PinHeader_2.54mm_1P, F.Cu at (259.0, 94.8)
- added J17: Conn_01x01, _Generic:PinHeader_2.54mm_1P, F.Cu at (256.4, 97.4)
- added J18: Conn_01x01, _Generic:PinHeader_2.54mm_1P, F.Cu at (143.0, 77.4)
- added J19: Conn_01x01, _Generic:PinHeader_2.54mm_1P, F.Cu at (148.2, 77.4)
- added J2: Conn_01x01, _Generic:PinHeader_2.54mm_1P, F.Cu at (261.6, 97.4)
- added J20: Conn_01x01, _Generic:PinHeader_2.54mm_1P, F.Cu at (145.6, 77.4)
- added J21: Conn_01x01, _Generic:PinHeader_2.54mm_1P, F.Cu at (143.0, 80.0)
- added J22: Conn_01x01, _Generic:PinHeader_2.54mm_1P, F.Cu at (148.2, 80.0)
- added J23: Conn_01x01, _Generic:PinHeader_2.54mm_1P, F.Cu at (145.6, 80.0)
- added J24: Conn_01x01, _Generic:PinHeader_2.54mm_1P, F.Cu at (259.0, 97.4)
- added J25: Conn_01x01, _Generic:PinHeader_2.54mm_1P, F.Cu at (253.7, 92.1)
- added J26: Conn_01x01, _Generic:PinHeader_2.54mm_1P, F.Cu at (322.6, 183.0)
- added J27: Conn_01x01, _Generic:PinHeader_2.54mm_1P, F.Cu at (158.0, 94.4)
- added J28: Conn_01x01, _Generic:PinHeader_2.54mm_1P, F.Cu at (160.6, 94.4)
- added J29: Conn_01x01, _Generic:PinHeader_2.54mm_1P, F.Cu at (163.2, 94.4)
- added J3: Conn_01x01, _Generic:PinHeader_2.54mm_1P, F.Cu at (145.6, 74.8)
- added J30: Conn_01x01, _Generic:PinHeader_2.54mm_1P, F.Cu at (155.4, 94.4)
- added J31: Conn_01x01, _Generic:PinHeader_2.54mm_1P, F.Cu at (269.6, 97.4)
- added J32: Conn_01x01, _Generic:PinHeader_2.54mm_1P, F.Cu at (266.9, 100.0)
- added J33: Conn_01x01, _Generic:PinHeader_2.54mm_1P, F.Cu at (264.3, 102.7)
- added J34: Conn_01x01, _Generic:PinHeader_2.54mm_1P, F.Cu at (272.2, 92.1)
- added J35: Conn_01x01, _Generic:PinHeader_2.54mm_1P, F.Cu at (269.6, 94.8)
- added J36: Conn_01x01, _Generic:PinHeader_2.54mm_1P, F.Cu at (266.9, 97.4)
- added J37: Conn_01x01, _Generic:PinHeader_2.54mm_1P, F.Cu at (317.3, 183.0)
- added J38: Conn_01x01, _Generic:PinHeader_2.54mm_1P, F.Cu at (264.3, 100.0)
- added J4: Conn_01x01, _Generic:PinHeader_2.54mm_1P, F.Cu at (148.2, 74.8)
- added J5: Conn_01x01, _Generic:PinHeader_2.54mm_1P, F.Cu at (256.4, 94.8)
- added J6: Conn_01x01, _Generic:PinHeader_2.54mm_1P, F.Cu at (266.9, 94.8)
- added J60: USB_C_Receptacle, _Generic:TYPE-C-31-M-12, F.Cu at (197.6, 96.2)
- added J62: Conn_01x02, _Generic:JST_XH_2P, F.Cu at (197.2, 75.6)
- added J63: Conn_01x02, _Generic:JST_XH_2P, F.Cu at (197.2, 83.6)
- added J64: Conn_01x04, _Generic:JST_XH_4P, F.Cu at (196.0, 111.0)
- added J65: Conn_01x04, _Generic:JST_XH_4P, F.Cu at (189.5, 111.0)
- added J66: Conn_01x03, _Generic:JST_XH_3P, F.Cu at (157.0, 120.0)
- added J67: Conn_01x03, _Generic:JST_XH_3P, F.Cu at (163.5, 120.0)
- added J68: Conn_01x03, _Generic:JST_XH_3P, F.Cu at (170.0, 120.0)
- added J69: Conn_01x03, _Generic:JST_XH_3P, F.Cu at (150.5, 120.0)
- added J7: Conn_01x01, _Generic:PinHeader_2.54mm_1P, F.Cu at (253.7, 97.4)
- added J71: Conn_01x02, _Generic:JST_XH_2P, F.Cu at (150.5, 100.0)
- added J72: Conn_01x02, _Generic:JST_XH_2P, F.Cu at (157.0, 100.0)
- added J73: Conn_01x02, _Generic:JST_XH_2P, F.Cu at (163.5, 100.0)
- added J74: Conn_01x02, _Generic:JST_XH_2P, F.Cu at (170.0, 100.0)
- added J75: Conn_01x01, _Generic:PinHeader_2.54mm_1P, F.Cu at (293.3, 152.0)
- added J76: Conn_01x01, _Generic:PinHeader_2.54mm_1P, F.Cu at (289.5, 156.3)
- added J77: Conn_01x01, _Generic:PinHeader_2.54mm_1P, F.Cu at (289.5, 153.7)
- added J78: Conn_01x01, _Generic:PinHeader_2.54mm_1P, F.Cu at (299.9, 146.9)
- added J79: Conn_01x03, _Generic:JST_XH_3P, F.Cu at (170.0, 109.5)
- added J8: Conn_01x01, _Generic:PinHeader_2.54mm_1P, F.Cu at (253.7, 94.8)
- added J80: Conn_01x03, _Generic:JST_XH_3P, F.Cu at (157.0, 109.5)
- added J81: Conn_01x03, _Generic:JST_XH_3P, F.Cu at (176.5, 120.0)
- added J83: Conn_01x03, _Generic:JST_XH_3P, F.Cu at (163.5, 109.5)
- added J84: Conn_01x03, _Generic:JST_XH_3P, F.Cu at (150.5, 109.5)
- added J85: Conn_01x03, _Generic:JST_XH_3P, F.Cu at (183.0, 120.0)
- added J86: Conn_01x03, _Generic:JST_XH_3P, F.Cu at (176.5, 109.5)
- added J87: Conn_01x03, _Generic:JST_XH_3P, F.Cu at (183.0, 109.5)
- added J9: Conn_01x01, _Generic:PinHeader_2.54mm_1P, F.Cu at (259.0, 100.0)
- added JP1: SolderJumper_2_Open, _Generic:Solder Jumper 2P, F.Cu at (268.7, 100.9)
- added JP10: SolderJumper_2_Open, _Generic:Solder Jumper 2P, F.Cu at (329.5, 185.1)
- added JP11: SolderJumper_2_Open, _Generic:Solder Jumper 2P, F.Cu at (268.1, 103.6)
- added JP12: SolderJumper_2_Open, _Generic:Solder Jumper 2P, F.Cu at (271.4, 98.3)
- added JP13: SolderJumper_2_Open, _Generic:Solder Jumper 2P, F.Cu at (273.4, 98.2)
- added JP14: SolderJumper_2_Open, _Generic:Solder Jumper 2P, F.Cu at (134.9, 157.4)
- added JP15: SolderJumper_2_Open, _Generic:Solder Jumper 2P, F.Cu at (291.3, 152.8)
- added JP16: SolderJumper_3_Open, _Generic:Solder Jumper 3P, F.Cu at (282.1, 160.5)
- added JP18: SolderJumper_2_Open, _Generic:Solder Jumper 2P, F.Cu at (283.4, 160.5)
- added JP19: SolderJumper_2_Open, _Generic:Solder Jumper 2P, F.Cu at (284.4, 160.5)
- added JP2: SolderJumper_2_Open, _Generic:Solder Jumper 2P, F.Cu at (276.0, 93.8)
- added JP20: SolderJumper_2_Open, _Generic:Solder Jumper 2P, F.Cu at (285.4, 160.5)
- added JP21: SolderJumper_2_Open, _Generic:Solder Jumper 2P, F.Cu at (286.4, 160.5)
- added JP22: SolderJumper_3_Open, _Generic:Solder Jumper 3P, F.Cu at (153.1, 146.2)
- added JP23: SolderJumper_3_Open, _Generic:Solder Jumper 3P, F.Cu at (155.1, 145.2)
- added JP24: SolderJumper_3_Open, _Generic:Solder Jumper 3P, F.Cu at (153.1, 147.0)
- added JP28: SolderJumper_3_Open, _Generic:Solder Jumper 3P, F.Cu at (155.1, 144.4)
- added JP29: SolderJumper_3_Open, _Generic:Solder Jumper 3P, F.Cu at (158.7, 141.3)
- added JP3: SolderJumper_2_Open, _Generic:Solder Jumper 2P, F.Cu at (330.5, 184.3)
- added JP30: SolderJumper_3_Open, _Generic:Solder Jumper 3P, F.Cu at (147.8, 152.6)
- added JP34: SolderJumper_3_Open, _Generic:Solder Jumper 3P, F.Cu at (164.1, 135.3)
- added JP35: SolderJumper_3_Open, _Generic:Solder Jumper 3P, F.Cu at (160.7, 140.4)
- added JP38: SolderJumper_2_Open, _Generic:Solder Jumper 2P, F.Cu at (316.5, 159.0)
- added JP39: SolderJumper_2_Open, _Generic:Solder Jumper 2P, F.Cu at (168.9, 131.7)
- added JP4: SolderJumper_2_Open, _Generic:Solder Jumper 2P, F.Cu at (276.0, 94.6)
- added JP40: SolderJumper_2_Open, _Generic:Solder Jumper 2P, F.Cu at (322.7, 159.0)
- added JP41: SolderJumper_2_Open, _Generic:Solder Jumper 2P, F.Cu at (328.8, 159.0)
- added JP42: SolderJumper_2_Open, _Generic:Solder Jumper 2P, F.Cu at (335.0, 159.0)
- added JP5: SolderJumper_2_Open, _Generic:Solder Jumper 2P, F.Cu at (272.4, 98.3)
- added JP6: SolderJumper_2_Open, _Generic:Solder Jumper 2P, F.Cu at (273.4, 97.4)
- added JP7: SolderJumper_2_Open, _Generic:Solder Jumper 2P, F.Cu at (329.5, 184.3)
- added JP8: SolderJumper_2_Open, _Generic:Solder Jumper 2P, F.Cu at (328.5, 185.1)
- added JP9: SolderJumper_2_Open, _Generic:Solder Jumper 2P, F.Cu at (328.5, 184.3)
- added L4: 470, _Generic:0603_IND, F.Cu at (192.8, 73.8)
- added L5: 470, _Generic:0603_IND, F.Cu at (192.8, 76.6)
- added L6: 470, _Generic:0603_IND, F.Cu at (192.8, 82.2)
- added L7: 470, _Generic:0603_IND, F.Cu at (192.8, 85.0)
- added Q10: AO3400, _Generic:SOT-23, F.Cu at (151.0, 145.6)
- added Q12: AO3400, _Generic:SOT-23, F.Cu at (148.3, 148.8)
- added Q13: AO3400, _Generic:SOT-23, F.Cu at (161.9, 135.2)
- added Q14: AO3400, _Generic:SOT-23, F.Cu at (159.2, 138.4)
- added Q2: AO3401, _Generic:SOT-23, F.Cu at (309.3, 133.6)
- added Q3: AO3400, _Generic:SOT-23, F.Cu at (161.9, 132.0)
- added Q4: AO3400, _Generic:SOT-23, F.Cu at (159.2, 132.0)
- added Q5: AO3400, _Generic:SOT-23, F.Cu at (148.3, 145.6)
- added Q8: AO3400, _Generic:SOT-23, F.Cu at (151.0, 148.8)
- added Q9: AO3400, _Generic:SOT-23, F.Cu at (159.2, 135.2)
- added R1: 10k, _Generic:0603_RES, F.Cu at (268.6, 102.7)
- added R2: 10k, _Generic:0603_RES, F.Cu at (317.0, 184.8)
- added R21: 4.7k, _Generic:0603_RES, F.Cu at (291.8, 155.5)
- added R22: 4.7k, _Generic:0603_RES, F.Cu at (284.3, 159.6)
- added R23: 0R, _Generic:0603_RES, F.Cu at (191.4, 76.6)
- added R24: 47R, _Generic:0603_RES, F.Cu at (301.6, 148.8)
- added R25: 47R, _Generic:0603_RES, F.Cu at (293.2, 158.3)
- added R26: 1.5k, _Generic:0603_RES, F.Cu at (293.2, 157.4)
- added R27: 10k, _Generic:0603_RES, F.Cu at (310.6, 140.1)
- added R28: 50k, _Generic:0603_RES, F.Cu at (290.3, 159.9)
- added R29: 10k, _Generic:0603_RES, F.Cu at (302.3, 147.9)
- added R3: 1k, _Generic:0603_RES, F.Cu at (321.0, 184.8)
- added R30: 10k, _Generic:0603_RES, F.Cu at (295.8, 154.7)
- added R31: 10k, _Generic:0603_RES, F.Cu at (297.6, 152.9)
- added R32: 47k, _Generic:0603_RES, F.Cu at (303.9, 144.3)
- added R33: 47k, _Generic:0603_RES, F.Cu at (297.6, 152.0)
- added R34: 0R, _Generic:0603_RES, F.Cu at (191.4, 85.0)
- added R35: 47k, _Generic:0603_RES, F.Cu at (288.3, 159.9)
- added R36: 47k, _Generic:0603_RES, F.Cu at (307.9, 144.3)
- added R37: 4.7k, _Generic:0603_RES, F.Cu at (293.8, 154.7)
- added R38: 4.7k, _Generic:0603_RES, F.Cu at (282.3, 159.6)
- added R39: 4.7k, _Generic:0603_RES, F.Cu at (308.9, 136.5)
- added R4: 1k, _Generic:0603_RES, F.Cu at (319.0, 184.8)
- added R40: 4.7k, _Generic:0603_RES, F.Cu at (308.9, 135.6)
- added R41: 4.7k, _Generic:0603_RES, F.Cu at (311.6, 133.3)
- added R42: 4.7k, _Generic:0603_RES, F.Cu at (286.3, 159.6)
- added R43: DNP, _Generic:0603_RES, F.Cu at (310.9, 135.6)
- added R44: 4.7k, _Generic:0603_RES, F.Cu at (304.3, 146.1)
- added R45: DNP, _Generic:0603_RES, F.Cu at (295.8, 153.8)
- added R46: 4.7k, _Generic:0603_RES, F.Cu at (291.2, 159.0)
- added R47: DNP, _Generic:0603_RES, F.Cu at (305.9, 144.3)
- added R48: 4.7k, _Generic:0603_RES, F.Cu at (299.6, 148.6)
- added R49: DNP, _Generic:0603_RES, F.Cu at (291.8, 156.4)
- added R5: 1k, _Generic:0603_RES, F.Cu at (266.6, 101.8)
- added R50: 4.7k, _Generic:0603_RES, F.Cu at (304.3, 147.0)
- added R51: 0R, _Generic:0603_RES, F.Cu at (305.9, 145.2)
- added R52: 0R, _Generic:0603_RES, F.Cu at (297.8, 153.8)
- added R53: 0R, _Generic:0603_RES, F.Cu at (299.6, 151.3)
- added R54: 0R, _Generic:0603_RES, F.Cu at (310.6, 141.0)
- added R55: 1k, _Generic:0603_RES, F.Cu at (164.3, 134.4)
- added R56: 50k, _Generic:0603_RES, F.Cu at (148.0, 151.7)
- added R57: 1k, _Generic:0603_RES, F.Cu at (164.3, 130.8)
- added R58: 50k, _Generic:0603_RES, F.Cu at (140.0, 152.6)
- added R59: 1k, _Generic:0603_RES, F.Cu at (136.0, 152.6)
- added R6: 2.2R, _Generic:0603_RES, F.Cu at (325.0, 185.2)
- added R60: 50k, _Generic:0603_RES, F.Cu at (150.0, 150.8)
- added R65: 1k, _Generic:0603_RES, F.Cu at (161.6, 137.2)
- added R66: 50k, _Generic:0603_RES, F.Cu at (163.6, 137.2)
- added R67: 1k, _Generic:0603_RES, F.Cu at (134.0, 152.6)
- added R68: 50k, _Generic:0603_RES, F.Cu at (161.6, 138.1)
- added R69: 1k, _Generic:0603_RES, F.Cu at (132.0, 152.6)
- added R7: 2.2R, _Generic:0603_RES, F.Cu at (327.0, 184.3)
- added R70: 50k, _Generic:0603_RES, F.Cu at (130.0, 152.6)
- added R71: 1k, _Generic:0603_RES, F.Cu at (128.0, 152.6)
- added R72: 50k, _Generic:0603_RES, F.Cu at (142.0, 152.6)
- added R73: 1k, _Generic:0603_RES, F.Cu at (153.3, 145.3)
- added R74: 50k, _Generic:0603_RES, F.Cu at (161.6, 139.0)
- added R78: 0R, _Generic:0603_RES, F.Cu at (126.0, 152.6)
- added R79: 10k, _Generic:0603_RES, F.Cu at (353.3, 159.9)
- added R80: 0R, _Generic:0603_RES, F.Cu at (353.3, 159.0)
- added SW1: 3x6mm, Button_Switch_SMD:SW_SPST_CK_RS282G05A3, F.Cu at (172.7, 162.6)
- added SW2: 3x6mm, Button_Switch_SMD:SW_SPST_CK_RS282G05A3, F.Cu at (186.1, 157.6)
- added U5: MAX6675, _Generic:SO-8, F.Cu at (187.2, 75.2)
- added U6: MAX6675, _Generic:SO-8, F.Cu at (187.2, 83.6)
- added X1: 12MHz, Oscillator:Oscillator_SMD_EuroQuartz_XO32-4Pin_3.2x2.5mm, F.Cu at (350.4, 159.2)
- C23, C24, C25, C27, C28, C32: footprint _Generic:0805_CAP -> _Generic:1210_CAP; moved to B.Cu
- C26, C31: footprint _Generic:0805_CAP -> _Generic:1210_CAP
- C41, C42: value 10u -> 4.7u; footprint _Generic:0603_CAP -> _Generic:1210_CAP; moved to B.Cu
- C43, C44: value 390u -> 220u; footprint Capacitor_SMD:CP_Elec_8x10 -> Capacitor_SMD:CP_Elec_6.3x7.7
- C79: moved to B.Cu
- R76: value 10R -> 1k
- moved R101 189.9 mm to (323.2, 158.1)
- moved R83 187.9 mm to (317.0, 158.1)
- moved R110 180.2 mm to (329.3, 158.1)
- moved R119 170.6 mm to (335.5, 158.1)
- moved C31 131.2 mm to (285.8, 94.7)
- moved C26 130.9 mm to (281.8, 92.1)
- moved C19 95.3 mm to (121.3, 156.7)
- moved C21 71.0 mm to (141.2, 83.1), turned to 270 degrees
- moved J41 70.4 mm to (123.9, 179.1)
- moved D4 69.4 mm to (145.4, 86.0), turned to 270 degrees
- moved R14 68.7 mm to (144.0, 83.1), turned to 270 degrees
- moved C22 68.4 mm to (142.6, 83.1), turned to 270 degrees
- moved L1 67.3 mm to (142.4, 86.0), turned to 90 degrees
- moved J42 66.8 mm to (109.4, 182.9)
- moved J48 64.5 mm to (145.0, 89.0)
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Connections:
- C77 pad 1: Net-(C77-Pad1) -> +24V
- D25 pad 1: Net-(C77-Pad1) -> Net-(D25-Pad1)
- J82 pad 1: Net-(D18-Pad1) -> Net-(F2-Pad1)
- J82 pad 3: Net-(D19-Pad1) -> Net-(F3-Pad1)
- J88 pad 1: Net-(C77-Pad1) -> Net-(F4-Pad1)
- Q1 pad 3: DCIN- -> Net-(F1-Pad1)
- Q11 pad 3: Net-(C77-Pad1) -> Net-(D25-Pad1)
- R76 pad 2: Net-(R76-Pad2) -> /P3.26_BUZ
- U3 pad 9: (no net) -> +24V
- U4 pad 9: (no net) -> +24V
- U8 pad 4: /P3.26_BUZ -> Net-(U8-Pad4)
- U8 pad 5: Net-(R76-Pad2) -> Net-(U8-Pad5)
Routing:
- net +12V: track 0.00 -> 10.1 mm
- net Net-(D19-Pad1): track 0.00 -> 6.62 mm, vias 0 -> 60
- net Net-(D25-Pad1): track 0.00 -> 5.28 mm, vias 0 -> 60
- net Net-(D18-Pad1): track 0.00 -> 5.10 mm, vias 0 -> 60
- net Net-(R61-Pad2): track 0.00 -> 3.96 mm
- net Net-(R75-Pad2): track 0.00 -> 3.84 mm
- net Net-(R62-Pad2): track 0.00 -> 3.65 mm
- net GND: track 179.8 -> 182.4 mm
- net Net-(D18-Pad2): track 0.00 -> 1.27 mm
- net Net-(D25-Pad2): track 0.00 -> 1.27 mm
- net Net-(D19-Pad2): track 0.00 -> 1.14 mm
- net Net-(F4-Pad1): vias 0 -> 42
- net Net-(F3-Pad1): vias 0 -> 42
- net Net-(F2-Pad1): vias 0 -> 42
- net Net-(F1-Pad1): vias 0 -> 8
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- added copper zone on B.Cu, net DCIN-
- added copper zone on F.Cu, net DCIN-
- added copper zone on B.Cu, net Net-(D18-Pad1)
- added copper zone on B.Cu, net Net-(D19-Pad1)
- added copper zone on B.Cu, net Net-(D25-Pad1)
- added copper zone on F.Cu, net Net-(D25-Pad1)
- added copper zone on B.Cu, net Net-(F1-Pad1)
- added copper zone on F.Cu, net Net-(F1-Pad1)
- added copper zone on B.Cu, net Net-(F2-Pad1)
- added copper zone on F.Cu, net Net-(F2-Pad1)
- added copper zone on B.Cu, net Net-(F3-Pad1)
- added copper zone on F.Cu, net Net-(F3-Pad1)
- added copper zone on B.Cu, net Net-(F4-Pad1)
- added copper zone on F.Cu, net Net-(F4-Pad1)
- removed copper zone on F.Cu, net Net-(C77-Pad1)

Commit message: continue routing
Parts:
- removed C19: 68u, Capacitor_SMD:CP_Elec_8x10
- removed C198, C199, C26, C31: 4.7u, _Generic:1210_CAP
- removed J68, J69: Conn_01x03, _Generic:JST_XH_3P
- added J46: Conn_01x03, _Generic:JST_XH_3P, F.Cu at (169.4, 109.2)
- added J47: Conn_01x03, _Generic:JST_XH_3P, F.Cu at (163.1, 109.2)
- added J61: Micro_SD_Card_Det, _Generic:HYC77-TF09-200, B.Cu at (196.8, 80.0)
- added JP17: SolderJumper_4_Open, _Generic:SolderJumper_JST, B.Cu at (151.9, 106.7)
- added JP25: SolderJumper_4_Open, _Generic:SolderJumper_JST, B.Cu at (158.2, 117.1)
- added JP26: SolderJumper_4_Open, _Generic:SolderJumper_JST, B.Cu at (164.6, 117.1)
- added JP27: SolderJumper_4_Open, _Generic:SolderJumper_JST, B.Cu at (151.9, 117.1)
- added JP31: SolderJumper_4_Open, _Generic:SolderJumper_JST, B.Cu at (177.3, 117.1)
- added JP32: SolderJumper_4_Open, _Generic:SolderJumper_JST, B.Cu at (170.9, 117.1)
- added JP33: SolderJumper_4_Open, _Generic:SolderJumper_JST, B.Cu at (183.6, 106.7)
- added JP36: SolderJumper_4_Open, _Generic:SolderJumper_JST, B.Cu at (183.6, 117.1)
- added JP37: SolderJumper_4_Open, _Generic:SolderJumper_JST, B.Cu at (177.3, 106.7)
- added JP43: SolderJumper_4_Open, _Generic:SolderJumper_JST, B.Cu at (158.2, 106.7)
- added JP44: SolderJumper_4_Open, _Generic:SolderJumper_JST, B.Cu at (170.9, 106.7)
- added JP45: SolderJumper_4_Open, _Generic:SolderJumper_JST, B.Cu at (164.6, 106.7)
- added LS1: Buzzer, _Generic:Buzzer-7525, F.Cu at (189.2, 120.1)
- C10, C11, C12, C13, C14, C2, C4, C54, C55, C56, C57, C58, C59, C6, C60, C61, C64, C65, C66, C7, C70, C71, C72, C75, C76, C8, C9, D10, D15, D16, D17, D20, D21, D22, D23, D24, D26, D7, D8, D9, JP16, JP18, JP19, JP20, JP21, JP22, JP23, JP24, JP28, JP29, JP30, JP34, JP35, JP38, Q10, Q12, Q13, Q14, Q3, Q4, Q5, Q8, Q9, R32, R35, R36, R38, R39, R41, R44, R46, R48, R50, R55, R56, R57, R58, R59, R60, R65, R66, R67, R68, R69, R70, R71, R72, R73, R74, R76, R78, R83: moved to B.Cu
- C3: value 12p -> 220p
- C5: value 12p -> 100n
- C80: value 100n -> 100p
- R33: value 47k -> 4.7k; moved to B.Cu
- R40: value 4.7k -> 47k; moved to B.Cu
- R80: value 0R -> 1k
- moved J42 238.8 mm to (304.0, 44.4)
- moved J41 230.8 mm to (309.3, 41.7)
- moved J43 228.8 mm to (309.3, 44.4)
- moved JP38 222.5 mm to (113.0, 69.1), turned to 180 degrees
- moved R80 216.9 mm to (148.8, 86.6)
- moved C80 216.9 mm to (148.8, 85.7)
- moved R79 216.9 mm to (148.8, 87.5)
- moved X1 216.9 mm to (147.3, 83.0)
- moved JP14 211.3 mm to (311.1, 40.8)
- moved JP7 207.1 mm to (155.3, 72.3)
- moved J40 205.7 mm to (306.6, 44.4)
- moved R6 200.2 mm to (154.4, 80.3)
- moved R7 197.5 mm to (156.8, 84.0)
- moved R83 196.1 mm to (138.8, 76.3)
- moved C4 194.6 mm to (163.6, 83.0)
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Connections:
- net /Stepper Driver/Driver1/CLK renamed /DRV_CLK
- C3 pad 1: Net-(C3-Pad1) -> /LPC_CLK
- C5 pad 1: Net-(C5-Pad1) -> +3V3
- C55 pad 1: Net-(C54-Pad1) -> Net-(C55-Pad1)
- C56 pad 1: Net-(C54-Pad1) -> Net-(C56-Pad1)
- C57 pad 1: Net-(C54-Pad1) -> Net-(C57-Pad1)
- C80 pad 1: +3V3 -> /LPC_CLK
- C80 pad 2: GND -> Net-(C80-Pad2)
- D7 pad 1: /P0.20_END -> /P0.19_END
- D8 pad 1: /P0.19_END -> /P0.20_END
- J67 pad 1: Net-(C54-Pad1) -> Net-(C55-Pad1)
- R32 pad 2: /P0.20_END -> /P0.19_END
- R33 pad 1: +3V3 -> /P0.19_END
- R33 pad 2: /P0.19_END -> Net-(J46-Pad3)
- R40 pad 1: /P0.19_END -> +3V3
- R40 pad 2: Net-(J68-Pad3) -> /P0.20_END
- R80 pad 2: Net-(R80-Pad2) -> Net-(C80-Pad2)
- U1 pad 22: Net-(U1-Pad22) -> /LPC_CLK
- X1 pad 3: Net-(R80-Pad2) -> Net-(C80-Pad2)
Routing:
- net /DRV_MISO: track 0.00 -> 86.8 mm, vias 0 -> 5
- net /DRV_MOSI: track 0.00 -> 86.0 mm, vias 0 -> 5
- net /DRV_SCK: track 0.00 -> 82.6 mm, vias 0 -> 5
- net /DRV_CLK: track 0.00 -> 80.4 mm, vias 0 -> 5
- net GND: track 182.4 -> 223.4 mm
- net /DRV1_STEP: track 0.00 -> 25.9 mm
- net /DRV1_DIR: track 0.00 -> 25.3 mm
- net /DRV1_CS: track 0.00 -> 24.4 mm
- net Net-(IC1-Pad28): track 2.44 -> 20.3 mm
- net +12V: track 10.1 -> 26.9 mm
- net /DRV1_EN: track 3.58 -> 19.8 mm
- net /Stepper Driver/DRV1_DIAG1: track 3.93 -> 19.0 mm
- net Net-(C38-Pad2): track 0.00 -> 12.5 mm
- net Net-(C37-Pad2): track 0.00 -> 12.3 mm
- net +5V: track 0.00 -> 12.1 mm
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Other:
- board text added: "P0.12"

Commit message: continue routing
Parts:
- removed D11, D12, D13, D14: DNP, _Generic:SOD-523_DIODE
- removed J64, J65: Conn_01x04, _Generic:JST_XH_4P
- removed R43, R45, R47, R49: DNP, _Generic:0603_RES
- removed R51, R52, R53, R54: 0R, _Generic:0603_RES
- added C19: 10u, _Generic:0603_CAP, B.Cu at (166.9, 76.0)
- added C198: 10u, _Generic:0603_CAP, F.Cu at (190.0, 80.9)
- added C199: 220u, Capacitor_SMD:CP_Elec_6.3x7.7, F.Cu at (194.1, 75.4)
- added C26: 10u, _Generic:0603_CAP, B.Cu at (155.5, 85.3)
- added C31: 10u, _Generic:0603_CAP, B.Cu at (160.4, 76.0)
- added J100: Conn_01x01, _Generic:PinHeader_2.54mm_1P, F.Cu at (189.9, 97.8)
- added J101: Conn_01x01, _Generic:PinHeader_2.54mm_1P, F.Cu at (187.3, 91.2)
- added J102: Conn_01x01, _Generic:PinHeader_2.54mm_1P, F.Cu at (197.5, 91.2)
- added J103: Conn_01x01, _Generic:PinHeader_2.54mm_1P, F.Cu at (218.8, 75.5)
- added J104: Conn_01x01, _Generic:PinHeader_2.54mm_1P, F.Cu at (187.3, 97.8)
- added J49: Conn_01x01, _Generic:PinHeader_2.54mm_1P, F.Cu at (144.5, 80.0)
- added J50: Conn_01x01, _Generic:PinHeader_2.54mm_1P, F.Cu at (142.0, 80.0)
- added J52: Conn_01x01, _Generic:PinHeader_2.54mm_1P, F.Cu at (177.2, 77.5)
- added J53: Conn_01x01, _Generic:PinHeader_2.54mm_1P, F.Cu at (197.5, 93.7)
- added J68: Conn_01x01, _Generic:PinHeader_2.54mm_1P, F.Cu at (182.2, 100.3)
- added J69: Conn_01x01, _Generic:PinHeader_2.54mm_1P, F.Cu at (179.7, 82.5)
- added J70: Conn_01x01, _Generic:PinHeader_2.54mm_1P, F.Cu at (197.5, 100.3)
- added J94: Conn_01x01, _Generic:PinHeader_2.54mm_1P, F.Cu at (182.2, 97.8)
- added J95: Conn_01x01, _Generic:PinHeader_2.54mm_1P, F.Cu at (179.7, 85.1)
- added J96: Conn_01x01, _Generic:PinHeader_2.54mm_1P, F.Cu at (189.9, 100.3)
- added J97: Conn_01x01, _Generic:PinHeader_2.54mm_1P, F.Cu at (224.1, 75.5)
- added J98: Conn_01x01, _Generic:PinHeader_2.54mm_1P, F.Cu at (187.3, 93.7)
- added J99: Conn_01x01, _Generic:PinHeader_2.54mm_1P, F.Cu at (197.5, 97.8)
- C15, C16, C17, JP39, JP40, JP41, JP42, R4, R5, R6, R7: moved to B.Cu
- JP16, R83: moved to F.Cu
- SW1, SW2: footprint Button_Switch_SMD:SW_SPST_CK_RS282G05A3 -> _Generic:Switch_3x4mm
- moved J41 220.6 mm to (108.9, 134.0)
- moved J43 217.1 mm to (111.6, 134.0)
- moved JP14 214.7 mm to (116.0, 130.5)
- moved J42 204.4 mm to (117.6, 128.3)
- moved J40 203.9 mm to (120.8, 128.3)
- moved J54 168.5 mm to (142.0, 77.5)
- moved J55 163.4 mm to (144.5, 77.5)
- moved JP39 118.6 mm to (129.8, 68.9), turned to 180 degrees
- moved R92 110.1 mm to (139.8, 72.2)
- moved JP40 107.9 mm to (146.8, 68.8), turned to 180 degrees
- moved R101 102.5 mm to (153.8, 72.2), turned to 180 degrees
- moved JP41 97.3 mm to (163.8, 68.9), turned to 180 degrees
- moved C1 92.1 mm to (152.4, 86.2), turned to 90 degrees
- moved R110 92.1 mm to (170.8, 72.2), turned to 180 degrees
- moved R37 90.0 mm to (153.8, 92.5), turned to 90 degrees
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Connections:
- J25 pad 1: /DRV5_EN -> /DRV5_DIR
- J26 pad 1: /DRV5_DIR -> /DRV5_EN
- J61 pad 10: /Interfaces/SD_DETECT -> GND
- J61 pad 9: GND -> /Interfaces/SD_DETECT
- J75 pad 1: Net-(J75-Pad1) -> /P1.30_GEN
- J76 pad 1: Net-(J76-Pad1) -> /P1.31_GEN
- J77 pad 1: Net-(J77-Pad1) -> /P4.28_GEN
- J78 pad 1: Net-(J78-Pad1) -> /P4.29_GEN
- U1 pad 86: /DRV5_DIR -> /DRV5_EN
- U1 pad 87: /DRV5_EN -> /DRV5_DIR
- U1 pad 88: /DRV4_DIR -> /DRV4_EN
- U1 pad 89: /DRV4_EN -> /DRV4_DIR
- U1 pad 90: /DRV3_DIR -> /DRV3_EN
- U1 pad 91: /DRV3_EN -> /DRV3_DIR
- U1 pad 92: /DRV2_DIR -> /DRV2_EN
- U1 pad 93: /DRV2_EN -> /DRV2_DIR
- U1 pad 94: /DRV1_DIR -> /DRV1_EN
- U1 pad 95: /DRV1_EN -> /DRV1_DIR
Routing:
- net GND: track 223.4 -> 329.0 mm, vias 383 -> 389
- net /Stepper Driver/DRV_DIAG0: track 0.00 -> 51.2 mm, vias 0 -> 5
- net /P0.19_END: track 0.00 -> 50.7 mm, vias 0 -> 1
- net /P2.3_POW: track 0.00 -> 50.4 mm, vias 0 -> 2
- net /RST: track 0.00 -> 50.4 mm
- net /P0.22_ADV: track 0.00 -> 50.2 mm, vias 0 -> 1
- net /DRV5_DIR: track 0.00 -> 49.6 mm, vias 0 -> 1
- net /DRV5_EN: track 0.00 -> 48.6 mm, vias 0 -> 1
- net /P2.4_POW: track 0.00 -> 48.3 mm, vias 0 -> 2
- net /DRV_MISO: track 86.8 -> 131.7 mm, vias 5 -> 8
- net /DRV3_DIAG1: track 0.00 -> 43.6 mm, vias 0 -> 2
- net /DRV2_DIAG1: track 0.00 -> 43.2 mm, vias 0 -> 2
- net /DRV1_DIAG1: track 0.00 -> 43.0 mm, vias 0 -> 2
- net /DRV4_DIAG1: track 0.00 -> 42.6 mm, vias 0 -> 2
- net /DRV_SCK: track 82.6 -> 125.2 mm, vias 5 -> 8
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- added copper zone on B.Cu, net +12V
- added copper zone on F.Cu, net +12V
- added copper zone on F.Cu, net +3V3
- added copper zone on B.Cu, net +5V
- added copper zone on F.Cu, net +5V
- added copper zone on F.Cu, net Net-(C37-Pad2)
- added copper zone on F.Cu, net Net-(C38-Pad2)
