File: hardware/kajikia/kajikia.kicad_pcb (KiCad board)
At the start: 4 copper layers, 100 x 75 mm, 571 parts, among them IC1 TMC5161, IC2 TMC5161, IC3 TMC5161, IC4 TMC5161, IC5 TMC5161, J1 Conn_01x01, J10 Conn_01x01, J100 Conn_01x01, J101 Conn_01x01, J102 Conn_01x01, J103 Conn_01x01, J104 Conn_01x01, J11 Conn_01x01, J12 Conn_01x01, J13 Conn_01x01, J14 Conn_01x01, J15 Conn_01x01, J16 Conn_01x01, J17 Conn_01x01, J18 Conn_01x01, J19 Conn_01x01, J2 Conn_01x01, J20 Conn_01x01, J21 Conn_01x01, J22 Conn_01x01, J23 Conn_01x01, J24 Conn_01x01, J25 Conn_01x01, J26 Conn_01x01, J27 Conn_01x01, J28 Conn_01x01, J29 Conn_01x01, J3 Conn_01x01, J30 Conn_01x01, J31 Conn_01x01, J32 Conn_01x01, J33 Conn_01x01, J34 Conn_01x01, J35 Conn_01x01, J36 Conn_01x01, J37 Conn_01x01, J38 Conn_01x01, J39 Screw_Terminal_01x02, J4 Conn_01x01, J40 Conn_01x01, J41 Conn_01x01, J42 Conn_01x01, J43 Conn_01x01, J44 Conn_01x01, J45 Conn_01x01, J46 Conn_01x03, J47 Conn_01x03, J48 Conn_01x01, J49 Conn_01x01, J5 Conn_01x01, J50 Conn_01x01, J51 Conn_01x01, J52 Conn_01x01, J53 Conn_01x01, J54 Conn_01x01, J55 Conn_01x01, J56 Conn_01x01, J57 Conn_01x01, J58 Conn_01x01, J59 Conn_01x01, J6 Conn_01x01, J60 USB_C_Receptacle, J61 Micro_SD_Card_Det, J62 Conn_01x02, J63 Conn_01x02, J66 Conn_01x03, J67 Conn_01x03, J68 Conn_01x01, J69 Conn_01x01, J7 Conn_01x01, J70 Conn_01x01, J71 Conn_01x02, J72 Conn_01x02, J73 Conn_01x02, J74 Conn_01x02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

Commit message: continue routing
Parts:
- removed J103, J40, J41, J42, J43, J97: Conn_01x01, _Generic:PinHeader_2.54mm_1P
- removed JP14: SolderJumper_2_Open, _Generic:Solder Jumper 2P
- C48, C53, L4, L5, L6, L7, R34: moved to B.Cu
- moved JP2 51.5 mm to (186.7, 102.6), turned to 90 degrees
- moved JP3 16.2 mm to (188.0, 102.6), turned to 90 degrees
- moved Q14 10.8 mm to (189.2, 120.1)
- moved R76 9.93 mm to (189.2, 117.7), turned to 180 degrees
- moved R78 7.32 mm to (186.8, 120.1), turned to 270 degrees
- moved D26 5.88 mm to (189.1, 122.6)
- moved C45 5.67 mm to (191.1, 103.0)
- moved R8 5.45 mm to (132.2, 79.1)
- moved R79 4.14 mm to (149.9, 72.2)
- moved C53 2.78 mm to (192.5, 114.3)
- moved C48 2.66 mm to (192.5, 106.2)
- moved L6 2.44 mm to (194.4, 113.4), turned to 0 degrees
- moved R34 2.07 mm to (191.1, 114.3)
- moved L7 1.82 mm to (194.4, 115.2), turned to 0 degrees
- moved R23 1.79 mm to (191.8, 109.5), turned to 0 degrees
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Routing:
- net +3V3: track 22.7 -> 266.5 mm, vias 6 -> 60
- net GND: track 329.0 -> 454.4 mm, vias 389 -> 478
- net +5V: track 13.8 -> 118.4 mm, vias 12 -> 65
- net +12V: track 26.9 -> 95.6 mm, vias 17 -> 27
- net VBUS: track 0.00 -> 35.8 mm
- net /DRV_SCK: track 125.2 -> 157.6 mm, vias 8 -> 10
- net /DRV_MISO: track 131.7 -> 155.1 mm, vias 8 -> 10
- net /P3.26_BUZ: track 33.5 -> 56.0 mm
- net /DRV3_CS: track 30.0 -> 42.7 mm
- net /MAX1_CS: track 18.5 -> 30.1 mm, vias 0 -> 1
- net /DRV4_CS: track 16.3 -> 27.7 mm
- net /Interfaces/MAX2_CS: track 0.00 -> 10.7 mm
- net +24V: track 96.2 -> 105.8 mm, vias 622 -> 632
- net /ISP_BOOT: track 24.3 -> 33.5 mm, vias 1 -> 2
- net /VDDA: track 0.00 -> 6.72 mm, vias 0 -> 1
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- added copper zone on In2.Cu, net +12V
- added copper zone on In2.Cu, net +3V3
- added copper zone on In2.Cu, net +5V
- added copper zone on In2.Cu, net DCIN-
- added copper zone on B.Cu, net GND
- added copper zone on In2.Cu, net GND
- added copper zone on In1.Cu, net Net-(D18-Pad1)
- added copper zone on In2.Cu, net Net-(D18-Pad1)
- added copper zone on In1.Cu, net Net-(D19-Pad1)
- added copper zone on In2.Cu, net Net-(D19-Pad1)
- added copper zone on In1.Cu, net Net-(D25-Pad1)
- added copper zone on In2.Cu, net Net-(D25-Pad1)
- added copper zone on In2.Cu, net Net-(F1-Pad1)
- added copper zone on In1.Cu, net Net-(F2-Pad1)
- added copper zone on In2.Cu, net Net-(F2-Pad1)
- added copper zone on In1.Cu, net Net-(F3-Pad1)
- added copper zone on In2.Cu, net Net-(F3-Pad1)
- added copper zone on In1.Cu, net Net-(F4-Pad1)
- added copper zone on In2.Cu, net Net-(F4-Pad1)
Other:
- net class 24v added: clearance 0.2, trace_width 0.127, via_dia 0.6, via_drill 0.4

Commit message: continue routing
Parts:
- added H5: MountingHole, MountingHole:MountingHole_2.2mm_M2_DIN965, F.Cu at (196.5, 63.9)
- added H6: MountingHole, MountingHole:MountingHole_2.2mm_M2_DIN965, F.Cu at (103.5, 63.9)
- added JP14: SolderJumper_2_Open, _Generic:Solder Jumper 2P, F.Cu at (133.3, 116.4)
- renumbered SW2 to ISP, SW1 to RST
Routing:
- net +24V: track 105.8 -> 109.5 mm, vias 632 -> 648
- net GND: vias 478 -> 504
- net DCIN-: vias 55 -> 98
- added copper zone on In1.Cu, net DCIN-
Other:
- board text added: "12V"
- board text added: "24V"
- board text added: "3.3V"
- board text added: "5V"
- board text added: "P0.0"
- board text added: "P0.1"
- board text added: "P0.19"
- board text added: "P0.20"
- board text added: "P0.22"
- board text added: "P0.23"
- board text added: "P0.24"
- board text added: "P0.25"
- board text added: "P0.26"
- board text added: "P0.28"
- board text added: "P1.18"
- board text added: "P1.19"
- board text added: "P1.22"
- board text added: "P1.25"
- board text added: "P1.26"
- board text added: "P1.29"
- board text removed: "P0.12"
