File: hardware/kajikia/kajikia.kicad_pcb (KiCad board)
At the start: 4 copper layers, 100 x 75 mm, 567 parts, among them IC1 TMC5161, IC2 TMC5161, IC3 TMC5161, IC4 TMC5161, IC5 TMC5161, J1 Conn_01x01, J10 Conn_01x01, J100 Conn_01x01, J101 Conn_01x01, J102 Conn_01x01, J104 Conn_01x01, J11 Conn_01x01, J12 Conn_01x01, J13 Conn_01x01, J14 Conn_01x01, J15 Conn_01x01, J16 Conn_01x01, J17 Conn_01x01, J18 Conn_01x01, J19 Conn_01x01, J2 Conn_01x01, J20 Conn_01x01, J21 Conn_01x01, J22 Conn_01x01, J23 Conn_01x01, J24 Conn_01x01, J25 Conn_01x01, J26 Conn_01x01, J27 Conn_01x01, J28 Conn_01x01, J29 Conn_01x01, J3 Conn_01x01, J30 Conn_01x01, J31 Conn_01x01, J32 Conn_01x01, J33 Conn_01x01, J34 Conn_01x01, J35 Conn_01x01, J36 Conn_01x01, J37 Conn_01x01, J38 Conn_01x01, J39 Screw_Terminal_01x02, J4 Conn_01x01, J44 Conn_01x01, J45 Conn_01x01, J46 Conn_01x03, J47 Conn_01x03, J48 Conn_01x01, J49 Conn_01x01, J5 Conn_01x01, J50 Conn_01x01, J51 Conn_01x01, J52 Conn_01x01, J53 Conn_01x01, J54 Conn_01x01, J55 Conn_01x01, J56 Conn_01x01, J57 Conn_01x01, J58 Conn_01x01, J59 Conn_01x01, J6 Conn_01x01, J60 USB_C_Receptacle, J61 Micro_SD_Card_Det, J62 Conn_01x02, J63 Conn_01x02, J66 Conn_01x03, J67 Conn_01x03, J68 Conn_01x01, J69 Conn_01x01, J7 Conn_01x01, J70 Conn_01x01, J71 Conn_01x02, J72 Conn_01x02, J73 Conn_01x02, J74 Conn_01x02, J75 Conn_01x01, J76 Conn_01x01, J77 Conn_01x01, J78 Conn_01x01, J79 Conn_01x03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

Commit message: PCB V1
Parts:
- R28, R56, R58, R60, R66, R68, R70, R72, R74: value 50k -> 47k
- renumbered RST to SW1, ISP to SW2
Connections:
- net /P1.30_GEN renamed /P1.30
- net /P1.31_GEN renamed /P1.31
- net /P4.28_GEN renamed /P4.28
- net /P4.29_GEN renamed /P4.29
- U8 pad 4: Net-(U8-Pad4) -> GND
Routing:
- net GND: track 454.4 -> 463.0 mm, vias 504 -> 556
- net Net-(C20-Pad1): track 5.00 -> 8.88 mm
- net /USB_CON: track 28.9 -> 30.2 mm
- net /DRV4_CS: track 27.7 -> 26.6 mm
- net /DRV3_CS: track 42.7 -> 42.0 mm
- net /DRV4_DIAG1: track 42.9 -> 42.2 mm
- net +5V: vias 65 -> 89
- net +24V: vias 648 -> 647
Other:
- board text added: "ISP"
- board text added: "Kajikia"
- board text added: "RST"
- board text added: "TH1"
- board text added: "TH2"
