File: hardware/kajikia/single_driver.sch (KiCad schematic (older format))
At the start: 45 parts, among them IC1 TMC5161

Commit message: footprints
Parts:
- C67: footprint (none) -> Capacitor_SMD:CP_Elec_8x10
- D21, D22, D23, D24, D25, D26, D27, D28: footprint (none) -> _Generic:SOD-523_DIODE

Commit message: layout test
Parts:
- removed C67: 68u, Capacitor_SMD:CP_Elec_8x10, symbol Device:CP1_Small
- added C94, C95: 4.7u, _Generic:1210_CAP, symbol Device:C_Small
- C91: renamed from C64; footprint _Generic:0805_CAP -> _Generic:1210_CAP
- R88: renamed from R75; footprint _Generic:0603_RES -> _Generic:1206_RES
- R89: renamed from R76; footprint _Generic:0603_RES -> _Generic:1206_RES
- renumbered C72 to C100, C73 to C101, C54 to C81, C55 to C82, C56 to C83, C57 to C84, C58 to C85, C59 to C86, C60 to C87, C61 to C88, C62 to C89, C63 to C90, C65 to C92, C66 to C93, C68 to C96, C69 to C97, C70 to C98, C71 to C99, D21 to D27, D22 to D28, D23 to D29, D24 to D30, D25 to D31, D26 to D32, D27 to D33, D28 to D34, JP37 to JP38, R68 to R81, R69 to R82, R70 to R83, R71 to R84, R72 to R85, R73 to R86, R74 to R87
Connections:
- net +24V: now also C94.1, C95.1
- net GND: now also C94.2, C95.2; no longer IC1.30 (×), IC1.36 (×)
- net VCC: now reaches C84.1, IC1.32 (VCC), R82.1, TP3.1
- net VCC: now also IC1.BR (×)
- net RSA: now reaches IC1.RSA, R84.1, R88.1
- net RSA: now also IC1.TR (×)
- net RSB: now reaches IC1.RSB, R86.1, R89.1
- net RSB: now also IC1.TL (×)
- no-connect marks 1 -> 5

Commit message: tmc layout
Parts:
- added C186: 4.7u, _Generic:1210_CAP, symbol Device:C_Small
Connections:
- net +24V: now also C186.1
- net GND: now also C186.2; no longer IC1.3 (×), IC1.5 (×), IC1.9 (×)
- net SRBH: now reaches IC1.11 (SRBH), R86.2
- net SRBH: now also IC1.BL (×)
- net 5V_out: now reaches C83.1, IC1.6 (5V_out), R82.2, TP2.1
- net 5V_out: now also IC1.5 (×)
- no-connect marks 5 -> 6
Other:
- moved on the sheet: C95
Changed lines of the file:
@@
 Wire Wire Line
 	4450 3100 4650 3100
-Wire Wire Line
-	4850 5550 4850 5650
-Wire Wire Line
-	4850 5650 4900 5650
-Connection ~ 5250 5650
-Wire Wire Line
-	4900 5550 4900 5650
-Connection ~ 4900 5650
 $Comp
 L power:PWR_FLAG #FLG011
@@
 L Device:C_Small C?
 U 1 1 5C3B22C5
-P 7500 2050
+P 7900 2050
 AR Path="/5B406A82/5B411670/5C3B22C5" Ref="C?"  Part="1"
 AR Path="/5B406A82/5B01DBD9/5C3B22C5" Ref="C?"  Part="1"
@@
 AR Path="/60C2EDFB/60ED586F/5C3B22C5" Ref="C158"  Part="1"
 AR Path="/60C2EDFB/60ED8641/5C3B22C5" Ref="C179"  Part="1"
-F 0 "C95" H 7592 2096 50  0000 L CNN
-F 1 "4.7u" H 7592 2005 50  0000 L CNN
-F 2 "_Generic:1210_CAP" H 7500 2050 50  0001 C CNN
-F 3 "~" H 7500 2050 50  0001 C CNN
-	1    7500 2050
-	1    0    0    -1
-$EndComp
-Wire Wire Line
-	7100 2250 7500 2250
-Wire Wire Line
-	7500 2250 7500 2150
-Connection ~ 7100 2250
-Wire Wire Line
-	7500 1950 7500 1750
-Wire Wire Line
-	7500 1750 7100 1750
-Connection ~ 7100 1750
-Wire Wire Line
-	4900 5650 4950 5650
-Connection ~ 4950 5650
-Wire Wire Line
-	4950 5650 4950 5550
-Wire Wire Line
-	4950 5650 5250 5650
+F 0 "C95" H 7992 2096 50  0000 L CNN
+F 1 "4.7u" H 7992 2005 50  0000 L CNN
+F 2 "_Generic:1210_CAP" H 7900 2050 50  0001 C CNN
+F 3 "~" H 7900 2050 50  0001 C CNN
+	1    7900 2050
+	1    0    0    -1
+$EndComp
+Wire Wire Line
+	7500 2250 7900 2250
+Wire Wire Line
+	7900 2250 7900 2150
+Wire Wire Line
+	7900 1950 7900 1750
+Wire Wire Line
+	7900 1750 7500 1750
 NoConn ~ 5000 5550
 NoConn ~ 5050 5550
@@
 Wire Wire Line
 	5750 5800 5750 5550
-NoConn ~ 5700 5550
 NoConn ~ 2600 4500
+Text Label 4200 2800 0    50   ~ 0
+5V_out
+Text Label 4900 6050 1    50   ~ 0
+5V_out
+Wire Wire Line
+	4900 6050 4900 5550
+NoConn ~ 4850 5550
+NoConn ~ 4950 5550
+Text Label 6300 4700 2    50   ~ 0
+SRBH
+Text Label 5700 5800 1    50   ~ 0
+SRBH
+Wire Wire Line
+	5700 5800 5700 5550
+$Comp
+L Device:C_Small C?
+U 1 1 5C3A821D
+P 7500 2050
+AR Path="/5B406A82/5B411670/5C3A821D" Ref="C?"  Part="1"
+AR Path="/5B406A82/5B01DBD9/5C3A821D" Ref="C?"  Part="1"
+AR Path="/5B406A82/5B01DBED/5C3A821D" Ref="C?"  Part="1"
+AR Path="/5B406A82/5B01DC01/5C3A821D" Ref="C?"  Part="1"
+AR Path="/5B406A82/5B01DC15/5C3A821D" Ref="C?"  Part="1"
+AR Path="/5AF7E834/60C2EDFB/5B411670/5C3A821D" Ref="C?"  Part="1"
+AR Path="/5AF7E834/60C2EDFB/5B01DBD9/5C3A821D" Ref="C?"  Part="1"
+AR Path="/5AF7E834/60C2EDFB/5B01DBED/5C3A821D" Ref="C?"  Part="1"
+AR Path="/5AF7E834/60C2EDFB/5B01DC01/5C3A821D" Ref="C?"  Part="1"
+AR Path="/5AF7E834/60C2EDFB/5B01DC15/5C3A821D" Ref="C?"  Part="1"
+AR Path="/5AF7E834/60C2EDFB/60ECA8FF/5C3A821D" Ref="C?"  Part="1"
+AR Path="/5B406A82/60ECA8FF/5C3A821D" Ref="C?"  Part="1"
+AR Path="/5AF7E834/60C2EDFB/60ECD6D9/5C3A821D" Ref="C?"  Part="1"
+AR Path="/5B406A82/60ECD6D9/5C3A821D" Ref="C?"  Part="1"
+AR Path="/5AF7E834/60C2EDFB/60ED586F/5C3A821D" Ref="C?"  Part="1"
+AR Path="/5B406A82/60ED586F/5C3A821D" Ref="C?"  Part="1"
+AR Path="/5AF7E834/60C2EDFB/60ED8641/5C3A821D" Ref="C?"  Part="1"
+AR Path="/5B406A82/60ED8641/5C3A821D" Ref="C?"  Part="1"
+AR Path="/60C2EDFB/5B411670/5C3A821D" Ref="C186"  Part="1"
+AR Path="/60C2EDFB/60ECA8FF/5C3A821D" Ref="C187"  Part="1"
+AR Path="/60C2EDFB/60ECD6D9/5C3A821D" Ref="C188"  Part="1"
+AR Path="/60C2EDFB/60ED586F/5C3A821D" Ref="C189"  Part="1"
+AR Path="/60C2EDFB/60ED8641/5C3A821D" Ref="C190"  Part="1"
+F 0 "C186" H 7592 2096 50  0000 L CNN
+F 1 "4.7u" H 7592 2005 50  0000 L CNN
+F 2 "_Generic:1210_CAP" H 7500 2050 50  0001 C CNN
+F 3 "~" H 7500 2050 50  0001 C CNN
+	1    7500 2050
+	1    0    0    -1
+$EndComp
+Wire Wire Line
+	7100 2250 7500 2250
+Wire Wire Line
+	7500 2250 7500 2150
+Wire Wire Line
+	7500 1950 7500 1750
+Wire Wire Line
+	7500 1750 7100 1750
 $EndSCHEMATC

Commit message: fuses
Parts:
- removed TP1, TP2, TP3, TP4, TP5, TP6: TestPoint, symbol #PCB_Only:TestPoint
- JP38: footprint (none) -> _Generic:Solder Jumper 2P
