File: hardware/kajikia/_saved_power.sch (KiCad schematic (older format))
At the start: 90 parts, among them J100 Conn_01x01, J101 Conn_01x01, J102 Conn_01x01, J39 Screw_Terminal_01x02, J44 Conn_01x01, J45 Conn_01x01, J48 Conn_01x01, J49 Conn_01x01, J50 Conn_01x01, J51 Conn_01x01, J53 Conn_01x01, J54 Conn_01x01, J55 Conn_01x01, J56 Conn_01x01, J57 Conn_01x01, J58 Conn_01x01, J59 Conn_01x01, J68 Conn_01x01, J69 Conn_01x01, J70 Conn_01x01, J94 Conn_01x01, J95 Conn_01x01, J96 Conn_01x01, J98 Conn_01x01, J99 Conn_01x01, Q1 AON6144, U2 LM1117-3.3, U3 AOZ1284, U4 AOZ1284

Commit message: continue routing
Parts:
- H5, H6: renamed from H?; footprint (none) -> MountingHole:MountingHole_2.2mm_M2_DIN965
Changed lines of the file:
@@
 Connection ~ 12200 4450
 $Comp
-L Mechanical:MountingHole H?
+L Mechanical:MountingHole H5
 U 1 1 5C4CA30F
 P 7050 6100
-F 0 "H?" H 7150 6146 50  0000 L CNN
+F 0 "H5" H 7150 6146 50  0000 L CNN
 F 1 "MountingHole" H 7150 6055 50  0000 L CNN
-F 2 "" H 7050 6100 50  0001 C CNN
+F 2 "MountingHole:MountingHole_2.2mm_M2_DIN965" H 7050 6100 50  0001 C CNN
 F 3 "~" H 7050 6100 50  0001 C CNN
 	1    7050 6100
@@
 $EndComp
 $Comp
-L Mechanical:MountingHole H?
+L Mechanical:MountingHole H6
 U 1 1 5C4CA407
 P 7050 6350
-F 0 "H?" H 7150 6396 50  0000 L CNN
+F 0 "H6" H 7150 6396 50  0000 L CNN
 F 1 "MountingHole" H 7150 6305 50  0000 L CNN
-F 2 "" H 7050 6350 50  0001 C CNN
+F 2 "MountingHole:MountingHole_2.2mm_M2_DIN965" H 7050 6350 50  0001 C CNN
 F 3 "~" H 7050 6350 50  0001 C CNN
 	1    7050 6350
