File: hardware/kajikia/interface.sch (KiCad schematic (older format))
At the start: 92 parts, among them J39 USB_C_Receptacle, J40 Micro_SD_Card_Det, J41 Conn_01x02, J42 Conn_01x02, J43 Conn_01x01, J44 Conn_01x01, J45 Conn_01x01, J46 Conn_01x01, J47 Conn_01x04, J48 Conn_01x04, J49 Conn_01x04, J50 Conn_01x02, J51 Conn_01x02, J52 Conn_01x02, J53 Conn_01x02, J54 Conn_01x03, J55 Conn_01x03, J56 Conn_01x03, J57 Conn_01x03, Q1 AO3401, U2 MAX6675, U3 MAX6675

Commit message: footprints
Parts:
- D1, D2, D3, D4, D5, D6, D7, D8: footprint (none) -> _Generic:SOD-523_DIODE
- L1, L2, L3, L4: footprint (none) -> _Generic:0603_IND
- Q1: footprint (none) -> _Generic:SOT-23
- U2, U3: footprint (none) -> _Generic:SO-8
Changed lines of the file:
@@
 $Descr A4 11693 8268
 encoding utf-8
-Sheet 2 10
+Sheet 3 10
 Title ""
 Date ""
@@
 F 0 "Q1" H 3656 1304 50  0000 L CNN
 F 1 "AO3401" H 3656 1395 50  0000 L CNN
-F 2 "" H 3650 1450 50  0001 C CNN
+F 2 "_Generic:SOT-23" H 3650 1450 50  0001 C CNN
 F 3 "~" H 3450 1350 50  0001 C CNN
 	1    3450 1350
@@
 F 0 "U3" H 5300 7615 50  0000 C CNN
 F 1 "MAX6675" H 5300 7524 50  0000 C CNN
-F 2 "" H 5350 7150 50  0001 C CNN
+F 2 "_Generic:SO-8" H 5350 7150 50  0001 C CNN
 F 3 "" H 5350 7150 50  0001 C CNN
 	1    5300 7100
@@
 F 0 "L3" V 6390 6950 50  0000 C CNN
 F 1 "470" V 6299 6950 50  0000 C CNN
-F 2 "" H 6200 6950 50  0001 C CNN
+F 2 "_Generic:0603_IND" H 6200 6950 50  0001 C CNN
 F 3 "~" H 6200 6950 50  0001 C CNN
 	1    6200 6950
@@
 F 0 "L4" V 6390 7250 50  0000 C CNN
 F 1 "470" V 6299 7250 50  0000 C CNN
-F 2 "" H 6200 7250 50  0001 C CNN
+F 2 "_Generic:0603_IND" H 6200 7250 50  0001 C CNN
 F 3 "~" H 6200 7250 50  0001 C CNN
 	1    6200 7250
@@
 F 0 "U2" H 2300 7615 50  0000 C CNN
 F 1 "MAX6675" H 2300 7524 50  0000 C CNN
-F 2 "" H 2350 7150 50  0001 C CNN
+F 2 "_Generic:SO-8" H 2350 7150 50  0001 C CNN
 F 3 "" H 2350 7150 50  0001 C CNN
 	1    2300 7100
@@
 F 0 "L1" V 3390 6950 50  0000 C CNN
 F 1 "470" V 3299 6950 50  0000 C CNN
-F 2 "" H 3200 6950 50  0001 C CNN
+F 2 "_Generic:0603_IND" H 3200 6950 50  0001 C CNN
 F 3 "~" H 3200 6950 50  0001 C CNN
 	1    3200 6950
@@
 F 0 "L2" V 3390 7250 50  0000 C CNN
 F 1 "470" V 3299 7250 50  0000 C CNN
-F 2 "" H 3200 7250 50  0001 C CNN
+F 2 "_Generic:0603_IND" H 3200 7250 50  0001 C CNN
 F 3 "~" H 3200 7250 50  0001 C CNN
 	1    3200 7250
@@
 F 0 "D6" V 5654 3179 50  0000 L CNN
 F 1 "3.6v" V 5745 3179 50  0000 L CNN
-F 2 "" H 5700 3100 50  0001 C CNN
+F 2 "_Generic:SOD-523_DIODE" H 5700 3100 50  0001 C CNN
 F 3 "~" H 5700 3100 50  0001 C CNN
 	1    5700 3100
@@
 F 0 "D7" V 5954 3179 50  0000 L CNN
 F 1 "3.6v" V 6045 3179 50  0000 L CNN
-F 2 "" H 6000 3100 50  0001 C CNN
+F 2 "_Generic:SOD-523_DIODE" H 6000 3100 50  0001 C CNN
 F 3 "~" H 6000 3100 50  0001 C CNN
 	1    6000 3100
@@
 F 0 "D8" V 6254 3179 50  0000 L CNN
 F 1 "3.6v" V 6345 3179 50  0000 L CNN
-F 2 "" H 6300 3100 50  0001 C CNN
+F 2 "_Generic:SOD-523_DIODE" H 6300 3100 50  0001 C CNN
 F 3 "~" H 6300 3100 50  0001 C CNN
 	1    6300 3100
@@
 F 0 "D5" V 5354 3179 50  0000 L CNN
 F 1 "3.6v" V 5445 3179 50  0000 L CNN
-F 2 "" H 5400 3100 50  0001 C CNN
+F 2 "_Generic:SOD-523_DIODE" H 5400 3100 50  0001 C CNN
 F 3 "~" H 5400 3100 50  0001 C CNN
 	1    5400 3100
@@
 F 0 "D1" V 9004 2629 50  0000 L CNN
 F 1 "DNP" V 9095 2629 50  0000 L CNN
-F 2 "" H 9050 2550 50  0001 C CNN
+F 2 "_Generic:SOD-523_DIODE" H 9050 2550 50  0001 C CNN
 F 3 "~" H 9050 2550 50  0001 C CNN
 	1    9050 2550
@@
 F 0 "D2" V 9404 2629 50  0000 L CNN
 F 1 "DNP" V 9495 2629 50  0000 L CNN
-F 2 "" H 9450 2550 50  0001 C CNN
+F 2 "_Generic:SOD-523_DIODE" H 9450 2550 50  0001 C CNN
 F 3 "~" H 9450 2550 50  0001 C CNN
 	1    9450 2550
@@
 F 0 "D3" V 9804 2629 50  0000 L CNN
 F 1 "DNP" V 9895 2629 50  0000 L CNN
-F 2 "" H 9850 2550 50  0001 C CNN
+F 2 "_Generic:SOD-523_DIODE" H 9850 2550 50  0001 C CNN
 F 3 "~" H 9850 2550 50  0001 C CNN
 	1    9850 2550
@@
 F 0 "D4" V 10204 2629 50  0000 L CNN
 F 1 "DNP" V 10295 2629 50  0000 L CNN
-F 2 "" H 10250 2550 50  0001 C CNN
+F 2 "_Generic:SOD-523_DIODE" H 10250 2550 50  0001 C CNN
 F 3 "~" H 10250 2550 50  0001 C CNN
 	1    10250 2550

Commit message: layout test
Parts:
- J62: renamed from J41; footprint (none) -> _Generic:JST_XH_2P
- J63: renamed from J42; footprint (none) -> _Generic:JST_XH_2P
- J64: renamed from J47; footprint (none) -> _Generic:JST_XH_4P
- J65: renamed from J48; footprint (none) -> _Generic:JST_XH_4P
- J66: renamed from J54; footprint (none) -> _Generic:JST_XH_3P
- J67: renamed from J55; footprint (none) -> _Generic:JST_XH_3P
- J68: renamed from J56; footprint (none) -> _Generic:JST_XH_3P
- J69: renamed from J57; footprint (none) -> _Generic:JST_XH_3P
- J70: renamed from J49; footprint (none) -> _Generic:JST_XH_4P
- J71: renamed from J50; footprint (none) -> _Generic:JST_XH_2P
- J72: renamed from J51; footprint (none) -> _Generic:JST_XH_2P
- J73: renamed from J52; footprint (none) -> _Generic:JST_XH_2P
- J74: renamed from J53; footprint (none) -> _Generic:JST_XH_2P
- J75: renamed from J43; footprint (none) -> _Generic:PinHeader_2.54mm_1P
- J76: renamed from J44; footprint (none) -> _Generic:PinHeader_2.54mm_1P
- J77: renamed from J45; footprint (none) -> _Generic:PinHeader_2.54mm_1P
- J78: renamed from J46; footprint (none) -> _Generic:PinHeader_2.54mm_1P
- renumbered C18 to C45, C20 to C46, C21 to C47, C19 to C48, C22 to C49, C23 to C50, C24 to C51, C25 to C52, C26 to C53, C30 to C54, C31 to C55, C32 to C56, C33 to C57, C27 to C58, C28 to C59, C29 to C60, C34 to C61, D8 to D10, D1 to D11, D2 to D12, D3 to D13, D4 to D14, D5 to D7, D6 to D8, D7 to D9, J39 to J60, J40 to J61, JP14 to JP15, JP15 to JP16, JP20 to JP17, JP16 to JP18, JP17 to JP19, JP18 to JP20, JP19 to JP21, L1 to L4, L2 to L5, L3 to L6, L4 to L7, Q1 to Q2, R8 to R21, R10 to R22, R9 to R23, R11 to R24, R12 to R25, R13 to R26, R14 to R27, R15 to R28, R16 to R29, R17 to R30, R18 to R31, R30 to R32, R31 to R33, R19 to R34, R33 to R35, R35 to R36, R24 to R37, R37 to R38, R38 to R39, R39 to R40, R40 to R41, R29 to R42, R20 to R43, R32 to R44, R21 to R45, R34 to R46, R22 to R47, R36 to R48, R23 to R49, R41 to R50, R25 to R51, R26 to R52, R27 to R53, R28 to R54, U2 to U5, U3 to U6

Commit message: fuses
Parts:
- J60: footprint (none) -> _Generic:TYPE-C-31-M-12
- JP15, JP18, JP19, JP20, JP21: footprint (none) -> _Generic:Solder Jumper 2P
- JP16: footprint (none) -> _Generic:Solder Jumper 3P
Changed lines of the file:
@@
 F 0 "J60" H 1205 3267 50  0000 C CNN
 F 1 "USB_C_Receptacle" H 1205 3176 50  0000 C CNN
-F 2 "" H 1250 2000 50  0001 C CNN
+F 2 "_Generic:TYPE-C-31-M-12" H 1250 2000 50  0001 C CNN
 F 3 "https://www.usb.org/sites/default/files/documents/usb_type-c.zip" H 1250 2000 50  0001 C CNN
 	1    1100 2000
@@
 F 0 "JP18" V 9050 4568 50  0000 L CNN
 F 1 "SolderJumper_2_Open" H 9050 4500 50  0001 C CNN
-F 2 "" H 9050 4500 50  0001 C CNN
+F 2 "_Generic:Solder Jumper 2P" H 9050 4500 50  0001 C CNN
 F 3 "~" H 9050 4500 50  0001 C CNN
 	1    9050 4500
@@
 F 0 "JP19" V 9450 4568 50  0000 L CNN
 F 1 "SolderJumper_2_Open" H 9450 4500 50  0001 C CNN
-F 2 "" H 9450 4500 50  0001 C CNN
+F 2 "_Generic:Solder Jumper 2P" H 9450 4500 50  0001 C CNN
 F 3 "~" H 9450 4500 50  0001 C CNN
 	1    9450 4500
@@
 F 0 "JP20" V 9850 4568 50  0000 L CNN
 F 1 "SolderJumper_2_Open" H 9850 4500 50  0001 C CNN
-F 2 "" H 9850 4500 50  0001 C CNN
+F 2 "_Generic:Solder Jumper 2P" H 9850 4500 50  0001 C CNN
 F 3 "~" H 9850 4500 50  0001 C CNN
 	1    9850 4500
@@
 F 0 "JP21" V 10250 4568 50  0000 L CNN
 F 1 "SolderJumper_2_Open" H 10250 4500 50  0001 C CNN
-F 2 "" H 10250 4500 50  0001 C CNN
+F 2 "_Generic:Solder Jumper 2P" H 10250 4500 50  0001 C CNN
 F 3 "~" H 10250 4500 50  0001 C CNN
 	1    10250 4500
@@
 F 0 "JP16" V 6453 4750 50  0000 C CNN
 F 1 "SolderJumper_3_Open" H 6300 4750 50  0001 C CNN
-F 2 "" H 6300 4750 50  0001 C CNN
+F 2 "_Generic:Solder Jumper 3P" H 6300 4750 50  0001 C CNN
 F 3 "~" H 6300 4750 50  0001 C CNN
 	1    6300 4750
@@
 F 0 "JP15" H 2850 1113 50  0000 C CNN
 F 1 "SolderJumper_2_Open" H 2850 1000 50  0001 C CNN
-F 2 "" H 2850 1000 50  0001 C CNN
+F 2 "_Generic:Solder Jumper 2P" H 2850 1000 50  0001 C CNN
 F 3 "~" H 2850 1000 50  0001 C CNN
 	1    2850 1000

Commit message: continue routing
Parts:
- removed J70: Conn_01x04, _Generic:JST_XH_4P, symbol Connector_Generic:Conn_01x04
Other:
- note removed: "Serial"
Changed lines of the file:
@@
 Wire Wire Line
 	5850 4650 5850 4800
-Wire Wire Line
-	9300 5950 9800 5950
-Wire Wire Line
-	9800 5850 9300 5850
-Wire Wire Line
-	9300 5750 9800 5750
-$Comp
-L #Power:GND #PWR?
-U 1 1 6017E91A
-P 9700 6150
-AR Path="/5AF7E834/6017E91A" Ref="#PWR?"  Part="1"
-AR Path="/5AF7E834/5C3B9892/6017E91A" Ref="#PWR?"  Part="1"
-AR Path="/5AF7E834/6043293F/6017E91A" Ref="#PWR?"  Part="1"
-AR Path="/5C3B9892/6017E91A" Ref="#PWR068"  Part="1"
-F 0 "#PWR068" H 9700 5900 50  0001 C CNN
-F 1 "GND" H 9700 6000 50  0001 C CNN
-F 2 "" H 9700 6150 50  0001 C CNN
-F 3 "" H 9700 6150 50  0001 C CNN
-	1    9700 6150
-	-1   0    0    -1
-$EndComp
-Wire Wire Line
-	9700 6150 9700 6050
-Wire Wire Line
-	9700 6050 9800 6050
-Text HLabel 9300 5750 0    50   Input ~ 0
-TXD
-Text HLabel 9300 5850 0    50   Output ~ 0
-RXD
-Text HLabel 9300 5950 0    50   Input ~ 0
-ISP_BOOT
 Text HLabel 5200 1650 0    50   Output ~ 0
 ENDSTOP1
@@
 	6450 4750 6400 4750
 Connection ~ 6450 4750
-$Comp
-L Connector_Generic:Conn_01x04 J70
-U 1 1 5CF11272
-P 10000 5850
-F 0 "J70" H 10080 5796 50  0000 L CNN
-F 1 "Conn_01x04" H 10080 5751 50  0001 L CNN
-F 2 "_Generic:JST_XH_4P" H 10000 5850 50  0001 C CNN
-F 3 "~" H 10000 5850 50  0001 C CNN
-	1    10000 5850
-	1    0    0    -1
-$EndComp
 $Comp
 L Device:R R?
@@
 Text Notes 5500 4100 0    100  ~ 20
 I2C
-Text Notes 8050 5450 0    100  ~ 20
-Serial
 Wire Notes Line
 	8000 3050 11150 3050

Commit message: continue routing
Parts:
- removed J68, J69: Conn_01x03, _Generic:JST_XH_3P, symbol Connector_Generic:Conn_01x03
- added J46, J47: Conn_01x03, _Generic:JST_XH_3P, symbol Connector_Generic:Conn_01x03
- added JP43, JP44, JP45: SolderJumper_4_Open, _Generic:SolderJumper_JST, symbol #PCB_Only:SolderJumper_4_Open
- J61: footprint (none) -> _Generic:HYC77-TF09-200
- JP17: footprint (none) -> _Generic:SolderJumper_JST
- R33: value 47k -> 4.7k
- R40: value 4.7k -> 47k
Connections:
- net +12V: now also JP43.3 (O2), JP44.3 (O2), JP45.3 (O2)
- net +24V: now also JP43.4 (O4), JP44.4 (O4), JP45.4 (O4)
- net +3V3: now also R40.1; no longer R33.1
- net +5V: now also JP43.2 (O1), JP44.2 (O1), JP45.2 (O1)
- net ENDSTOP3: now also D7.1 (K), R32.2, R33.1; no longer D8.1 (K), R33.2, R40.1
- net ENDSTOP4: now also D8.1 (K), R40.2; no longer D7.1 (K), R32.2
- net GND: now also J46.2 (Pin_2), J47.2 (Pin_2)
- net at R41.2: now also J47.3 (Pin_3)
- new net: C54.1, J66.1 (Pin_1), JP17.1 (IN)
- new net: C55.1, J67.1 (Pin_1), JP43.1 (IN)
- new net: C56.1, J46.1 (Pin_1), JP44.1 (IN)
- new net: J46.3 (Pin_3), R33.2
- new net: C57.1, J47.1 (Pin_1), JP45.1 (IN)
Other:
- moved on the sheet: C54, C55, C58, C59, C60, C61, D10, D11, D12, D13, D14, D9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

Commit message: continue routing
Parts:
- removed D11, D12, D13, D14: DNP, _Generic:SOD-523_DIODE, symbol Device:D_Zener
- removed J64, J65: Conn_01x04, _Generic:JST_XH_4P, symbol Connector_Generic:Conn_01x04
- removed J75, J76, J77, J78: Conn_01x01, _Generic:PinHeader_2.54mm_1P, symbol #Connector:Conn_01x01
- removed R43, R45, R47, R49: DNP, _Generic:0603_RES, symbol Device:R
- removed R51, R52, R53, R54: 0R, _Generic:0603_RES, symbol Device:R
- added C198: 10u, _Generic:0603_CAP, symbol Device:C_Small
- added C199: 220u, Capacitor_SMD:CP_Elec_6.3x7.7, symbol Device:CP1_Small
Connections:
- net GND: now also J61.10 (DET_A), C198.2, C199.2; no longer J61.9 (DET_B)
- net SD_DETECT: now also J61.9 (DET_B); no longer J61.10 (DET_A)
- net VBUS: now also C198.1, C199.1
Other:
- note removed: "Generic IOs"
- moved on the sheet: C46, C50, C51, JP15, Q2, R21, R22, R24, R25, R26, R28

Commit message: PCB V1
Parts:
- removed JP16: SolderJumper_3_Open, _Generic:Solder Jumper 3P, symbol #PCB_Only:SolderJumper_3_Open
- removed R37, R42: 4.7k, _Generic:0603_RES, symbol Device:R
- R28: value 50k -> 47k
Other:
- note removed: "I2C"
- moved on the sheet: C198, C199, C46, C50, C51, C54, C55, C56, C57, C58, C59, C60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
