File: hardware/kajikia/output.sch (KiCad schematic (older format))
At the start: 80 parts

Commit message: power
Parts:
- removed C?: 100n, symbol Device:C_Small
- removed C?: 10u, symbol Device:C_Small
- removed D? (x2): LED, symbol Device:LED_Small
- removed D? (x8): D_Schottky, symbol Device:D_Schottky
- removed J?: Screw_Terminal_01x04, symbol Connector:Screw_Terminal_01x04
- removed J? (x8): Conn_01x03, symbol Connector_Generic:Conn_01x03
- removed JP? (x8): SolderJumper_3_Open, symbol #PCB_Only:SolderJumper_3_Open
- removed JP? (x8): SolderJumper_4_Open, symbol #PCB_Only:SolderJumper_4_Open
- removed Q? (x2): AON6144, symbol Device:Q_NMOS_SGD
- removed Q? (x8): AO3400, symbol Device:Q_NMOS_GSD
- removed R? (x2): 10, symbol Device:R
- removed R? (x10): 1k, symbol Device:R
- removed R? (x8): 50k, symbol Device:R
- removed U?: IR4427S, symbol Driver_FET:MIC4427
- added C? (x12): 4.7u, symbol Device:C_Small
- added C? (x2): 68u, symbol Device:CP1_Small
- added C?: 100n, symbol Device:C_Small
- added C?: 10u, symbol Device:C_Small
- added D17, D? (x7): 3.6v, symbol Device:D_Zener
- added D? (x2): LED, symbol Device:LED_Small
- added F1, F2, F? (x2): FUSE, symbol Device:Fuse
- added J58, J? (x7): Conn_01x03, symbol Connector_Generic:Conn_01x03
- added J?: Screw_Terminal_01x04, symbol Connector:Screw_Terminal_01x04
- added JP20, JP? (x7): SolderJumper_3_Open, symbol #PCB_Only:SolderJumper_3_Open
- added JP23, JP? (x7): SolderJumper_4_Open, symbol #PCB_Only:SolderJumper_4_Open
- added Q2, Q? (x7): AO3400, symbol Device:Q_NMOS_GSD
- added Q? (x2): AON6144, symbol Device:Q_NMOS_SGD
- added R50, R? (x9): 1k, symbol Device:R
- added R51, R? (x7): 50k, symbol Device:R
- added R? (x2): 10, symbol Device:R
- added U?: IR4427S, symbol Driver_FET:MIC4427
- gave numbers to parts that had none: 12
Connections:
- net +12V: now also C?.1, C?.1, JP23.3 (O2), JP?.3 (O2), JP?.3 (O2), JP?.3 (O2), JP?.3 (O2), JP?.3 (O2), JP?.3 (O2), JP?.3 (O2), U?.6 (V+)
- net +24V: now also C?.1, C?.1, F1.1, F2.1, F?.1, F?.1, JP23.4 (O4), JP?.4 (O4), JP?.4 (O4), JP?.4 (O4), JP?.4 (O4), JP?.4 (O4), JP?.4 (O4), JP?.4 (O4); no longer J61.2 (Pin_2), J61.4 (Pin_4)
- net +3V3: now also R?.1, R?.1
- net +5V: now also JP23.2 (O1), JP?.2 (O1), JP?.2 (O1), JP?.2 (O1), JP?.2 (O1), JP?.2 (O1), JP?.2 (O1), JP?.2 (O1)
- net GND: now also C?.2, C?.2, C?.2, C?.2, C?.2, C?.2, C?.2, C?.2, C?.2, C?.2, C?.2, C?.2, C?.2, C?.2, C?.2, C?.2, D17.2 (A), D?.2 (A), D?.2 (A), D?.2 (A), D?.2 (A), D?.2 (A), D?.2 (A), D?.2 (A), J58.2 (Pin_2), J?.2 (Pin_2), J?.2 (Pin_2), J?.2 (Pin_2), J?.2 (Pin_2), J?.2 (Pin_2), J?.2 (Pin_2), J?.2 (Pin_2), Q2.2 (S), Q?.1 (S), Q?.1 (S), Q?.2 (S), Q?.2 (S), Q?.2 (S), Q?.2 (S), Q?.2 (S), Q?.2 (S), Q?.2 (S), R51.1, R?.1, R?.1, R?.1, R?.1, R?.1, R?.1, R?.1, U?.3 (GND)
- net HV_IO1: now also D17.1 (K), R50.1
- net HV_IO2: now also D?.1 (K), R?.1
- net HV_IO3: now also D?.1 (K), R?.1
- net HV_IO4: now also D?.1 (K), R?.1
- net HV_IO5: now also D?.1 (K), R?.1
- net HV_IO6: now also D?.1 (K), R?.1
- net HV_IO7: now also D?.1 (K), R?.1
- net HV_IO8: now also D?.1 (K), R?.1
- net POWER_OUT3: now also U?.2 (IN_A)
- net POWER_OUT4: now also U?.4 (IN_B)
- net at D20.1 (K), Q5.3 (D): now also J61.2 (Pin_2); no longer J61.1 (Pin_1)
- net at D21.1 (K), Q6.3 (D): now also J61.4 (Pin_4); no longer J61.3 (Pin_3)
- new net: C?.1, J58.1 (Pin_1), JP23.1 (IN)
- new net: C?.1, F1.2, J61.3 (Pin_3)
- new net: C?.1, F2.2, J61.1 (Pin_1)
- new net: JP?.2 (C), R?.2 (x7)
- new net: J?.3 (Pin_3), JP?.1 (A), Q?.3 (D) (x7)
- new net: JP?.3 (B), Q?.1 (G), R?.2 (x7)
- new net: C?.1, J?.1 (Pin_1), JP?.1 (IN) (x7)
- new net: C?.1, F?.2, J?.1 (Pin_1)
- new net: D?.1 (K), J?.2 (Pin_2), Q?.3 (D)
- new net: C?.1, F?.2, J?.3 (Pin_3)
- new net: D?.1 (K), J?.4 (Pin_4), Q?.3 (D)
- new net: Q?.2 (G), R?.1 (x2)
- new net: R?.2, U?.5 (OUT_B)
- new net: R?.2, U?.7 (OUT_A)
- new net: D?.2 (A), R?.2 (x2)
- new net: JP20.2 (C), R50.2
- new net: J58.3 (Pin_3), JP20.1 (A), Q2.3 (D)
- new net: JP20.3 (B), Q2.1 (G), R51.2
Other:
- moved on the sheet: C53, C54, D20, D21, J61, Q5, Q6, R56, R57, R58, R59, U4

Commit message: fancy
Parts:
- C35: renamed from C53; footprint (none) -> _Generic:0603_CAP
- C36: renamed from C54; footprint (none) -> _Generic:0603_CAP
- C37, C38, C39, C41, C42, C43, C44, C45, C48, C49, C51, C52: renamed from C?; footprint (none) -> _Generic:0805_CAP
- C46, C47: renamed from C?; footprint (none) -> _Generic:0603_CAP
- D12: renamed from D20; footprint (none) -> _Generic:0603_LED
- D13: renamed from D21; footprint (none) -> _Generic:0603_LED
- D19, D20: renamed from D?; footprint (none) -> _Generic:0603_LED
- R42: renamed from R50; footprint (none) -> _Generic:0603_RES
- R43: renamed from R51; footprint (none) -> _Generic:0603_RES
- R44, R45, R46, R47, R52, R53, R54, R55, R56, R57, R58, R59, R60, R61, R64, R65: renamed from R?; footprint (none) -> _Generic:0603_RES
- R48: renamed from R56; value 10 -> 10R; footprint (none) -> _Generic:0603_RES
- R49: renamed from R57; value 10 -> 10R; footprint (none) -> _Generic:0603_RES
- R50: renamed from R58; footprint (none) -> _Generic:0603_RES
- R51: renamed from R59; footprint (none) -> _Generic:0603_RES
- R62, R63: renamed from R?; value 10 -> 10R; footprint (none) -> _Generic:0603_RES
- gave numbers to parts that had none: 43
- renumbered D17 to D9, JP20 to JP21, JP23 to JP24
Other:
- note added: "High Power Outputs"
- note added: "Medium Power Outputs"
- moved on the sheet: C35, C36, C40, C41, C42, C46, C47, C50, C51, C52, D12, D13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

Commit message: footprints
Parts:
- C40, C50: footprint (none) -> Capacitor_SMD:CP_Elec_8x10
- D10, D11, D14, D15, D16, D17, D18, D9: footprint (none) -> _Generic:SOD-523_DIODE
- Q10, Q13, Q5, Q6: footprint (none) -> _Generic:DFN5x6-8
- Q11, Q12, Q2, Q3, Q4, Q7, Q8, Q9: footprint (none) -> _Generic:SOT-23
- U4, U5: footprint (none) -> _Generic:SO-8
Changed lines of the file:
@@
 F 0 "Q6" H 4205 2346 50  0000 L CNN
 F 1 "AON6144" H 4205 2255 50  0000 L CNN
-F 2 "" H 4200 2400 50  0001 C CNN
+F 2 "_Generic:DFN5x6-8" H 4200 2400 50  0001 C CNN
 F 3 "~" H 4000 2300 50  0001 C CNN
 	1    4000 2300
@@
 F 0 "Q5" H 3655 2046 50  0000 L CNN
 F 1 "AON6144" H 3655 1955 50  0000 L CNN
-F 2 "" H 3650 2100 50  0001 C CNN
+F 2 "_Generic:DFN5x6-8" H 3650 2100 50  0001 C CNN
 F 3 "~" H 3450 2000 50  0001 C CNN
 	1    3450 2000
@@
 F 0 "U4" H 2000 2550 50  0000 C CNN
 F 1 "IR4427S" H 2550 2550 50  0000 C CNN
-F 2 "" H 2250 1900 50  0001 C CNN
+F 2 "_Generic:SO-8" H 2250 1900 50  0001 C CNN
 F 3 "http://ww1.microchip.com/downloads/en/DeviceDoc/mic4426.pdf" H 2250 1900 50  0001 C CNN
 	1    2250 2200
@@
 F 0 "Q2" V 2750 4200 50  0000 C CNN
 F 1 "AO3400" V 2841 4200 50  0000 C CNN
-F 2 "" H 2700 4300 50  0001 C CNN
+F 2 "_Generic:SOT-23" H 2700 4300 50  0001 C CNN
 F 3 "~" H 2500 4200 50  0001 C CNN
 	1    2500 4200
@@
 F 0 "D9" V 1204 4179 50  0000 L CNN
 F 1 "3.6v" V 1295 4179 50  0000 L CNN
-F 2 "" H 1250 4100 50  0001 C CNN
+F 2 "_Generic:SOD-523_DIODE" H 1250 4100 50  0001 C CNN
 F 3 "~" H 1250 4100 50  0001 C CNN
 	1    1250 4100
@@
 F 0 "C40" H 4741 1346 50  0000 L CNN
 F 1 "68u" H 4741 1255 50  0000 L CNN
-F 2 "" H 4650 1300 50  0001 C CNN
+F 2 "Capacitor_SMD:CP_Elec_8x10" H 4650 1300 50  0001 C CNN
 F 3 "~" H 4650 1300 50  0001 C CNN
 	1    4650 1300
@@
 F 0 "Q7" V 5750 4200 50  0000 C CNN
 F 1 "AO3400" V 5841 4200 50  0000 C CNN
-F 2 "" H 5700 4300 50  0001 C CNN
+F 2 "_Generic:SOT-23" H 5700 4300 50  0001 C CNN
 F 3 "~" H 5500 4200 50  0001 C CNN
 	1    5500 4200
@@
 F 0 "D14" V 4204 4179 50  0000 L CNN
 F 1 "3.6v" V 4295 4179 50  0000 L CNN
-F 2 "" H 4250 4100 50  0001 C CNN
+F 2 "_Generic:SOD-523_DIODE" H 4250 4100 50  0001 C CNN
 F 3 "~" H 4250 4100 50  0001 C CNN
 	1    4250 4100
@@
 F 0 "Q8" V 5750 5700 50  0000 C CNN
 F 1 "AO3400" V 5841 5700 50  0000 C CNN
-F 2 "" H 5700 5800 50  0001 C CNN
+F 2 "_Generic:SOT-23" H 5700 5800 50  0001 C CNN
 F 3 "~" H 5500 5700 50  0001 C CNN
 	1    5500 5700
@@
 F 0 "D15" V 4204 5679 50  0000 L CNN
 F 1 "3.6v" V 4295 5679 50  0000 L CNN
-F 2 "" H 4250 5600 50  0001 C CNN
+F 2 "_Generic:SOD-523_DIODE" H 4250 5600 50  0001 C CNN
 F 3 "~" H 4250 5600 50  0001 C CNN
 	1    4250 5600
@@
 F 0 "Q9" V 5750 7200 50  0000 C CNN
 F 1 "AO3400" V 5841 7200 50  0000 C CNN
-F 2 "" H 5700 7300 50  0001 C CNN
+F 2 "_Generic:SOT-23" H 5700 7300 50  0001 C CNN
 F 3 "~" H 5500 7200 50  0001 C CNN
 	1    5500 7200
@@
 F 0 "D16" V 4204 7179 50  0000 L CNN
 F 1 "3.6v" V 4295 7179 50  0000 L CNN
-F 2 "" H 4250 7100 50  0001 C CNN
+F 2 "_Generic:SOD-523_DIODE" H 4250 7100 50  0001 C CNN
 F 3 "~" H 4250 7100 50  0001 C CNN
 	1    4250 7100
@@
 F 0 "Q3" V 2750 5700 50  0000 C CNN
 F 1 "AO3400" V 2841 5700 50  0000 C CNN
-F 2 "" H 2700 5800 50  0001 C CNN
+F 2 "_Generic:SOT-23" H 2700 5800 50  0001 C CNN
 F 3 "~" H 2500 5700 50  0001 C CNN
 	1    2500 5700
@@
 F 0 "D10" V 1204 5679 50  0000 L CNN
 F 1 "3.6v" V 1295 5679 50  0000 L CNN
-F 2 "" H 1250 5600 50  0001 C CNN
+F 2 "_Generic:SOD-523_DIODE" H 1250 5600 50  0001 C CNN
 F 3 "~" H 1250 5600 50  0001 C CNN
 	1    1250 5600
@@
 F 0 "Q4" V 2750 7200 50  0000 C CNN
 F 1 "AO3400" V 2841 7200 50  0000 C CNN
-F 2 "" H 2700 7300 50  0001 C CNN
+F 2 "_Generic:SOT-23" H 2700 7300 50  0001 C CNN
 F 3 "~" H 2500 7200 50  0001 C CNN
 	1    2500 7200
@@
 F 0 "D11" V 1204 7179 50  0000 L CNN
 F 1 "3.6v" V 1295 7179 50  0000 L CNN
-F 2 "" H 1250 7100 50  0001 C CNN
+F 2 "_Generic:SOD-523_DIODE" H 1250 7100 50  0001 C CNN
 F 3 "~" H 1250 7100 50  0001 C CNN
 	1    1250 7100
@@
 F 0 "Q12" V 8750 5700 50  0000 C CNN
 F 1 "AO3400" V 8841 5700 50  0000 C CNN
-F 2 "" H 8700 5800 50  0001 C CNN
+F 2 "_Generic:SOT-23" H 8700 5800 50  0001 C CNN
 F 3 "~" H 8500 5700 50  0001 C CNN
 	1    8500 5700
@@
 F 0 "D18" V 7204 5679 50  0000 L CNN
 F 1 "3.6v" V 7295 5679 50  0000 L CNN
-F 2 "" H 7250 5600 50  0001 C CNN
+F 2 "_Generic:SOD-523_DIODE" H 7250 5600 50  0001 C CNN
 F 3 "~" H 7250 5600 50  0001 C CNN
 	1    7250 5600
@@
 F 0 "Q11" V 8750 4200 50  0000 C CNN
 F 1 "AO3400" V 8841 4200 50  0000 C CNN
-F 2 "" H 8700 4300 50  0001 C CNN
+F 2 "_Generic:SOT-23" H 8700 4300 50  0001 C CNN
 F 3 "~" H 8500 4200 50  0001 C CNN
 	1    8500 4200
@@
 F 0 "D17" V 7204 4179 50  0000 L CNN
 F 1 "3.6v" V 7295 4179 50  0000 L CNN
-F 2 "" H 7250 4100 50  0001 C CNN
+F 2 "_Generic:SOD-523_DIODE" H 7250 4100 50  0001 C CNN
 F 3 "~" H 7250 4100 50  0001 C CNN
 	1    7250 4100
@@
 F 0 "Q13" H 9205 2346 50  0000 L CNN
 F 1 "AON6144" H 9205 2255 50  0000 L CNN
-F 2 "" H 9200 2400 50  0001 C CNN
+F 2 "_Generic:DFN5x6-8" H 9200 2400 50  0001 C CNN
 F 3 "~" H 9000 2300 50  0001 C CNN
 	1    9000 2300
@@
 F 0 "Q10" H 8655 2046 50  0000 L CNN
 F 1 "AON6144" H 8655 1955 50  0000 L CNN
-F 2 "" H 8650 2100 50  0001 C CNN
+F 2 "_Generic:DFN5x6-8" H 8650 2100 50  0001 C CNN
 F 3 "~" H 8450 2000 50  0001 C CNN
 	1    8450 2000
@@
 F 0 "U5" H 7000 2550 50  0000 C CNN
 F 1 "IR4427S" H 7550 2550 50  0000 C CNN
-F 2 "" H 7250 1900 50  0001 C CNN
+F 2 "_Generic:SO-8" H 7250 1900 50  0001 C CNN
 F 3 "http://ww1.microchip.com/downloads/en/DeviceDoc/mic4426.pdf" H 7250 1900 50  0001 C CNN
 	1    7250 2200
@@
 F 0 "C50" H 9741 1346 50  0000 L CNN
 F 1 "68u" H 9741 1255 50  0000 L CNN
-F 2 "" H 9650 1300 50  0001 C CNN
+F 2 "Capacitor_SMD:CP_Elec_8x10" H 9650 1300 50  0001 C CNN
 F 3 "~" H 9650 1300 50  0001 C CNN
 	1    9650 1300

Commit message: layout test
Parts:
- F2: renamed from F1; footprint (none) -> _Generic:SMD_Fuseholder
- F3: renamed from F2; footprint (none) -> _Generic:SMD_Fuseholder
- F4: renamed from F3; footprint (none) -> _Generic:SMD_Fuseholder
- F5: renamed from F4; footprint (none) -> _Generic:SMD_Fuseholder
- J79: renamed from J58; footprint (none) -> _Generic:JST_XH_3P
- J80: renamed from J59; footprint (none) -> _Generic:JST_XH_3P
- J81: renamed from J60; footprint (none) -> _Generic:JST_XH_3P
- J82: renamed from J61; footprint (none) -> _Generic:KF635-4P
- J83: renamed from J62; footprint (none) -> _Generic:JST_XH_3P
- J84: renamed from J63; footprint (none) -> _Generic:JST_XH_3P
- J85: renamed from J64; footprint (none) -> _Generic:JST_XH_3P
- J86: renamed from J65; footprint (none) -> _Generic:JST_XH_3P
- J87: renamed from J66; footprint (none) -> _Generic:JST_XH_3P
- J88: renamed from J67; footprint (none) -> _Generic:KF635-4P
- renumbered C35 to C62, C36 to C63, C37 to C64, C38 to C65, C39 to C66, C40 to C67, C41 to C68, C42 to C69, C43 to C70, C44 to C71, C45 to C72, C46 to C73, C47 to C74, C48 to C75, C49 to C76, C50 to C77, C51 to C78, C52 to C79, D9 to D15, D10 to D16, D11 to D17, D12 to D18, D13 to D19, D14 to D20, D15 to D21, D16 to D22, D17 to D23, D18 to D24, D19 to D25, D20 to D26, JP21 to JP22, JP22 to JP23, JP23 to JP24, JP24 to JP25, JP25 to JP26, JP26 to JP27, JP27 to JP28, JP28 to JP29, JP29 to JP30, JP30 to JP31, JP31 to JP32, JP32 to JP33, JP33 to JP34, JP34 to JP35, JP35 to JP36, JP36 to JP37, Q9 to Q10, Q10 to Q11, Q11 to Q12, Q12 to Q13, Q13 to Q14, Q2 to Q3, Q3 to Q4, Q4 to Q5, Q5 to Q6, Q6 to Q7, Q7 to Q8, Q8 to Q9, R42 to R55, R43 to R56, R44 to R57, R45 to R58, R46 to R59, R47 to R60, R48 to R61, R49 to R62, R50 to R63, R51 to R64, R52 to R65, R53 to R66, R54 to R67, R55 to R68, R56 to R69, R57 to R70, R58 to R71, R59 to R72, R60 to R73, R61 to R74, R62 to R75, R63 to R76, R64 to R77, R65 to R78, U4 to U7, U5 to U8

Commit message: driver polys
Connections:
- net +24V: no longer C67.1, C77.1, F2.1, F3.1, F4.1, F5.1
- net GND: no longer C67.2, C68.2, C69.2, C77.2, C78.2, C79.2, Q11.1 (S), Q14.1 (S), Q6.1 (S), Q7.1 (S)
- new net DCIN+: C67.1, C77.1, F2.1, F3.1, F4.1, F5.1
- new net DCIN-: C67.2, C68.2, C69.2, C77.2, C78.2, C79.2, Q11.1 (S), Q14.1 (S), Q6.1 (S), Q7.1 (S)
Changed lines of the file:
@@
 $EndComp
-Wire Wire Line
-	3550 2650 2250 2650
 Wire Wire Line
 	3550 2200 3550 2650
@@
 Wire Wire Line
 	3800 2300 3050 2300
-Wire Wire Line
-	2250 2650 2250 2600
-Connection ~ 3550 2650
 Wire Wire Line
 	4100 2650 3550 2650
@@
 Wire Wire Line
 	4100 1950 5550 1950
-Wire Wire Line
-	2250 2700 2250 2650
-Connection ~ 2250 2650
 Text HLabel 1700 2100 0    50   Input ~ 0
 POWER_OUT1
@@
 Text HLabel 4150 6900 0    50   BiDi ~ 0
 HV_IO6
-$Comp
-L power:+24V #PWR092
-U 1 1 61250C08
-P 5050 1050
-F 0 "#PWR092" H 5050 900 50  0001 C CNN
-F 1 "+24V" H 5065 1223 50  0000 C CNN
-F 2 "" H 5050 1050 50  0001 C CNN
-F 3 "" H 5050 1050 50  0001 C CNN
-	1    5050 1050
-	1    0    0    -1
-$EndComp
 $Comp
 L Device:R R?
@@
 	5050 1850 5550 1850
 Wire Wire Line
-	5050 1050 5050 1100
-Wire Wire Line
 	5050 1100 5450 1100
 Wire Wire Line
@@
 Wire Wire Line
 	4650 1100 5050 1100
-$Comp
-L #Power:GND #PWR091
-U 1 1 5CBF343D
-P 4650 1500
-F 0 "#PWR091" H 4650 1250 50  0001 C CNN
-F 1 "GND" H 4650 1350 50  0001 C CNN
-F 2 "" H 4650 1500 50  0001 C CNN
-F 3 "" H 4650 1500 50  0001 C CNN
-	1    4650 1500
-	1    0    0    -1
-$EndComp
-Wire Wire Line
-	4650 1500 4650 1400
 Wire Wire Line
 	5450 2100 5450 1650
@@
 	5050 1850 5050 2100
 Connection ~ 5050 1850
-$Comp
-L #Power:GND #PWR093
-U 1 1 5CCF98B4
-P 5250 2450
-F 0 "#PWR093" H 5250 2200 50  0001 C CNN
-F 1 "GND" H 5250 2300 50  0001 C CNN
-F 2 "" H 5250 2450 50  0001 C CNN
-F 3 "" H 5250 2450 50  0001 C CNN
-	1    5250 2450
-	1    0    0    -1
-$EndComp
-Wire Wire Line
-	5250 2450 5250 2400
-Wire Wire Line
-	5050 2400 5050 2300
-Wire Wire Line
-	5450 2400 5450 2300
-Connection ~ 5250 2400
-Wire Wire Line
-	5250 2400 5450 2400
-Wire Wire Line
-	5050 2400 5250 2400
+Wire Wire Line
+	5050 2650 5050 2300
+Wire Wire Line
+	5450 2650 5450 2300
 Wire Wire Line
 	6700 2300 6850 2300
@@
 $EndComp
 Wire Wire Line
-	8550 2650 7250 2650
-Wire Wire Line
 	8550 2200 8550 2650
 Wire Wire Line
@@
 Wire Wire Line
 	8800 2300 8050 2300
-Wire Wire Line
-	7250 2650 7250 2600
-Connection ~ 8550 2650
 Wire Wire Line
 	9100 2650 8550 2650
@@
 Wire Wire Line
 	9100 1950 10550 1950
-Wire Wire Line
-	7250 2700 7250 2650
-Connection ~ 7250 2650
 Connection ~ 7900 1650
 Wire Wire Line
@@
 	8550 1100 8550 1150
 $Comp
-L power:+24V #PWR0121
-U 1 1 5CEA84BF
-P 10050 1050
-F 0 "#PWR0121" H 10050 900 50  0001 C CNN
-F 1 "+24V" H 10065 1223 50  0000 C CNN
-F 2 "" H 10050 1050 50  0001 C CNN
-F 3 "" H 10050 1050 50  0001 C CNN
-	1    10050 1050
-	1    0    0    -1
-$EndComp
-$Comp
 L Device:Fuse F5
 U 1 1 5CEA84C5
@@
 	10050 1850 10550 1850
 Wire Wire Line
-	10050 1050 10050 1100
-Wire Wire Line
-	10050 1100 10450 1100
-Wire Wire Line
 	10450 1100 10450 1150
 Connection ~ 10050 1100
@@
 Wire Wire Line
 	9650 1100 10050 1100
-$Comp
-L #Power:GND #PWR0120
-U 1 1 5CEA84F3
-P 9650 1500
-F 0 "#PWR0120" H 9650 1250 50  0001 C CNN
-F 1 "GND" H 9650 1350 50  0001 C CNN
-F 2 "" H 9650 1500 50  0001 C CNN
-F 3 "" H 9650 1500 50  0001 C CNN
-	1    9650 1500
-	1    0    0    -1
-$EndComp
-Wire Wire Line
-	9650 1500 9650 1400
 Wire Wire Line
 	10450 2100 10450 1650
@@
 	10050 1850 10050 2100
 Connection ~ 10050 1850
-$Comp
-L #Power:GND #PWR0122
-U 1 1 5CEA84FE
-P 10250 2450
-F 0 "#PWR0122" H 10250 2200 50  0001 C CNN
-F 1 "GND" H 10250 2300 50  0001 C CNN
-F 2 "" H 10250 2450 50  0001 C CNN
-F 3 "" H 10250 2450 50  0001 C CNN
-	1    10250 2450
-	1    0    0    -1
-$EndComp
-Wire Wire Line
-	10250 2450 10250 2400
-Wire Wire Line
-	10050 2400 10050 2300
-Wire Wire Line
-	10450 2400 10450 2300
-Connection ~ 10250 2400
-Wire Wire Line
-	10250 2400 10450 2400
-Wire Wire Line
-	10050 2400 10250 2400
+Wire Wire Line
+	10050 2650 10050 2300
+Wire Wire Line
+	10450 2650 10450 2300
 Wire Wire Line
 	1250 5800 1550 5800
@@
 Text Notes 550  750  0    100  ~ 20
 High Power Outputs
+Text GLabel 5500 1100 2    50   Input ~ 0
+DCIN+
+Wire Wire Line
+	5500 1100 5450 1100
+Connection ~ 5450 1100
+Text GLabel 5500 2650 2    50   Input ~ 0
+DCIN-
+Wire Wire Line
+	5500 2650 5450 2650
+Connection ~ 5450 2650
+Wire Wire Line
+	5050 2650 5450 2650
+Text GLabel 10500 1100 2    50   Input ~ 0
+DCIN+
+Wire Wire Line
+	10050 1100 10450 1100
+Connection ~ 10450 1100
+Wire Wire Line
+	10450 1100 10500 1100
+Text GLabel 10500 2650 2    50   Input ~ 0
+DCIN-
+Wire Wire Line
+	10500 2650 10450 2650
+Connection ~ 10450 2650
+Wire Wire Line
+	10050 2650 10450 2650
+Wire Wire Line
+	7250 2600 7250 2700
+Wire Wire Line
+	9100 2650 9650 2650
+Connection ~ 9100 2650
+Connection ~ 10050 2650
+Wire Wire Line
+	9650 1400 9650 2650
+Connection ~ 9650 2650
+Wire Wire Line
+	9650 2650 10050 2650
+Wire Wire Line
+	4650 2650 5050 2650
+Wire Wire Line
+	4650 1400 4650 2650
+Connection ~ 5050 2650
+Wire Wire Line
+	2250 2600 2250 2700
+Wire Wire Line
+	4100 2650 4650 2650
+Connection ~ 4100 2650
+Connection ~ 4650 2650
 $EndSCHEMATC

Commit message: fuses
Parts:
- removed C78: 4.7u, _Generic:0805_CAP, symbol Device:C_Small
- removed D26: LED, _Generic:0603_LED, symbol Device:LED_Small
- removed F5: FUSE, _Generic:SMD_Fuseholder, symbol Device:Fuse
- removed J88: Screw_Terminal_01x04, _Generic:KF635-4P, symbol Connector:Screw_Terminal_01x04
- removed Q14: AON6144, _Generic:DFN5x6-8, symbol Device:Q_NMOS_SGD
- added C192: 4.7u, _Generic:1210_CAP, symbol Device:C_Small
- added D26: MSK4010, _Generic:SOD-523_DIODE, symbol Device:D_Schottky
- added J88: Screw_Terminal_01x02, _Generic:KF635-2P, symbol Connector:Screw_Terminal_01x02
- added LS1: Buzzer, symbol Device:Speaker
- added Q14: AO3400, _Generic:SOT-23, symbol Device:Q_NMOS_GSD
- C67, C77: value 68u -> 220u; footprint Capacitor_SMD:CP_Elec_8x10 -> Capacitor_SMD:CP_Elec_6.3x7.7
- C68, C69, C79: footprint _Generic:0805_CAP -> _Generic:1210_CAP
- F2, F3, F4: value FUSE -> Fuse
- JP22, JP23, JP24, JP28, JP29, JP30, JP34, JP35: footprint (none) -> _Generic:Solder Jumper 3P
- R76: value 10R -> 1k
- R78: value 1k -> 0R
Connections:
- net +24V: now also C67.1, C68.1, C69.1, C77.1, C79.1, J82.2 (Pin_2), J82.4 (Pin_4), C192.1, J88.2 (Pin_2)
- net DCIN-: now also C192.2
- net GND: now also Q14.2 (S)
- net at D25.1 (K), Q11.3 (D): now also F4.2
- net at R76.1: now also Q14.1 (G)
- net at U8.5 (OUT_B): no longer R76.2
- net at R78.2: now also D26.1 (K), LS1.1
- net at D18.1 (K), Q6.3 (D): now also F2.2; no longer J82.2 (Pin_2)
- net at D19.1 (K), Q7.3 (D): now also F3.2; no longer J82.4 (Pin_4)
- net at Q7.2 (G): now also R61.1; no longer R62.1
- net at Q6.2 (G): now also R62.1; no longer R61.1
- removed net DCIN+: C67.1, C77.1, F2.1, F3.1, F4.1
- net POWER_OUT4: no longer names the net of U8.4 (IN_B)
- new net: F4.1, J88.1 (Pin_1)
- new net: F2.1, J82.1 (Pin_1)
- new net: F3.1, J82.3 (Pin_3)
- new net: D26.2 (A), LS1.2, Q14.3 (D)
- new net BUZZER: R76.2
- no-connect marks 0 -> 2
Other:
- note added: "Buzzer"
- moved on the sheet: C62, C63, C67, C68, C69, C73, C74, C79, D18, D19, D25, J82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

Commit message: continue routing
Parts:
- JP25, JP26, JP27, JP31, JP32, JP33, JP36, JP37: footprint (none) -> _Generic:SolderJumper_JST
- LS1: footprint (none) -> _Generic:Buzzer-7525
Changed lines of the file:
@@
 F 0 "JP25" H 3358 3850 50  0000 L CNN
 F 1 "SolderJumper_4_Open" H 3200 3850 50  0001 C CNN
-F 2 "" H 3200 3850 50  0001 C CNN
+F 2 "_Generic:SolderJumper_JST" H 3200 3850 50  0001 C CNN
 F 3 "~" H 3200 3850 50  0001 C CNN
 	1    3200 3850
@@
 F 0 "JP31" H 6358 3850 50  0000 L CNN
 F 1 "SolderJumper_4_Open" H 6200 3850 50  0001 C CNN
-F 2 "" H 6200 3850 50  0001 C CNN
+F 2 "_Generic:SolderJumper_JST" H 6200 3850 50  0001 C CNN
 F 3 "~" H 6200 3850 50  0001 C CNN
 	1    6200 3850
@@
 F 0 "JP32" H 6358 5350 50  0000 L CNN
 F 1 "SolderJumper_4_Open" H 6200 5350 50  0001 C CNN
-F 2 "" H 6200 5350 50  0001 C CNN
+F 2 "_Generic:SolderJumper_JST" H 6200 5350 50  0001 C CNN
 F 3 "~" H 6200 5350 50  0001 C CNN
 	1    6200 5350
@@
 F 0 "JP33" H 6358 6850 50  0000 L CNN
 F 1 "SolderJumper_4_Open" H 6200 6850 50  0001 C CNN
-F 2 "" H 6200 6850 50  0001 C CNN
+F 2 "_Generic:SolderJumper_JST" H 6200 6850 50  0001 C CNN
 F 3 "~" H 6200 6850 50  0001 C CNN
 	1    6200 6850
@@
 F 0 "JP26" H 3358 5350 50  0000 L CNN
 F 1 "SolderJumper_4_Open" H 3200 5350 50  0001 C CNN
-F 2 "" H 3200 5350 50  0001 C CNN
+F 2 "_Generic:SolderJumper_JST" H 3200 5350 50  0001 C CNN
 F 3 "~" H 3200 5350 50  0001 C CNN
 	1    3200 5350
@@
 F 0 "JP27" H 3358 6850 50  0000 L CNN
 F 1 "SolderJumper_4_Open" H 3200 6850 50  0001 C CNN
-F 2 "" H 3200 6850 50  0001 C CNN
+F 2 "_Generic:SolderJumper_JST" H 3200 6850 50  0001 C CNN
 F 3 "~" H 3200 6850 50  0001 C CNN
 	1    3200 6850
@@
 F 0 "JP37" H 9358 5350 50  0000 L CNN
 F 1 "SolderJumper_4_Open" H 9200 5350 50  0001 C CNN
-F 2 "" H 9200 5350 50  0001 C CNN
+F 2 "_Generic:SolderJumper_JST" H 9200 5350 50  0001 C CNN
 F 3 "~" H 9200 5350 50  0001 C CNN
 	1    9200 5350
@@
 F 0 "JP36" H 9358 3850 50  0000 L CNN
 F 1 "SolderJumper_4_Open" H 9200 3850 50  0001 C CNN
-F 2 "" H 9200 3850 50  0001 C CNN
+F 2 "_Generic:SolderJumper_JST" H 9200 3850 50  0001 C CNN
 F 3 "~" H 9200 3850 50  0001 C CNN
 	1    9200 3850
@@
 F 0 "LS1" H 10869 1796 50  0000 L CNN
 F 1 "Buzzer" H 10869 1705 50  0000 L CNN
-F 2 "" H 10700 1600 50  0001 C CNN
+F 2 "_Generic:Buzzer-7525" H 10700 1600 50  0001 C CNN
 F 3 "~" H 10690 1750 50  0001 C CNN
 	1    10700 1800
