File: hardware/kajikia/output.sch (KiCad schematic (older format))
At the start: 98 parts, among them J79 Conn_01x03, J80 Conn_01x03, J81 Conn_01x03, J82 Screw_Terminal_01x04, J83 Conn_01x03, J84 Conn_01x03, J85 Conn_01x03, J86 Conn_01x03, J87 Conn_01x03, J88 Screw_Terminal_01x02, Q10 AO3400, Q11 AON6144, Q12 AO3400, Q13 AO3400, Q14 AO3400, Q3 AO3400, Q4 AO3400, Q5 AO3400, Q6 AON6144, Q7 AON6144, Q8 AO3400, Q9 AO3400, U7 IR4427S, U8 IR4427S

Commit message: PCB V1
Parts:
- R56, R58, R60, R66, R68, R70, R72, R74: value 50k -> 47k
Connections:
- net GND: now also U8.4 (IN_B)
- no-connect marks 2 -> 1
Changed lines of the file:
@@
 Text HLabel 2600 2400 0    50   Input ~ 0
 POWER_OUT3
-Text HLabel 9750 2350 0    50   Input ~ 0
-BUZZER
 Wire Wire Line
 	2600 1500 2700 1500
@@
 P 1750 4200
 F 0 "R56" V 1957 4200 50  0000 C CNN
-F 1 "50k" V 1866 4200 50  0000 C CNN
+F 1 "47k" V 1866 4200 50  0000 C CNN
 F 2 "_Generic:0603_RES" V 1680 4200 50  0001 C CNN
 F 3 "~" H 1750 4200 50  0001 C CNN
@@
 P 4750 4200
 F 0 "R66" V 4957 4200 50  0000 C CNN
-F 1 "50k" V 4866 4200 50  0000 C CNN
+F 1 "47k" V 4866 4200 50  0000 C CNN
 F 2 "_Generic:0603_RES" V 4680 4200 50  0001 C CNN
 F 3 "~" H 4750 4200 50  0001 C CNN
@@
 P 4750 5700
 F 0 "R68" V 4957 5700 50  0000 C CNN
-F 1 "50k" V 4866 5700 50  0000 C CNN
+F 1 "47k" V 4866 5700 50  0000 C CNN
 F 2 "_Generic:0603_RES" V 4680 5700 50  0001 C CNN
 F 3 "~" H 4750 5700 50  0001 C CNN
@@
 P 4750 7200
 F 0 "R70" V 4957 7200 50  0000 C CNN
-F 1 "50k" V 4866 7200 50  0000 C CNN
+F 1 "47k" V 4866 7200 50  0000 C CNN
 F 2 "_Generic:0603_RES" V 4680 7200 50  0001 C CNN
 F 3 "~" H 4750 7200 50  0001 C CNN
@@
 P 1750 5700
 F 0 "R58" V 1957 5700 50  0000 C CNN
-F 1 "50k" V 1866 5700 50  0000 C CNN
+F 1 "47k" V 1866 5700 50  0000 C CNN
 F 2 "_Generic:0603_RES" V 1680 5700 50  0001 C CNN
 F 3 "~" H 1750 5700 50  0001 C CNN
@@
 P 1750 7200
 F 0 "R60" V 1957 7200 50  0000 C CNN
-F 1 "50k" V 1866 7200 50  0000 C CNN
+F 1 "47k" V 1866 7200 50  0000 C CNN
 F 2 "_Generic:0603_RES" V 1680 7200 50  0001 C CNN
 F 3 "~" H 1750 7200 50  0001 C CNN
@@
 P 7750 5700
 F 0 "R74" V 7957 5700 50  0000 C CNN
-F 1 "50k" V 7866 5700 50  0000 C CNN
+F 1 "47k" V 7866 5700 50  0000 C CNN
 F 2 "_Generic:0603_RES" V 7680 5700 50  0001 C CNN
 F 3 "~" H 7750 5700 50  0001 C CNN
@@
 P 7750 4200
 F 0 "R72" V 7957 4200 50  0000 C CNN
-F 1 "50k" V 7866 4200 50  0000 C CNN
+F 1 "47k" V 7866 4200 50  0000 C CNN
 F 2 "_Generic:0603_RES" V 7680 4200 50  0001 C CNN
 F 3 "~" H 7750 4200 50  0001 C CNN
@@
 	9200 4000 9200 3950
 Wire Wire Line
-	9750 2350 9800 2350
-Wire Wire Line
 	2600 2400 2700 2400
 $Comp
 L #Power:GND #PWR?
 U 1 1 5CEA8429
-P 3100 2950
+P 3100 3000
 AR Path="/5AF7E834/5CEA8429" Ref="#PWR?"  Part="1"
 AR Path="/5AF7E834/606BF39C/5CEA8429" Ref="#PWR?"  Part="1"
 AR Path="/606BF39C/5CEA8429" Ref="#PWR0107"  Part="1"
-F 0 "#PWR0107" H 3100 2700 50  0001 C CNN
-F 1 "GND" H 3100 2800 50  0001 C CNN
-F 2 "" H 3100 2950 50  0001 C CNN
-F 3 "" H 3100 2950 50  0001 C CNN
-	1    3100 2950
-	1    0    0    -1
-$EndComp
-$Comp
-L power:+12V #PWR?
-U 1 1 5CEA8439
-P 8450 -2350
-AR Path="/5AF7E834/5CEA8439" Ref="#PWR?"  Part="1"
-AR Path="/5AF7E834/606BF39C/5CEA8439" Ref="#PWR?"  Part="1"
-AR Path="/606BF39C/5CEA8439" Ref="#PWR0106"  Part="1"
-F 0 "#PWR0106" H 8450 -2500 50  0001 C CNN
-F 1 "+12V" H 8465 -2177 50  0000 C CNN
-F 2 "" H 8450 -2350 50  0001 C CNN
-F 3 "" H 8450 -2350 50  0001 C CNN
-	1    8450 -2350
+F 0 "#PWR0107" H 3100 2750 50  0001 C CNN
+F 1 "GND" H 3100 2850 50  0001 C CNN
+F 2 "" H 3100 3000 50  0001 C CNN
+F 3 "" H 3100 3000 50  0001 C CNN
+	1    3100 3000
 	1    0    0    -1
 $EndComp
@@
 Wire Wire Line
 	6200 2100 6400 2100
-NoConn ~ 2700 2600
 NoConn ~ 3500 2600
-$Comp
-L Device:Speaker LS1
-U 1 1 5CB60C79
-P 10700 1800
-F 0 "LS1" H 10869 1796 50  0000 L CNN
-F 1 "Buzzer" H 10869 1705 50  0000 L CNN
-F 2 "_Generic:Buzzer-7525" H 10700 1600 50  0001 C CNN
-F 3 "~" H 10690 1750 50  0001 C CNN
-	1    10700 1800
-	1    0    0    -1
-$EndComp
-$Comp
-L Device:R R76
-U 1 1 5CC01ACE
-P 9950 2350
-F 0 "R76" V 9743 2350 50  0000 C CNN
-F 1 "1k" V 9834 2350 50  0000 C CNN
-F 2 "_Generic:0603_RES" V 9880 2350 50  0001 C CNN
-F 3 "~" H 9950 2350 50  0001 C CNN
-	1    9950 2350
-	0    1    1    0
-$EndComp
-Wire Wire Line
-	10100 2350 10150 2350
-$Comp
-L Device:Q_NMOS_GSD Q14
-U 1 1 5CC01FD3
-P 10350 2350
-F 0 "Q14" H 10555 2396 50  0000 L CNN
-F 1 "AO3400" H 10555 2305 50  0000 L CNN
-F 2 "_Generic:SOT-23" H 10550 2450 50  0001 C CNN
-F 3 "~" H 10350 2350 50  0001 C CNN
-	1    10350 2350
-	1    0    0    -1
-$EndComp
-$Comp
-L power:+3.3V #PWR0110
-U 1 1 5CC6115D
-P 10450 1250
-F 0 "#PWR0110" H 10450 1100 50  0001 C CNN
-F 1 "+3.3V" H 10465 1423 50  0000 C CNN
-F 2 "" H 10450 1250 50  0001 C CNN
-F 3 "" H 10450 1250 50  0001 C CNN
-	1    10450 1250
-	1    0    0    -1
-$EndComp
-Wire Wire Line
-	10450 1250 10450 1300
-$Comp
-L Device:D_Schottky D26
-U 1 1 5CC8149F
-P 9950 1850
-F 0 "D26" V 9904 1929 50  0000 L CNN
-F 1 "MSK4010" V 9995 1929 50  0000 L CNN
-F 2 "_Generic:SOD-523_DIODE" H 9950 1850 50  0001 C CNN
-F 3 "~" H 9950 1850 50  0001 C CNN
-	1    9950 1850
-	0    1    1    0
-$EndComp
-Wire Wire Line
-	9950 2000 9950 2050
-Wire Wire Line
-	9950 2050 10450 2050
-Wire Wire Line
-	10450 2050 10450 2150
-Wire Wire Line
-	9950 1700 9950 1650
-Wire Wire Line
-	9950 1650 10450 1650
-Wire Wire Line
-	10500 1800 10450 1800
-Wire Wire Line
-	10450 1800 10450 1650
-Connection ~ 10450 1650
-Wire Wire Line
-	10500 1900 10450 1900
-Wire Wire Line
-	10450 1900 10450 2050
-Connection ~ 10450 2050
-$Comp
-L Device:R R78
-U 1 1 5CFB2C79
-P 10450 1450
-F 0 "R78" H 10520 1496 50  0000 L CNN
-F 1 "0R" H 10520 1405 50  0000 L CNN
-F 2 "_Generic:0603_RES" V 10380 1450 50  0001 C CNN
-F 3 "~" H 10450 1450 50  0001 C CNN
-	1    10450 1450
-	1    0    0    -1
-$EndComp
-Wire Wire Line
-	10450 1600 10450 1650
-$Comp
-L #Power:GND #PWR0111
-U 1 1 5CFB318C
-P 10450 2600
-F 0 "#PWR0111" H 10450 2350 50  0001 C CNN
-F 1 "GND" H 10450 2450 50  0001 C CNN
-F 2 "" H 10450 2600 50  0001 C CNN
-F 3 "" H 10450 2600 50  0001 C CNN
-	1    10450 2600
-	1    0    0    -1
-$EndComp
-Wire Wire Line
-	10450 2600 10450 2550
 $Comp
 L Device:Q_NMOS_SGD Q?
@@
 Wire Notes Line
 	9300 3200 9300 550
-Text Notes 9400 750  0    100  ~ 20
-Buzzer
 Wire Wire Line
 	4500 1600 4500 1650
@@
 Wire Wire Line
 	5600 2700 6000 2700
-Wire Wire Line
-	8450 -2350 8450 -1750
 $Comp
 L #Power:GND #PWR?
@@
 	7500 2050 7500 2100
 Connection ~ 7500 2100
+Wire Wire Line
+	3100 2950 2650 2950
+Wire Wire Line
+	2650 2950 2650 2600
+Wire Wire Line
+	2650 2600 2700 2600
+Connection ~ 3100 2950
+Wire Wire Line
+	3100 2950 3100 3000
+Text Notes 9400 750  0    100  ~ 20
+Buzzer
+Wire Wire Line
+	10450 2600 10450 2550
+$Comp
+L #Power:GND #PWR0111
+U 1 1 5CFB318C
+P 10450 2600
+F 0 "#PWR0111" H 10450 2350 50  0001 C CNN
+F 1 "GND" H 10450 2450 50  0001 C CNN
+F 2 "" H 10450 2600 50  0001 C CNN
+F 3 "" H 10450 2600 50  0001 C CNN
+	1    10450 2600
+	1    0    0    -1
+$EndComp
+$Comp
+L Device:R R78
+U 1 1 5CFB2C79
+P 10450 1450
+F 0 "R78" H 10520 1496 50  0000 L CNN
+F 1 "0R" H 10520 1405 50  0000 L CNN
+F 2 "_Generic:0603_RES" V 10380 1450 50  0001 C CNN
+F 3 "~" H 10450 1450 50  0001 C CNN
+	1    10450 1450
+	1    0    0    -1
+$EndComp
+Wire Wire Line
+	10500 1900 10450 1900
+Wire Wire Line
+	10500 1800 10450 1800
+Wire Wire Line
+	10450 1600 10450 1650
+Wire Wire Line
+	10450 1800 10450 1650
+Connection ~ 10450 1650
+Wire Wire Line
+	9950 1650 10450 1650
+Wire Wire Line
+	9950 1700 9950 1650
+Wire Wire Line
+	10450 1900 10450 2050
+Wire Wire Line
+	10450 2050 10450 2150
+Connection ~ 10450 2050
+Wire Wire Line
+	9950 2050 10450 2050
+Wire Wire Line
+	9950 2000 9950 2050
+$Comp
+L Device:D_Schottky D26
+U 1 1 5CC8149F
+P 9950 1850
+F 0 "D26" V 9904 1929 50  0000 L CNN
+F 1 "MSK4010" V 9995 1929 50  0000 L CNN
+F 2 "_Generic:SOD-523_DIODE" H 9950 1850 50  0001 C CNN
+F 3 "~" H 9950 1850 50  0001 C CNN
+	1    9950 1850
+	0    1    1    0
+$EndComp
+Wire Wire Line
+	10450 1250 10450 1300
+$Comp
+L power:+3.3V #PWR0110
+U 1 1 5CC6115D
+P 10450 1250
+F 0 "#PWR0110" H 10450 1100 50  0001 C CNN
+F 1 "+3.3V" H 10465 1423 50  0000 C CNN
+F 2 "" H 10450 1250 50  0001 C CNN
+F 3 "" H 10450 1250 50  0001 C CNN
+	1    10450 1250
+	1    0    0    -1
+$EndComp
+$Comp
+L Device:Q_NMOS_GSD Q14
+U 1 1 5CC01FD3
+P 10350 2350
+F 0 "Q14" H 10555 2396 50  0000 L CNN
+F 1 "AO3400" H 10555 2305 50  0000 L CNN
+F 2 "_Generic:SOT-23" H 10550 2450 50  0001 C CNN
+F 3 "~" H 10350 2350 50  0001 C CNN
+	1    10350 2350
+	1    0    0    -1
+$EndComp
+Wire Wire Line
+	10100 2350 10150 2350
+$Comp
+L Device:R R76
+U 1 1 5CC01ACE
+P 9950 2350
+F 0 "R76" V 9743 2350 50  0000 C CNN
+F 1 "1k" V 9834 2350 50  0000 C CNN
+F 2 "_Generic:0603_RES" V 9880 2350 50  0001 C CNN
+F 3 "~" H 9950 2350 50  0001 C CNN
+	1    9950 2350
+	0    1    1    0
+$EndComp
+$Comp
+L Device:Speaker LS1
+U 1 1 5CB60C79
+P 10700 1800
+F 0 "LS1" H 10869 1796 50  0000 L CNN
+F 1 "Buzzer" H 10869 1705 50  0000 L CNN
+F 2 "_Generic:Buzzer-7525" H 10700 1600 50  0001 C CNN
+F 3 "~" H 10690 1750 50  0001 C CNN
+	1    10700 1800
+	1    0    0    -1
+$EndComp
+Wire Wire Line
+	9750 2350 9800 2350
+Text HLabel 9750 2350 0    50   Input ~ 0
+BUZZER
 $EndSCHEMATC
